Commit message: Fixed package names in urdf files

File: abb_irb4400_support/urdf/irb4400l30.urdf (robot description, URDF)
Before this commit: robot irb_4400_l30, 8 links, 7 joints
Links:
- link base_link: geometry collision mesh filename=package://abb_irb4400_support/meshes/irb4400l30/collision/b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; visual mesh filename=package://abb_irb4400_support/meshes/irb4400l30/visual/base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
- link link_1: geometry collision mesh filename=package://abb_irb4400_support/meshes/irb4400l30/collision/l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; visual mesh filename=package://abb_irb4400_support/meshes/irb4400l30/visual/link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
- link link_2: geometry collision mesh filename=package://abb_irb4400_support/meshes/irb4400l30/collision/l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; visual mesh filename=package://abb_irb4400_support/meshes/irb4400l30/visual/link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
- link link_3: geometry collision mesh filename=package://abb_irb4400_support/meshes/irb4400l30/collision/l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; visual mesh filename=package://abb_irb4400_support/meshes/irb4400l30/visual/link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
- link link_4: geometry collision mesh filename=package://abb_irb4400_support/meshes/irb4400l30/collision/l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; visual mesh filename=package://abb_irb4400_support/meshes/irb4400l30/visual/link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
- link link_5: geometry collision mesh filename=package://abb_irb4400_support/meshes/irb4400l30/collision/l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; visual mesh filename=package://abb_irb4400_support/meshes/irb4400l30/visual/link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
- link link_6: geometry collision mesh filename=package://abb_irb4400_support/meshes/irb4400l30/collision/l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; visual mesh filename=package://abb_irb4400_support/meshes/irb4400l30/visual/link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

File: abb_irb4400_support/urdf/irb4400l30.xacro (robot description, xacro)
@@ -1,5 +1,5 @@
 <?xml version="1.0" ?>
-<robot name="irb_4400_l30" xmlns:xacro="http://ros.org/wiki/xacro">
-	<include filename="$(find abb_common)/urdf/irb_4400_l30.macro.xacro"/>
-	<xacro:irb_4400_l30 prefix=""/>
+<robot name="abb_irb4400l30" xmlns:xacro="http://ros.org/wiki/xacro">
+	<include filename="$(find abb_irb4400_support)/urdf/irb4400l30_macro.xacro"/>
+	<xacro:irb4400l30 prefix=""/>
 </robot>

File: abb_irb4400_support/urdf/irb4400l30_macro.xacro (robot description, xacro)
@@ -1,5 +1,5 @@
 <?xml version="1.0" ?>
 <robot xmlns:xacro="http://ros.org/wiki/xacro">
-	<xacro:macro name="irb_4400_l30" params="prefix">
+	<xacro:macro name="irb4400l30" params="prefix">
 		<!-- link list -->
 		<link name="${prefix}base_link">
@@ -10,5 +10,5 @@
       			<geometry>
         			<mesh
-          			filename="package://abb_common/meshes/irb_4400_l30/visual/base_link.STL" />
+          			filename="package://abb_irb4400_support/meshes/irb4400l30/visual/base_link.STL" />
       			</geometry>
       			<material
@@ -20,5 +20,5 @@
  			<collision>
 				<geometry>
-					<mesh filename="package://abb_common/meshes/irb_4400_l30/collision/base_link.STL" />
+					<mesh filename="package://abb_irb4400_support/meshes/irb4400l30/collision/base_link.STL" />
 				</geometry>
 				<material name="yellow">
@@ -34,5 +34,5 @@
       			<geometry>
         			<mesh
-          			filename="package://abb_common/meshes/irb_4400_l30/visual/link_1.STL" />
+          			filename="package://abb_irb4400_support/meshes/irb4400l30/visual/link_1.STL" />
       			</geometry>
       			<material name="abb_orange"/>
@@ -43,5 +43,5 @@
         			rpy="0 0 0" />
 				<geometry>
-					<mesh filename="package://abb_common/meshes/irb_4400_l30/collision/link_1.STL" />
+					<mesh filename="package://abb_irb4400_support/meshes/irb4400l30/collision/link_1.STL" />
 				</geometry>
 				<material name="yellow"/>
@@ -55,5 +55,5 @@
       			<geometry>
         			<mesh
-          			filename="package://abb_common/meshes/irb_4400_l30/visual/link_2.STL" />
+          			filename="package://abb_irb4400_support/meshes/irb4400l30/visual/link_2.STL" />
       			</geometry>
       			<material name="abb_orange"/>
@@ -64,5 +64,5 @@
         			rpy="0 0 0" />
 				<geometry>
-					<mesh filename="package://abb_common/meshes/irb_4400_l30/collision/link_2.STL" />
+					<mesh filename="package://abb_irb4400_support/meshes/irb4400l30/collision/link_2.STL" />
 				</geometry>
 				<material name="yellow"/>
@@ -76,5 +76,5 @@
 			  	<geometry>
 					<mesh
-				  	filename="package://abb_common/meshes/irb_4400_l30/visual/link_3.STL" />
+				  	filename="package://abb_irb4400_support/meshes/irb4400l30/visual/link_3.STL" />
 			  	</geometry>
 			  	<material name="abb_orange"/>
@@ -85,5 +85,5 @@
         			rpy="0 0 0" />
 				<geometry>
-					<mesh filename="package://abb_common/meshes/irb_4400_l30/collision/link_3.STL" />
+					<mesh filename="package://abb_irb4400_support/meshes/irb4400l30/collision/link_3.STL" />
 				</geometry>
 				<material name="yellow"/>
@@ -97,5 +97,5 @@
 				  <geometry>
 					<mesh
-					  filename="package://abb_common/meshes/irb_4400_l30/visual/link_4.STL" />
+					  filename="package://abb_irb4400_support/meshes/irb4400l30/visual/link_4.STL" />
 				  </geometry>
 				  <material name="abb_orange"/>
@@ -106,5 +106,5 @@
         			rpy="0 0 0" />
 				<geometry>
-					<mesh filename="package://abb_common/meshes/irb_4400_l30/collision/link_4.STL" />
+					<mesh filename="package://abb_irb4400_support/meshes/irb4400l30/collision/link_4.STL" />
 				</geometry>
 				<material name="yellow"/>
@@ -118,5 +118,5 @@
 				<geometry>
 					<mesh
-					  filename="package://abb_common/meshes/irb_4400_l30/visual/link_5.STL" />
+					  filename="package://abb_irb4400_support/meshes/irb4400l30/visual/link_5.STL" />
 				</geometry>
 				<material name="abb_orange"/>
@@ -127,5 +127,5 @@
         			rpy="0 0 0" />
 				<geometry>
-					<mesh filename="package://abb_common/meshes/irb_4400_l30/collision/link_5.STL" />
+					<mesh filename="package://abb_irb4400_support/meshes/irb4400l30/collision/link_5.STL" />
 				</geometry>
 				<material name="yellow"/>
@@ -139,5 +139,5 @@
 				<geometry>
 					<mesh
-					  filename="package://abb_common/meshes/irb_4400_l30/visual/link_6.STL" />
+					  filename="package://abb_irb4400_support/meshes/irb4400l30/visual/link_6.STL" />
 				</geometry>
 				<material name="abb_orange"/>
@@ -148,5 +148,5 @@
         			rpy="0 0 0" />
 				<geometry>
-					<mesh filename="package://abb_common/meshes/irb_4400_l30/collision/link_6.STL" />
+					<mesh filename="package://abb_irb4400_support/meshes/irb4400l30/collision/link_6.STL" />
 				</geometry>
 				<material name="yellow"/>
