Commit message: Prefix xacro macro with mfg name. Fix #2.

File: abb_irb4400_support/urdf/irb4400l30.xacro (robot description, xacro)
@@ -2,4 +2,4 @@
 <robot name="abb_irb4400l30" xmlns:xacro="http://ros.org/wiki/xacro">
 	<include filename="$(find abb_irb4400_support)/urdf/irb4400l30_macro.xacro"/>
-	<xacro:irb4400l30 prefix=""/>
+	<xacro:abb_irb4400l30 prefix=""/>
 </robot>

File: abb_irb4400_support/urdf/irb4400l30_macro.xacro (robot description, xacro)
@@ -1,5 +1,5 @@
 <?xml version="1.0" ?>
 <robot xmlns:xacro="http://ros.org/wiki/xacro">
-	<xacro:macro name="irb4400l30" params="prefix">
+	<xacro:macro name="abb_irb4400l30" params="prefix">
 		<!-- link list -->
 		<link name="${prefix}base_link">
