Commit message: Change irb4400l30 mesh extensions to lowercase. Fix #3.
The ROS Industrial repository style guide (wiki) prefers lowercase filenames and extensions.

File: abb_irb4400_support/urdf/irb4400l30_macro.xacro (robot description, xacro)
@@ -10,5 +10,5 @@
       			<geometry>
         			<mesh
-          			filename="package://abb_irb4400_support/meshes/irb4400l30/visual/base_link.STL" />
+          			filename="package://abb_irb4400_support/meshes/irb4400l30/visual/base_link.stl" />
       			</geometry>
       			<material
@@ -20,5 +20,5 @@
  			<collision>
 				<geometry>
-					<mesh filename="package://abb_irb4400_support/meshes/irb4400l30/collision/base_link.STL" />
+					<mesh filename="package://abb_irb4400_support/meshes/irb4400l30/collision/base_link.stl" />
 				</geometry>
 				<material name="yellow">
@@ -34,5 +34,5 @@
       			<geometry>
         			<mesh
-          			filename="package://abb_irb4400_support/meshes/irb4400l30/visual/link_1.STL" />
+          			filename="package://abb_irb4400_support/meshes/irb4400l30/visual/link_1.stl" />
       			</geometry>
       			<material name="abb_orange"/>
@@ -43,5 +43,5 @@
         			rpy="0 0 0" />
 				<geometry>
-					<mesh filename="package://abb_irb4400_support/meshes/irb4400l30/collision/link_1.STL" />
+					<mesh filename="package://abb_irb4400_support/meshes/irb4400l30/collision/link_1.stl" />
 				</geometry>
 				<material name="yellow"/>
@@ -55,5 +55,5 @@
       			<geometry>
         			<mesh
-          			filename="package://abb_irb4400_support/meshes/irb4400l30/visual/link_2.STL" />
+          			filename="package://abb_irb4400_support/meshes/irb4400l30/visual/link_2.stl" />
       			</geometry>
       			<material name="abb_orange"/>
@@ -64,5 +64,5 @@
         			rpy="0 0 0" />
 				<geometry>
-					<mesh filename="package://abb_irb4400_support/meshes/irb4400l30/collision/link_2.STL" />
+					<mesh filename="package://abb_irb4400_support/meshes/irb4400l30/collision/link_2.stl" />
 				</geometry>
 				<material name="yellow"/>
@@ -76,5 +76,5 @@
 			  	<geometry>
 					<mesh
-				  	filename="package://abb_irb4400_support/meshes/irb4400l30/visual/link_3.STL" />
+				  	filename="package://abb_irb4400_support/meshes/irb4400l30/visual/link_3.stl" />
 			  	</geometry>
 			  	<material name="abb_orange"/>
@@ -85,5 +85,5 @@
         			rpy="0 0 0" />
 				<geometry>
-					<mesh filename="package://abb_irb4400_support/meshes/irb4400l30/collision/link_3.STL" />
+					<mesh filename="package://abb_irb4400_support/meshes/irb4400l30/collision/link_3.stl" />
 				</geometry>
 				<material name="yellow"/>
@@ -97,5 +97,5 @@
 				  <geometry>
 					<mesh
-					  filename="package://abb_irb4400_support/meshes/irb4400l30/visual/link_4.STL" />
+					  filename="package://abb_irb4400_support/meshes/irb4400l30/visual/link_4.stl" />
 				  </geometry>
 				  <material name="abb_orange"/>
@@ -106,5 +106,5 @@
         			rpy="0 0 0" />
 				<geometry>
-					<mesh filename="package://abb_irb4400_support/meshes/irb4400l30/collision/link_4.STL" />
+					<mesh filename="package://abb_irb4400_support/meshes/irb4400l30/collision/link_4.stl" />
 				</geometry>
 				<material name="yellow"/>
@@ -118,5 +118,5 @@
 				<geometry>
 					<mesh
-					  filename="package://abb_irb4400_support/meshes/irb4400l30/visual/link_5.STL" />
+					  filename="package://abb_irb4400_support/meshes/irb4400l30/visual/link_5.stl" />
 				</geometry>
 				<material name="abb_orange"/>
@@ -127,5 +127,5 @@
         			rpy="0 0 0" />
 				<geometry>
-					<mesh filename="package://abb_irb4400_support/meshes/irb4400l30/collision/link_5.STL" />
+					<mesh filename="package://abb_irb4400_support/meshes/irb4400l30/collision/link_5.stl" />
 				</geometry>
 				<material name="yellow"/>
@@ -139,5 +139,5 @@
 				<geometry>
 					<mesh
-					  filename="package://abb_irb4400_support/meshes/irb4400l30/visual/link_6.STL" />
+					  filename="package://abb_irb4400_support/meshes/irb4400l30/visual/link_6.stl" />
 				</geometry>
 				<material name="abb_orange"/>
@@ -148,5 +148,5 @@
         			rpy="0 0 0" />
 				<geometry>
-					<mesh filename="package://abb_irb4400_support/meshes/irb4400l30/collision/link_6.STL" />
+					<mesh filename="package://abb_irb4400_support/meshes/irb4400l30/collision/link_6.stl" />
 				</geometry>
 				<material name="yellow"/>
