Commit message: Updated abb_irb4400_support package: Corrected joint limits, translated joint_4 and joint_6-tool0, updated meshes, reformatted.

File: abb_irb4400_support/urdf/irb4400l_30.urdf (robot description, URDF)
Before this commit: robot abb_irb4400l30, 8 links, 7 joints
Links:
- added link base
- link base_link: geometry collision mesh filename=package://abb_irb4400_support/meshes/irb4400l_30/collision/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; visual mesh filename=package://abb_irb4400_support/meshes/irb4400l_30/visual/bas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
- link link_1: geometry collision mesh filename=package://abb_irb4400_support/meshes/irb4400l_30/collision/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; visual mesh filename=package://abb_irb4400_support/meshes/irb4400l_30/visual/lin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
- link link_2: geometry collision mesh filename=package://abb_irb4400_support/meshes/irb4400l_30/collision/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; visual mesh filename=package://abb_irb4400_support/meshes/irb4400l_30/visual/lin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
- link link_3: geometry collision mesh filename=package://abb_irb4400_support/meshes/irb4400l_30/collision/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; visual mesh filename=package://abb_irb4400_support/meshes/irb4400l_30/visual/lin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
- link link_4: geometry collision mesh filename=package://abb_irb4400_support/meshes/irb4400l_30/collision/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; visual mesh filename=package://abb_irb4400_support/meshes/irb4400l_30/visual/lin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
- link link_5: geometry collision mesh filename=package://abb_irb4400_support/meshes/irb4400l_30/collision/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; visual mesh filename=package://abb_irb4400_support/meshes/irb4400l_30/visual/lin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
- link link_6: geometry collision mesh filename=package://abb_irb4400_support/meshes/irb4400l_30/collision/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; visual mesh filename=package://abb_irb4400_support/meshes/irb4400l_30/visual/lin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
Joints:
- added joint base_link-base: type fixed, parent base_link, child base, origin xyz=0 0 0 rpy=0 0 0
- joint joint_1: limit lower=-2.87 upper=2.87 effort=0 velocity=1.00 -> lower=-2.87979 upper=2.87979 effort=0 velocity=2.618
- joint joint_2: limit lower=-1.7453 upper=1.9199 effort=0 velocity=1.00 -> lower=-1.2217 upper=1.658 effort=0 velocity=2.0944
- joint joint_3: limit lower=-1.0472 upper=1.1345 effort=0 velocity=2.618 -> lower=-1.0472 upper=1.1345 effort=0 velocity=2.0944
- joint joint_4: limit lower=-3.49 upper=3.49 effort=0 velocity=3.14 -> lower=-3.49 upper=3.49 effort=0 velocity=3.927; origin xyz=1.3809 0 0.15 rpy=0 0 0 -> xyz=1.38 0 0.15 rpy=0 0 0
- joint joint_5: limit lower=-2.094 upper=2.094 effort=0 velocity=3.14 -> lower=-2.0944 upper=2.0944 effort=0 velocity=4.3633
- joint joint_6: limit lower=-6.98 upper=6.98 effort=0 velocity=3.14 -> lower=-6.9813 upper=6.9813 effort=0 velocity=5.7596
- joint joint_6-tool0: origin xyz=0.1391 0 0 rpy=0 0 0 -> xyz=0.14 0 0 rpy=0 0 0
