Commit message: Find and replace every instance of 'irb4400l_30' with 'irb4400l_243_30' to comply with new naming conventions.

File: abb_irb4400_support/urdf/irb4400l_243_30.urdf (robot description, URDF)
Before this commit: robot abb_irb4400l_30, 9 links, 8 joints
Links:
- link base_link: geometry collision mesh filename=package://abb_irb4400_support/meshes/irb4400l_243_30/collis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; visual mesh filename=package://abb_irb4400_support/meshes/irb4400l_243_30/visual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
- link link_1: geometry collision mesh filename=package://abb_irb4400_support/meshes/irb4400l_243_30/collis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; visual mesh filename=package://abb_irb4400_support/meshes/irb4400l_243_30/visual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
- link link_2: geometry collision mesh filename=package://abb_irb4400_support/meshes/irb4400l_243_30/collis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; visual mesh filename=package://abb_irb4400_support/meshes/irb4400l_243_30/visual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
- link link_3: geometry collision mesh filename=package://abb_irb4400_support/meshes/irb4400l_243_30/collis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; visual mesh filename=package://abb_irb4400_support/meshes/irb4400l_243_30/visual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
- link link_4: geometry collision mesh filename=package://abb_irb4400_support/meshes/irb4400l_243_30/collis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; visual mesh filename=package://abb_irb4400_support/meshes/irb4400l_243_30/visual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
- link link_5: geometry collision mesh filename=package://abb_irb4400_support/meshes/irb4400l_243_30/collis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; visual mesh filename=package://abb_irb4400_support/meshes/irb4400l_243_30/visual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
- link link_6: geometry collision mesh filename=package://abb_irb4400_support/meshes/irb4400l_243_30/collis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; visual mesh filename=package://abb_irb4400_support/meshes/irb4400l_243_30/visual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

File: abb_irb4400_support/urdf/irb4400l_243_30_macro.xacro (robot description, xacro)
@@ -2,5 +2,5 @@
 <robot xmlns:xacro="http://ros.org/wiki/xacro">
   <xacro:include filename="$(find abb_resources)/urdf/common_materials.xacro"/>
-  <xacro:macro name="abb_irb4400l_30" params="prefix">
+  <xacro:macro name="abb_irb4400l_243_30" params="prefix">
     <!-- link list -->
     <link name="${prefix}base_link">
@@ -8,5 +8,5 @@
         <origin xyz="0 0 0" rpy="0 0 0"/>
         <geometry>
-          <mesh filename="package://abb_irb4400_support/meshes/irb4400l_30/visual/base_link.stl"/>
+          <mesh filename="package://abb_irb4400_support/meshes/irb4400l_243_30/visual/base_link.stl"/>
         </geometry>
         <xacro:material_abb_orange />
@@ -14,5 +14,5 @@
       <collision>
         <geometry>
-          <mesh filename="package://abb_irb4400_support/meshes/irb4400l_30/collision/base_link.stl"/>
+          <mesh filename="package://abb_irb4400_support/meshes/irb4400l_243_30/collision/base_link.stl"/>
         </geometry>
         <xacro:material_abb_yellow />
@@ -23,5 +23,5 @@
         <origin xyz="0 0 0" rpy="0 0 0"/>
         <geometry>
-          <mesh filename="package://abb_irb4400_support/meshes/irb4400l_30/visual/link_1.stl"/>
+          <mesh filename="package://abb_irb4400_support/meshes/irb4400l_243_30/visual/link_1.stl"/>
         </geometry>
         <xacro:material_abb_orange />
@@ -30,5 +30,5 @@
         <origin xyz="0 0 0" rpy="0 0 0"/>
         <geometry>
-          <mesh filename="package://abb_irb4400_support/meshes/irb4400l_30/collision/link_1.stl"/>
+          <mesh filename="package://abb_irb4400_support/meshes/irb4400l_243_30/collision/link_1.stl"/>
         </geometry>
         <xacro:material_abb_yellow />
@@ -39,5 +39,5 @@
         <origin xyz="0 0 0" rpy="0 0 0"/>
         <geometry>
-          <mesh filename="package://abb_irb4400_support/meshes/irb4400l_30/visual/link_2.stl"/>
+          <mesh filename="package://abb_irb4400_support/meshes/irb4400l_243_30/visual/link_2.stl"/>
         </geometry>
         <xacro:material_abb_orange />
@@ -46,5 +46,5 @@
         <origin xyz="0 0 0" rpy="0 0 0"/>
         <geometry>
-          <mesh filename="package://abb_irb4400_support/meshes/irb4400l_30/collision/link_2.stl"/>
+          <mesh filename="package://abb_irb4400_support/meshes/irb4400l_243_30/collision/link_2.stl"/>
         </geometry>
         <xacro:material_abb_yellow />
@@ -55,5 +55,5 @@
         <origin xyz="0 0 0" rpy="0 0 0"/>
         <geometry>
-          <mesh filename="package://abb_irb4400_support/meshes/irb4400l_30/visual/link_3.stl"/>
+          <mesh filename="package://abb_irb4400_support/meshes/irb4400l_243_30/visual/link_3.stl"/>
         </geometry>
         <xacro:material_abb_orange />
@@ -62,5 +62,5 @@
         <origin xyz="0 0 0" rpy="0 0 0"/>
         <geometry>
-          <mesh filename="package://abb_irb4400_support/meshes/irb4400l_30/collision/link_3.stl"/>
+          <mesh filename="package://abb_irb4400_support/meshes/irb4400l_243_30/collision/link_3.stl"/>
         </geometry>
         <xacro:material_abb_yellow />
@@ -71,5 +71,5 @@
         <origin xyz="0 0 0" rpy="0 0 0"/>
         <geometry>
-          <mesh filename="package://abb_irb4400_support/meshes/irb4400l_30/visual/link_4.stl"/>
+          <mesh filename="package://abb_irb4400_support/meshes/irb4400l_243_30/visual/link_4.stl"/>
         </geometry>
         <xacro:material_abb_orange />
@@ -78,5 +78,5 @@
         <origin xyz="0 0 0" rpy="0 0 0"/>
         <geometry>
-          <mesh filename="package://abb_irb4400_support/meshes/irb4400l_30/collision/link_4.stl"/>
+          <mesh filename="package://abb_irb4400_support/meshes/irb4400l_243_30/collision/link_4.stl"/>
         </geometry>
         <xacro:material_abb_yellow />
@@ -87,5 +87,5 @@
         <origin xyz="0 0 0" rpy="0 0 0"/>
         <geometry>
-          <mesh filename="package://abb_irb4400_support/meshes/irb4400l_30/visual/link_5.stl"/>
+          <mesh filename="package://abb_irb4400_support/meshes/irb4400l_243_30/visual/link_5.stl"/>
         </geometry>
         <xacro:material_abb_orange />
@@ -94,5 +94,5 @@
         <origin xyz="0 0 0" rpy="0 0 0"/>
         <geometry>
-          <mesh filename="package://abb_irb4400_support/meshes/irb4400l_30/collision/link_5.stl"/>
+          <mesh filename="package://abb_irb4400_support/meshes/irb4400l_243_30/collision/link_5.stl"/>
         </geometry>
         <xacro:material_abb_yellow />
@@ -103,5 +103,5 @@
         <origin xyz="0 0 0" rpy="0 0 0"/>
         <geometry>
-          <mesh filename="package://abb_irb4400_support/meshes/irb4400l_30/visual/link_6.stl"/>
+          <mesh filename="package://abb_irb4400_support/meshes/irb4400l_243_30/visual/link_6.stl"/>
         </geometry>
         <xacro:material_abb_black />
@@ -110,5 +110,5 @@
         <origin xyz="0 0 0" rpy="0 0 0"/>
         <geometry>
-          <mesh filename="package://abb_irb4400_support/meshes/irb4400l_30/collision/link_6.stl"/>
+          <mesh filename="package://abb_irb4400_support/meshes/irb4400l_243_30/collision/link_6.stl"/>
         </geometry>
         <xacro:material_abb_yellow />
