Commit message: removed dynamic and calibration elements from xacros, and modified package.xml files

File: abb_irb120_support/urdf/irb120_macro.xacro (robot description, xacro)
@@ -129,6 +129,4 @@
     <limit effort="0" lower="-2.87979" upper="2.87979" velocity="4.36332"/>
     <axis xyz="0 0 1"/>
-    <calibration rising="0" falling="0"/>
-    <dynamics damping="0" friction="0"/>
   </joint>
   <joint name="${prefix}joint_2" type="revolute">
@@ -138,6 +136,4 @@
     <limit effort="0" lower="-1.91986" upper="1.91986" velocity="4.36332"/>
     <axis xyz="0 1 0"/>
-    <calibration rising="0" falling="0"/>
-    <dynamics damping="0" friction="0"/>
   </joint>
   <joint name="${prefix}joint_3" type="revolute">
@@ -147,6 +143,4 @@
     <limit effort="0" lower="-1.91986" upper="1.22173" velocity="4.36332"/>
     <axis xyz="0 1 0"/>
-    <calibration rising="0" falling="0"/>
-    <dynamics damping="0" friction="0"/>
   </joint>
   <joint name="${prefix}joint_4" type="revolute">
@@ -156,6 +150,4 @@
     <limit effort="0" lower="-2.79253" upper="2.79253" velocity="5.58505"/>
     <axis xyz="1 0 0"/>
-    <calibration rising="0" falling="0"/>
-    <dynamics damping="0" friction="0"/>
   </joint>
   <joint name="${prefix}joint_5" type="revolute">
@@ -165,6 +157,4 @@
     <limit effort="0" lower="-2.094395" upper="2.094395" velocity="5.58505"/>
     <axis xyz="0 1 0"/>
-    <calibration rising="0" falling="0"/>
-    <dynamics damping="0" friction="0"/>
   </joint>
   <joint name="${prefix}joint_6" type="revolute">
@@ -174,6 +164,4 @@
     <limit effort="0" lower="-6.98132" upper="6.98132" velocity="7.33038"/>
     <axis xyz="1 0 0"/>
-    <calibration rising="0" falling="0"/>
-    <dynamics damping="0" friction="0"/>
   </joint>
   <joint name="${prefix}joint6-tool0" type="fixed">

File: abb_irb120_support/urdf/irb120t_macro.xacro (robot description, xacro)
@@ -129,6 +129,4 @@
     <limit effort="0" lower="-2.87979" upper="2.87979" velocity="4.36332"/>
     <axis xyz="0 0 1"/>
-    <calibration rising="0" falling="0"/>
-    <dynamics damping="0" friction="0"/>
   </joint>
   <joint name="${prefix}joint_2" type="revolute">
@@ -138,6 +136,4 @@
     <limit effort="0" lower="-1.91986" upper="1.91986" velocity="4.36332"/>
     <axis xyz="0 1 0"/>
-    <calibration rising="0" falling="0"/>
-    <dynamics damping="0" friction="0"/>
   </joint>
   <joint name="${prefix}joint_3" type="revolute">
@@ -147,6 +143,4 @@
     <limit effort="0" lower="-1.91986" upper="1.22173" velocity="4.36332"/>
     <axis xyz="0 1 0"/>
-    <calibration rising="0" falling="0"/>
-    <dynamics damping="0" friction="0"/>
   </joint>
   <joint name="${prefix}joint_4" type="revolute">
@@ -156,6 +150,4 @@
     <limit effort="0" lower="-2.79253" upper="2.79253" velocity="7.33038"/>
     <axis xyz="1 0 0"/>
-    <calibration rising="0" falling="0"/>
-    <dynamics damping="0" friction="0"/>
   </joint>
   <joint name="${prefix}joint_5" type="revolute">
@@ -165,6 +157,4 @@
     <limit effort="0" lower="-2.094395" upper="2.094395" velocity="10.29744"/>
     <axis xyz="0 1 0"/>
-    <calibration rising="0" falling="0"/>
-    <dynamics damping="0" friction="0"/>
   </joint>
   <joint name="${prefix}joint_6" type="revolute">
@@ -174,6 +164,4 @@
     <limit effort="0" lower="-6.98132" upper="6.98132" velocity="10.471975"/>
     <axis xyz="1 0 0"/>
-    <calibration rising="0" falling="0"/>
-    <dynamics damping="0" friction="0"/>
   </joint>
   <joint name="${prefix}joint6-tool0" type="fixed">
