Commit message: Add abb_resource materials to urdf/macro

File: abb_irb4400_support/urdf/irb4400l_30_macro.xacro (robot description, xacro)
@@ -1,179 +1,176 @@
 <?xml version="1.0"?>
 <robot xmlns:xacro="http://ros.org/wiki/xacro">
-<xacro:macro name="abb_irb4400l_30" params="prefix">
-  <!-- link list -->
-  <link name="${prefix}base_link">
-    <visual>
+  <xacro:include filename="$(find abb_resources)/urdf/common_materials.xacro"/>
+  <xacro:macro name="abb_irb4400l_30" params="prefix">
+    <!-- link list -->
+    <link name="${prefix}base_link">
+      <visual>
+        <origin xyz="0 0 0" rpy="0 0 0"/>
+        <geometry>
+          <mesh filename="package://abb_irb4400_support/meshes/irb4400l_30/visual/base_link.stl"/>
+        </geometry>
+        <xacro:material_abb_orange />
+      </visual>
+      <collision>
+        <geometry>
+          <mesh filename="package://abb_irb4400_support/meshes/irb4400l_30/collision/base_link.stl"/>
+        </geometry>
+        <xacro:material_abb_yellow />
+      </collision>
+    </link>
+    <link name="${prefix}link_1">
+      <visual>
+        <origin xyz="0 0 0" rpy="0 0 0"/>
+        <geometry>
+          <mesh filename="package://abb_irb4400_support/meshes/irb4400l_30/visual/link_1.stl"/>
+        </geometry>
+        <xacro:material_abb_orange />
+      </visual>
+      <collision>
+        <origin xyz="0 0 0" rpy="0 0 0"/>
+        <geometry>
+          <mesh filename="package://abb_irb4400_support/meshes/irb4400l_30/collision/link_1.stl"/>
+        </geometry>
+        <xacro:material_abb_yellow />
+      </collision>
+    </link>
+    <link name="${prefix}link_2">
+      <visual>
+        <origin xyz="0 0 0" rpy="0 0 0"/>
+        <geometry>
+          <mesh filename="package://abb_irb4400_support/meshes/irb4400l_30/visual/link_2.stl"/>
+        </geometry>
+        <xacro:material_abb_orange />
+      </visual>
+      <collision>
+        <origin xyz="0 0 0" rpy="0 0 0"/>
+        <geometry>
+          <mesh filename="package://abb_irb4400_support/meshes/irb4400l_30/collision/link_2.stl"/>
+        </geometry>
+        <xacro:material_abb_yellow />
+      </collision>
+    </link>
+    <link name="${prefix}link_3">
+      <visual>
+        <origin xyz="0 0 0" rpy="0 0 0"/>
+        <geometry>
+          <mesh filename="package://abb_irb4400_support/meshes/irb4400l_30/visual/link_3.stl"/>
+        </geometry>
+        <xacro:material_abb_orange />
+      </visual>
+      <collision>
+        <origin xyz="0 0 0" rpy="0 0 0"/>
+        <geometry>
+          <mesh filename="package://abb_irb4400_support/meshes/irb4400l_30/collision/link_3.stl"/>
+        </geometry>
+        <xacro:material_abb_yellow />
+      </collision>
+    </link>
+    <link name="${prefix}link_4">
+      <visual>
+        <origin xyz="0 0 0" rpy="0 0 0"/>
+        <geometry>
+          <mesh filename="package://abb_irb4400_support/meshes/irb4400l_30/visual/link_4.stl"/>
+        </geometry>
+        <xacro:material_abb_orange />
+      </visual>
+      <collision>
+        <origin xyz="0 0 0" rpy="0 0 0"/>
+        <geometry>
+          <mesh filename="package://abb_irb4400_support/meshes/irb4400l_30/collision/link_4.stl"/>
+        </geometry>
+        <xacro:material_abb_yellow />
+      </collision>
+    </link>
+    <link name="${prefix}link_5">
+      <visual>
+        <origin xyz="0 0 0" rpy="0 0 0"/>
+        <geometry>
+          <mesh filename="package://abb_irb4400_support/meshes/irb4400l_30/visual/link_5.stl"/>
+        </geometry>
+        <xacro:material_abb_orange />
+      </visual>
+      <collision>
+        <origin xyz="0 0 0" rpy="0 0 0"/>
+        <geometry>
+          <mesh filename="package://abb_irb4400_support/meshes/irb4400l_30/collision/link_5.stl"/>
+        </geometry>
+        <xacro:material_abb_yellow />
+      </collision>
+    </link>
+    <link name="${prefix}link_6">
+      <visual>
+        <origin xyz="0 0 0" rpy="0 0 0"/>
+        <geometry>
+          <mesh filename="package://abb_irb4400_support/meshes/irb4400l_30/visual/link_6.stl"/>
+        </geometry>
+        <xacro:material_abb_black />
+      </visual>
+      <collision>
+        <origin xyz="0 0 0" rpy="0 0 0"/>
+        <geometry>
+          <mesh filename="package://abb_irb4400_support/meshes/irb4400l_30/collision/link_6.stl"/>
+        </geometry>
+        <xacro:material_abb_yellow />
+      </collision>
+    </link>
+    <link name="${prefix}tool0"/>
+    <!-- end of link list -->
+    <!-- joint list -->
+    <joint name="${prefix}joint_1" type="revolute">
       <origin xyz="0 0 0" rpy="0 0 0"/>
-      <geometry>
-        <mesh filename="package://abb_irb4400_support/meshes/irb4400l_30/visual/base_link.stl"/>
-      </geometry>
-      <material name="abb_orange">
-        <color rgba="1 0.43 0 1"/>
-      </material>
-    </visual>
-    <collision>
-      <geometry>
-        <mesh filename="package://abb_irb4400_support/meshes/irb4400l_30/collision/base_link.stl"/>
-      </geometry>
-      <material name="yellow">
-        <color rgba="1 1 0 1"/>
-      </material>
-    </collision>
-  </link>
-  <link name="${prefix}link_1">
-    <visual>
+      <parent link="${prefix}base_link"/>
+      <child link="${prefix}link_1"/>
+      <axis xyz="0 0 1"/>
+      <limit effort="0" lower="-2.87979" upper="2.87979" velocity="2.618"/>
+    </joint>
+    <joint name="${prefix}joint_2" type="revolute">
+      <origin xyz="0.2 0 0.68" rpy="0 0 0"/>
+      <parent link="${prefix}link_1"/>
+      <child link="${prefix}link_2"/>
+      <axis xyz="0 1 0"/>
+      <limit effort="0" lower="-1.2217" upper="1.658" velocity="2.0944"/>
+      </joint>
+    <joint name="${prefix}joint_3" type="revolute">
+      <origin xyz="0 0 0.89" rpy="0 0 0"/>
+      <parent link="${prefix}link_2"/>
+      <child link="${prefix}link_3"/>
+      <axis xyz="0 1 0"/>
+      <limit effort="0" lower="-1.0472" upper="1.1345" velocity="2.0944"/>
+    </joint>
+    <joint name="${prefix}joint_4" type="revolute">
+      <origin xyz="1.38 0 0.15" rpy="0 0 0"/>
+      <parent link="${prefix}link_3"/>
+      <child link="${prefix}link_4"/>
+      <axis xyz="1 0 0"/>
+      <limit effort="0" lower="-3.49" upper="3.49" velocity="3.927"/>
+    </joint>
+    <joint name="${prefix}joint_5" type="revolute">
       <origin xyz="0 0 0" rpy="0 0 0"/>
-      <geometry>
-        <mesh filename="package://abb_irb4400_support/meshes/irb4400l_30/visual/link_1.stl"/>
-      </geometry>
-      <material name="abb_orange"/>
-    </visual>
-    <collision>
+      <parent link="${prefix}link_4"/>
+      <child link="${prefix}link_5"/>
+      <axis xyz="0 1 0"/>
+      <limit effort="0" lower="-2.0944" upper="2.0944" velocity="4.3633"/>
+    </joint>
+    <joint name="${prefix}joint_6" type="revolute">
       <origin xyz="0 0 0" rpy="0 0 0"/>
-      <geometry>
-        <mesh filename="package://abb_irb4400_support/meshes/irb4400l_30/collision/link_1.stl"/>
-      </geometry>
-      <material name="yellow"/>
-    </collision>
-  </link>
-  <link name="${prefix}link_2">
-    <visual>
+      <parent link="${prefix}link_5"/>
+      <child link="${prefix}link_6"/>
+      <axis xyz="1 0 0"/>
+      <limit effort="0" lower="-6.9813" upper="6.9813" velocity="5.7596"/>
+    </joint>
+    <joint name="${prefix}joint_6-tool0" type="fixed">
+      <parent link="${prefix}link_6"/>
+      <child link="${prefix}tool0"/>
+      <origin xyz="0.14 0 0" rpy="0 0 0"/>
+    </joint>
+    <!-- end of joint list -->
+    <!-- ROS base_link to ABB World Coordinates transform -->
+    <link name="${prefix}base" />
+    <joint name="${prefix}base_link-base" type="fixed">
       <origin xyz="0 0 0" rpy="0 0 0"/>
-      <geometry>
-        <mesh filename="package://abb_irb4400_support/meshes/irb4400l_30/visual/link_2.stl"/>
-      </geometry>
-      <material name="abb_orange"/>
-    </visual>
-    <collision>
-      <origin xyz="0 0 0" rpy="0 0 0"/>
-      <geometry>
-        <mesh filename="package://abb_irb4400_support/meshes/irb4400l_30/collision/link_2.stl"/>
-      </geometry>
-      <material name="yellow"/>
-    </collision>
-  </link>
-  <link name="${prefix}link_3">
-    <visual>
-      <origin xyz="0 0 0" rpy="0 0 0"/>
-      <geometry>
-        <mesh filename="package://abb_irb4400_support/meshes/irb4400l_30/visual/link_3.stl"/>
-      </geometry>
-      <material name="abb_orange"/>
-    </visual>
-    <collision>
-      <origin xyz="0 0 0" rpy="0 0 0"/>
-      <geometry>
-        <mesh filename="package://abb_irb4400_support/meshes/irb4400l_30/collision/link_3.stl"/>
-      </geometry>
-      <material name="yellow"/>
-    </collision>
-  </link>
-  <link name="${prefix}link_4">
-    <visual>
-      <origin xyz="0 0 0" rpy="0 0 0"/>
-      <geometry>
-        <mesh filename="package://abb_irb4400_support/meshes/irb4400l_30/visual/link_4.stl"/>
-      </geometry>
-      <material name="abb_orange"/>
-    </visual>
-    <collision>
-      <origin xyz="0 0 0" rpy="0 0 0"/>
-      <geometry>
-        <mesh filename="package://abb_irb4400_support/meshes/irb4400l_30/collision/link_4.stl"/>
-      </geometry>
-      <material name="yellow"/>
-    </collision>
-  </link>
-  <link name="${prefix}link_5">
-    <visual>
-      <origin xyz="0 0 0" rpy="0 0 0"/>
-      <geometry>
-        <mesh filename="package://abb_irb4400_support/meshes/irb4400l_30/visual/link_5.stl"/>
-      </geometry>
-      <material name="abb_orange"/>
-    </visual>
-    <collision>
-      <origin xyz="0 0 0" rpy="0 0 0"/>
-      <geometry>
-        <mesh filename="package://abb_irb4400_support/meshes/irb4400l_30/collision/link_5.stl"/>
-      </geometry>
-      <material name="yellow"/>
-    </collision>
-  </link>
-  <link name="${prefix}link_6">
-    <visual>
-      <origin xyz="0 0 0" rpy="0 0 0"/>
-      <geometry>
-        <mesh filename="package://abb_irb4400_support/meshes/irb4400l_30/visual/link_6.stl"/>
-      </geometry>
-      <material name="abb_orange"/>
-    </visual>
-    <collision>
-      <origin xyz="0 0 0" rpy="0 0 0"/>
-      <geometry>
-        <mesh filename="package://abb_irb4400_support/meshes/irb4400l_30/collision/link_6.stl"/>
-      </geometry>
-      <material name="yellow"/>
-    </collision>
-  </link>
-  <link name="${prefix}tool0"/>
-  <!-- end of link list -->
-  <!-- joint list -->
-  <joint name="${prefix}joint_1" type="revolute">
-    <origin xyz="0 0 0" rpy="0 0 0"/>
-    <parent link="${prefix}base_link"/>
-    <child link="${prefix}link_1"/>
-    <axis xyz="0 0 1"/>
-    <limit effort="0" lower="-2.87979" upper="2.87979" velocity="2.618"/>
-  </joint>
-  <joint name="${prefix}joint_2" type="revolute">
-    <origin xyz="0.2 0 0.68" rpy="0 0 0"/>
-    <parent link="${prefix}link_1"/>
-    <child link="${prefix}link_2"/>
-    <axis xyz="0 1 0"/>
-    <limit effort="0" lower="-1.2217" upper="1.658" velocity="2.0944"/>
+      <parent link="${prefix}base_link"/>
+      <child link="${prefix}base"/>
     </joint>
-  <joint name="${prefix}joint_3" type="revolute">
-    <origin xyz="0 0 0.89" rpy="0 0 0"/>
-    <parent link="${prefix}link_2"/>
-    <child link="${prefix}link_3"/>
-    <axis xyz="0 1 0"/>
-    <limit effort="0" lower="-1.0472" upper="1.1345" velocity="2.0944"/>
-  </joint>
-  <joint name="${prefix}joint_4" type="revolute">
-    <origin xyz="1.38 0 0.15" rpy="0 0 0"/>
-    <parent link="${prefix}link_3"/>
-    <child link="${prefix}link_4"/>
-    <axis xyz="1 0 0"/>
-    <limit effort="0" lower="-3.49" upper="3.49" velocity="3.927"/>
-  </joint>
-  <joint name="${prefix}joint_5" type="revolute">
-    <origin xyz="0 0 0" rpy="0 0 0"/>
-    <parent link="${prefix}link_4"/>
-    <child link="${prefix}link_5"/>
-    <axis xyz="0 1 0"/>
-    <limit effort="0" lower="-2.0944" upper="2.0944" velocity="4.3633"/>
-  </joint>
-  <joint name="${prefix}joint_6" type="revolute">
-    <origin xyz="0 0 0" rpy="0 0 0"/>
-    <parent link="${prefix}link_5"/>
-    <child link="${prefix}link_6"/>
-    <axis xyz="1 0 0"/>
-    <limit effort="0" lower="-6.9813" upper="6.9813" velocity="5.7596"/>
-  </joint>
-  <joint name="${prefix}joint_6-tool0" type="fixed">
-    <parent link="${prefix}link_6"/>
-    <child link="${prefix}tool0"/>
-    <origin xyz="0.14 0 0" rpy="0 0 0"/>
-  </joint>
-  <!-- end of joint list -->
-  <!-- ROS base_link to ABB World Coordinates transform -->
-  <link name="${prefix}base" />
-  <joint name="${prefix}base_link-base" type="fixed">
-    <origin xyz="0 0 0" rpy="0 0 0"/>
-    <parent link="${prefix}base_link"/>
-    <child link="${prefix}base"/>
-  </joint>
-</xacro:macro>
+  </xacro:macro>
 </robot>

Commit message: Introduction of Gazebo simulator support for IRB 120

File: abb_irb120_support/urdf/irb120.urdf (robot description, URDF)
Before this commit: robot abb_irb120, 9 links, 8 joints
Links:
- link base_link: mass None -> 6.215
- link link_1: mass None -> 3.067
- link link_2: mass None -> 3.909
- link link_3: mass None -> 2.944
- link link_4: mass None -> 1.328
- link link_5: mass None -> 0.546
- link link_6: mass None -> 0.137

File: abb_irb120_support/urdf/irb120_macro.xacro (robot description, xacro)
@@ -5,4 +5,9 @@
     <!-- link list -->
     <link name="${prefix}base_link">
+      <inertial>
+        <mass value="6.215"/>
+        <origin xyz="-0.04204 8.01E-05 0.07964" rpy="0 0 0"/>
+        <inertia ixx="0.0247272" ixy="-8.0784E-05" ixz="0.00130902" iyy="0.0491285" iyz="-8.0419E-06" izz="0.0472376"/>
+      </inertial>
       <visual>
         <origin xyz="0 0 0" rpy="0 0 0"/>
@@ -21,4 +26,9 @@
     </link>
     <link name="${prefix}link_1">
+      <inertial>
+        <mass value="3.067" />
+        <origin xyz="9.77E-05 -0.00012 0.23841" rpy="0 0 0"/>
+        <inertia ixx="0.0142175" ixy="-1.28579E-05" ixz="-2.31364E-05" iyy="0.0144041" iyz="1.93404E-05" izz="0.0104533"/>
+      </inertial>
       <visual>
         <origin xyz="0 0 0" rpy="0 0 0"/>
@@ -37,4 +47,9 @@
     </link>
     <link name="${prefix}link_2">
+      <inertial>
+        <mass value="3.909"/>
+        <origin xyz="0.00078 -0.00212 0.10124" rpy="0 0 0"/>
+        <inertia ixx="0.0603111" ixy="9.83431E-06" ixz="5.72407E-05" iyy="0.041569" iyz="-0.00050497" izz="0.0259548"/>
+      </inertial>
       <visual>
         <origin xyz="0 0 0" rpy="0 0 0"/>
@@ -53,4 +68,9 @@
     </link>
     <link name="${prefix}link_3">
+      <inertial>
+        <mass value="2.944"/>
+        <origin xyz="0.02281 0.00106 0.05791" rpy="0 0 0"/>
+        <inertia ixx="0.00835606" ixy="-8.01545E-05" ixz="0.00142884" iyy="0.016713" iyz="-0.000182227" izz="0.0126984"/>
+      </inertial>
       <visual>
         <origin xyz="0 0 0" rpy="0 0 0"/>
@@ -69,4 +89,9 @@
     </link>
     <link name="${prefix}link_4">
+      <inertial>
+        <mass value="1.328"/>
+        <origin xyz="0.2247 0.00015 0.00041" rpy="0 0 0"/>
+        <inertia ixx="0.00284661" ixy="-2.12765E-05" ixz="-1.6435E-05" iyy="0.00401346" iyz="1.31336E-05" izz="0.0052535"/>
+      </inertial>
       <visual>
         <origin xyz="0 0 0" rpy="0 0 0"/>
@@ -85,4 +110,9 @@
     </link>
     <link name="${prefix}link_5">
+      <inertial>
+        <mass value="0.546"/>
+        <origin xyz="-0.00109 3.68E-05 6.22E-05" rpy="0 0 0"/>
+        <inertia ixx="0.000404891" ixy="1.61943E-06" ixz="8.46805E-07" iyy="0.000892825" iyz="-1.51792E-08" izz="0.000815468"/>
+      </inertial>
       <visual>
         <origin xyz="0 0 0" rpy="0 0 0"/>
@@ -101,4 +131,9 @@
     </link>
     <link name="${prefix}link_6">
+      <inertial>
+        <mass value="0.137"/>
+        <origin xyz="-0.00706 -0.00017 -1.32E-06" rpy="0 0 0"/>
+        <inertia ixx="0.001" ixy="0" ixz="0" iyy="0.001" iyz="0" izz="0.001"/>
+      </inertial>
       <visual>
         <origin xyz="0 0 0" rpy="0 0 0"/>
@@ -125,4 +160,5 @@
       <limit effort="0" lower="-2.87979" upper="2.87979" velocity="4.36332"/>
       <axis xyz="0 0 1"/>
+      <dynamics damping="0.0" friction="0.0"/>
     </joint>
     <joint name="${prefix}joint_2" type="revolute">
@@ -132,4 +168,5 @@
       <limit effort="0" lower="-1.91986" upper="1.91986" velocity="4.36332"/>
       <axis xyz="0 1 0"/>
+      <dynamics damping="0.0" friction="0.0"/>
     </joint>
     <joint name="${prefix}joint_3" type="revolute">
@@ -139,4 +176,5 @@
       <limit effort="0" lower="-1.91986" upper="1.22173" velocity="4.36332"/>
       <axis xyz="0 1 0"/>
+      <dynamics damping="0.0" friction="0.0"/>
     </joint>
     <joint name="${prefix}joint_4" type="revolute">
@@ -146,4 +184,5 @@
       <limit effort="0" lower="-2.79253" upper="2.79253" velocity="5.58505"/>
       <axis xyz="1 0 0"/>
+      <dynamics damping="0.0" friction="0.0"/>
     </joint>
     <joint name="${prefix}joint_5" type="revolute">
@@ -153,4 +192,5 @@
       <limit effort="0" lower="-2.094395" upper="2.094395" velocity="5.58505"/>
       <axis xyz="0 1 0"/>
+      <dynamics damping="0.0" friction="0.0"/>
     </joint>
     <joint name="${prefix}joint_6" type="revolute">
@@ -160,4 +200,5 @@
       <limit effort="0" lower="-6.98132" upper="6.98132" velocity="7.33038"/>
       <axis xyz="1 0 0"/>
+      <dynamics damping="0.0" friction="0.0"/>
     </joint>
     <joint name="${prefix}joint6-tool0" type="fixed">

File: abb_irb120_support/urdf/irb120t.urdf (robot description, URDF)
Before this commit: robot abb_irb120t, 9 links, 8 joints
Links:
- link base_link: mass None -> 6.215
- link link_1: mass None -> 3.067
- link link_2: mass None -> 3.909
- link link_3: mass None -> 2.944
- link link_4: mass None -> 1.328
- link link_5: mass None -> 0.546
- link link_6: mass None -> 0.137

File: abb_irb120_support/urdf/irb120t_macro.xacro (robot description, xacro)
@@ -5,4 +5,9 @@
     <!-- link list -->
     <link name="${prefix}base_link">
+    	<inertial>
+    	  <mass value="6.215"/>
+    	  <origin xyz="-0.04204 8.01E-05 0.07964" rpy="0 0 0"/>
+    	  <inertia ixx="0.0247272" ixy="-8.0784E-05" ixz="0.00130902" iyy="0.0491285" iyz="-8.0419E-06" izz="0.0472376"/>
+    	</inertial>
       <visual>
         <origin xyz="0 0 0" rpy="0 0 0"/>
@@ -21,4 +26,9 @@
     </link>
     <link name="${prefix}link_1">
+    	<inertial>
+    	  <mass value="3.067" />
+    	  <origin xyz="9.77E-05 -0.00012 0.23841" rpy="0 0 0"/>
+    	  <inertia ixx="0.0142175" ixy="-1.28579E-05" ixz="-2.31364E-05" iyy="0.0144041" iyz="1.93404E-05" izz="0.0104533"/>
+    	</inertial>
       <visual>
         <origin xyz="0 0 0" rpy="0 0 0"/>
@@ -37,4 +47,9 @@
     </link>
     <link name="${prefix}link_2">
+    	<inertial>
+    	  <mass value="3.909"/>
+    	  <origin xyz="0.00078 -0.00212 0.10124" rpy="0 0 0"/>
+    	  <inertia ixx="0.0603111" ixy="9.83431E-06" ixz="5.72407E-05" iyy="0.041569" iyz="-0.00050497" izz="0.0259548"/>
+    	</inertial>
       <visual>
         <origin xyz="0 0 0" rpy="0 0 0"/>
@@ -53,4 +68,9 @@
     </link>
     <link name="${prefix}link_3">
+    	<inertial>
+    	  <mass value="2.944"/>
+    	  <origin xyz="0.02281 0.00106 0.05791" rpy="0 0 0"/>
+    	  <inertia ixx="0.00835606" ixy="-8.01545E-05" ixz="0.00142884" iyy="0.016713" iyz="-0.000182227" izz="0.0126984"/>
+    	</inertial>
       <visual>
         <origin xyz="0 0 0" rpy="0 0 0"/>
@@ -69,4 +89,9 @@
     </link>
     <link name="${prefix}link_4">
+    	<inertial>
+    	  <mass value="1.328"/>
+    	  <origin xyz="0.2247 0.00015 0.00041" rpy="0 0 0"/>
+    	  <inertia ixx="0.00284661" ixy="-2.12765E-05" ixz="-1.6435E-05" iyy="0.00401346" iyz="1.31336E-05" izz="0.0052535"/>
+    	</inertial>
       <visual>
         <origin xyz="0 0 0" rpy="0 0 0"/>
@@ -85,4 +110,9 @@
     </link>
     <link name="${prefix}link_5">
+    	<inertial>
+    	  <mass value="0.546"/>
+    	  <origin xyz="-0.00109 3.68E-05 6.22E-05" rpy="0 0 0"/>
+    	  <inertia ixx="0.000404891" ixy="1.61943E-06" ixz="8.46805E-07" iyy="0.000892825" iyz="-1.51792E-08" izz="0.000815468"/>
+    	</inertial>
       <visual>
         <origin xyz="0 0 0" rpy="0 0 0"/>
@@ -101,4 +131,9 @@
     </link>
     <link name="${prefix}link_6">
+    	<inertial>
+    	  <mass value="0.137"/>
+    	  <origin xyz="-0.00706 -0.00017 -1.32E-06" rpy="0 0 0"/>
+    	  <inertia ixx="0.001" ixy="0" ixz="0" iyy="0.001" iyz="0" izz="0.001"/>
+    	</inertial>
       <visual>
         <origin xyz="0 0 0" rpy="0 0 0"/>
@@ -125,4 +160,5 @@
       <limit effort="0" lower="-2.87979" upper="2.87979" velocity="4.36332"/>
       <axis xyz="0 0 1"/>
+    	<dynamics damping="0.0" friction="0.0"/>
     </joint>
     <joint name="${prefix}joint_2" type="revolute">
@@ -132,4 +168,5 @@
       <limit effort="0" lower="-1.91986" upper="1.91986" velocity="4.36332"/>
       <axis xyz="0 1 0"/>
+    	<dynamics damping="0.0" friction="0.0"/>
     </joint>
     <joint name="${prefix}joint_3" type="revolute">
@@ -139,4 +176,5 @@
       <limit effort="0" lower="-1.91986" upper="1.22173" velocity="4.36332"/>
       <axis xyz="0 1 0"/>
+    	<dynamics damping="0.0" friction="0.0"/>
     </joint>
     <joint name="${prefix}joint_4" type="revolute">
@@ -146,4 +184,5 @@
       <limit effort="0" lower="-2.79253" upper="2.79253" velocity="7.33038"/>
       <axis xyz="1 0 0"/>
+    	<dynamics damping="0.0" friction="0.0"/>
     </joint>
     <joint name="${prefix}joint_5" type="revolute">
@@ -153,4 +192,5 @@
       <limit effort="0" lower="-2.094395" upper="2.094395" velocity="10.29744"/>
       <axis xyz="0 1 0"/>
+    	<dynamics damping="0.0" friction="0.0"/>
     </joint>
     <joint name="${prefix}joint_6" type="revolute">
@@ -160,4 +200,5 @@
       <limit effort="0" lower="-6.98132" upper="6.98132" velocity="10.471975"/>
       <axis xyz="1 0 0"/>
+    	<dynamics damping="0.0" friction="0.0"/>
     </joint>
     <joint name="${prefix}joint6-tool0" type="fixed">
