Commit message: Revert "Merge pull request #18 from culletom/gazebo-devel"
This reverts commit e7a9e988d4f09801b47a0cf3d9e091f87442be36, reversing
changes made to 0efd1214fe3706347eade07f6433a9d3479f2974.

File: abb_irb120_support/urdf/irb120.urdf (robot description, URDF)
Before this commit: robot abb_irb120, 9 links, 8 joints
Links:
- link base_link: mass 6.215 -> None
- link link_1: mass 3.067 -> None
- link link_2: mass 3.909 -> None
- link link_3: mass 2.944 -> None
- link link_4: mass 1.328 -> None
- link link_5: mass 0.546 -> None
- link link_6: mass 0.137 -> None

File: abb_irb120_support/urdf/irb120_macro.xacro (robot description, xacro)
@@ -5,9 +5,4 @@
     <!-- link list -->
     <link name="${prefix}base_link">
-      <inertial>
-        <mass value="6.215"/>
-        <origin xyz="-0.04204 8.01E-05 0.07964" rpy="0 0 0"/>
-        <inertia ixx="0.0247272" ixy="-8.0784E-05" ixz="0.00130902" iyy="0.0491285" iyz="-8.0419E-06" izz="0.0472376"/>
-      </inertial>
       <visual>
         <origin xyz="0 0 0" rpy="0 0 0"/>
@@ -26,9 +21,4 @@
     </link>
     <link name="${prefix}link_1">
-      <inertial>
-        <mass value="3.067" />
-        <origin xyz="9.77E-05 -0.00012 0.23841" rpy="0 0 0"/>
-        <inertia ixx="0.0142175" ixy="-1.28579E-05" ixz="-2.31364E-05" iyy="0.0144041" iyz="1.93404E-05" izz="0.0104533"/>
-      </inertial>
       <visual>
         <origin xyz="0 0 0" rpy="0 0 0"/>
@@ -47,9 +37,4 @@
     </link>
     <link name="${prefix}link_2">
-      <inertial>
-        <mass value="3.909"/>
-        <origin xyz="0.00078 -0.00212 0.10124" rpy="0 0 0"/>
-        <inertia ixx="0.0603111" ixy="9.83431E-06" ixz="5.72407E-05" iyy="0.041569" iyz="-0.00050497" izz="0.0259548"/>
-      </inertial>
       <visual>
         <origin xyz="0 0 0" rpy="0 0 0"/>
@@ -68,9 +53,4 @@
     </link>
     <link name="${prefix}link_3">
-      <inertial>
-        <mass value="2.944"/>
-        <origin xyz="0.02281 0.00106 0.05791" rpy="0 0 0"/>
-        <inertia ixx="0.00835606" ixy="-8.01545E-05" ixz="0.00142884" iyy="0.016713" iyz="-0.000182227" izz="0.0126984"/>
-      </inertial>
       <visual>
         <origin xyz="0 0 0" rpy="0 0 0"/>
@@ -89,9 +69,4 @@
     </link>
     <link name="${prefix}link_4">
-      <inertial>
-        <mass value="1.328"/>
-        <origin xyz="0.2247 0.00015 0.00041" rpy="0 0 0"/>
-        <inertia ixx="0.00284661" ixy="-2.12765E-05" ixz="-1.6435E-05" iyy="0.00401346" iyz="1.31336E-05" izz="0.0052535"/>
-      </inertial>
       <visual>
         <origin xyz="0 0 0" rpy="0 0 0"/>
@@ -110,9 +85,4 @@
     </link>
     <link name="${prefix}link_5">
-      <inertial>
-        <mass value="0.546"/>
-        <origin xyz="-0.00109 3.68E-05 6.22E-05" rpy="0 0 0"/>
-        <inertia ixx="0.000404891" ixy="1.61943E-06" ixz="8.46805E-07" iyy="0.000892825" iyz="-1.51792E-08" izz="0.000815468"/>
-      </inertial>
       <visual>
         <origin xyz="0 0 0" rpy="0 0 0"/>
@@ -131,9 +101,4 @@
     </link>
     <link name="${prefix}link_6">
-      <inertial>
-        <mass value="0.137"/>
-        <origin xyz="-0.00706 -0.00017 -1.32E-06" rpy="0 0 0"/>
-        <inertia ixx="0.001" ixy="0" ixz="0" iyy="0.001" iyz="0" izz="0.001"/>
-      </inertial>
       <visual>
         <origin xyz="0 0 0" rpy="0 0 0"/>
@@ -160,5 +125,4 @@
       <limit effort="0" lower="-2.87979" upper="2.87979" velocity="4.36332"/>
       <axis xyz="0 0 1"/>
-      <dynamics damping="0.0" friction="0.0"/>
     </joint>
     <joint name="${prefix}joint_2" type="revolute">
@@ -168,5 +132,4 @@
       <limit effort="0" lower="-1.91986" upper="1.91986" velocity="4.36332"/>
       <axis xyz="0 1 0"/>
-      <dynamics damping="0.0" friction="0.0"/>
     </joint>
     <joint name="${prefix}joint_3" type="revolute">
@@ -176,5 +139,4 @@
       <limit effort="0" lower="-1.91986" upper="1.22173" velocity="4.36332"/>
       <axis xyz="0 1 0"/>
-      <dynamics damping="0.0" friction="0.0"/>
     </joint>
     <joint name="${prefix}joint_4" type="revolute">
@@ -184,5 +146,4 @@
       <limit effort="0" lower="-2.79253" upper="2.79253" velocity="5.58505"/>
       <axis xyz="1 0 0"/>
-      <dynamics damping="0.0" friction="0.0"/>
     </joint>
     <joint name="${prefix}joint_5" type="revolute">
@@ -192,5 +153,4 @@
       <limit effort="0" lower="-2.094395" upper="2.094395" velocity="5.58505"/>
       <axis xyz="0 1 0"/>
-      <dynamics damping="0.0" friction="0.0"/>
     </joint>
     <joint name="${prefix}joint_6" type="revolute">
@@ -200,5 +160,4 @@
       <limit effort="0" lower="-6.98132" upper="6.98132" velocity="7.33038"/>
       <axis xyz="1 0 0"/>
-      <dynamics damping="0.0" friction="0.0"/>
     </joint>
     <joint name="${prefix}joint6-tool0" type="fixed">

File: abb_irb120_support/urdf/irb120t.urdf (robot description, URDF)
Before this commit: robot abb_irb120t, 9 links, 8 joints
Links:
- link base_link: mass 6.215 -> None
- link link_1: mass 3.067 -> None
- link link_2: mass 3.909 -> None
- link link_3: mass 2.944 -> None
- link link_4: mass 1.328 -> None
- link link_5: mass 0.546 -> None
- link link_6: mass 0.137 -> None

File: abb_irb120_support/urdf/irb120t_macro.xacro (robot description, xacro)
@@ -5,9 +5,4 @@
     <!-- link list -->
     <link name="${prefix}base_link">
-    	<inertial>
-    	  <mass value="6.215"/>
-    	  <origin xyz="-0.04204 8.01E-05 0.07964" rpy="0 0 0"/>
-    	  <inertia ixx="0.0247272" ixy="-8.0784E-05" ixz="0.00130902" iyy="0.0491285" iyz="-8.0419E-06" izz="0.0472376"/>
-    	</inertial>
       <visual>
         <origin xyz="0 0 0" rpy="0 0 0"/>
@@ -26,9 +21,4 @@
     </link>
     <link name="${prefix}link_1">
-    	<inertial>
-    	  <mass value="3.067" />
-    	  <origin xyz="9.77E-05 -0.00012 0.23841" rpy="0 0 0"/>
-    	  <inertia ixx="0.0142175" ixy="-1.28579E-05" ixz="-2.31364E-05" iyy="0.0144041" iyz="1.93404E-05" izz="0.0104533"/>
-    	</inertial>
       <visual>
         <origin xyz="0 0 0" rpy="0 0 0"/>
@@ -47,9 +37,4 @@
     </link>
     <link name="${prefix}link_2">
-    	<inertial>
-    	  <mass value="3.909"/>
-    	  <origin xyz="0.00078 -0.00212 0.10124" rpy="0 0 0"/>
-    	  <inertia ixx="0.0603111" ixy="9.83431E-06" ixz="5.72407E-05" iyy="0.041569" iyz="-0.00050497" izz="0.0259548"/>
-    	</inertial>
       <visual>
         <origin xyz="0 0 0" rpy="0 0 0"/>
@@ -68,9 +53,4 @@
     </link>
     <link name="${prefix}link_3">
-    	<inertial>
-    	  <mass value="2.944"/>
-    	  <origin xyz="0.02281 0.00106 0.05791" rpy="0 0 0"/>
-    	  <inertia ixx="0.00835606" ixy="-8.01545E-05" ixz="0.00142884" iyy="0.016713" iyz="-0.000182227" izz="0.0126984"/>
-    	</inertial>
       <visual>
         <origin xyz="0 0 0" rpy="0 0 0"/>
@@ -89,9 +69,4 @@
     </link>
     <link name="${prefix}link_4">
-    	<inertial>
-    	  <mass value="1.328"/>
-    	  <origin xyz="0.2247 0.00015 0.00041" rpy="0 0 0"/>
-    	  <inertia ixx="0.00284661" ixy="-2.12765E-05" ixz="-1.6435E-05" iyy="0.00401346" iyz="1.31336E-05" izz="0.0052535"/>
-    	</inertial>
       <visual>
         <origin xyz="0 0 0" rpy="0 0 0"/>
@@ -110,9 +85,4 @@
     </link>
     <link name="${prefix}link_5">
-    	<inertial>
-    	  <mass value="0.546"/>
-    	  <origin xyz="-0.00109 3.68E-05 6.22E-05" rpy="0 0 0"/>
-    	  <inertia ixx="0.000404891" ixy="1.61943E-06" ixz="8.46805E-07" iyy="0.000892825" iyz="-1.51792E-08" izz="0.000815468"/>
-    	</inertial>
       <visual>
         <origin xyz="0 0 0" rpy="0 0 0"/>
@@ -131,9 +101,4 @@
     </link>
     <link name="${prefix}link_6">
-    	<inertial>
-    	  <mass value="0.137"/>
-    	  <origin xyz="-0.00706 -0.00017 -1.32E-06" rpy="0 0 0"/>
-    	  <inertia ixx="0.001" ixy="0" ixz="0" iyy="0.001" iyz="0" izz="0.001"/>
-    	</inertial>
       <visual>
         <origin xyz="0 0 0" rpy="0 0 0"/>
@@ -160,5 +125,4 @@
       <limit effort="0" lower="-2.87979" upper="2.87979" velocity="4.36332"/>
       <axis xyz="0 0 1"/>
-    	<dynamics damping="0.0" friction="0.0"/>
     </joint>
     <joint name="${prefix}joint_2" type="revolute">
@@ -168,5 +132,4 @@
       <limit effort="0" lower="-1.91986" upper="1.91986" velocity="4.36332"/>
       <axis xyz="0 1 0"/>
-    	<dynamics damping="0.0" friction="0.0"/>
     </joint>
     <joint name="${prefix}joint_3" type="revolute">
@@ -176,5 +139,4 @@
       <limit effort="0" lower="-1.91986" upper="1.22173" velocity="4.36332"/>
       <axis xyz="0 1 0"/>
-    	<dynamics damping="0.0" friction="0.0"/>
     </joint>
     <joint name="${prefix}joint_4" type="revolute">
@@ -184,5 +146,4 @@
       <limit effort="0" lower="-2.79253" upper="2.79253" velocity="7.33038"/>
       <axis xyz="1 0 0"/>
-    	<dynamics damping="0.0" friction="0.0"/>
     </joint>
     <joint name="${prefix}joint_5" type="revolute">
@@ -192,5 +153,4 @@
       <limit effort="0" lower="-2.094395" upper="2.094395" velocity="10.29744"/>
       <axis xyz="0 1 0"/>
-    	<dynamics damping="0.0" friction="0.0"/>
     </joint>
     <joint name="${prefix}joint_6" type="revolute">
@@ -200,5 +160,4 @@
       <limit effort="0" lower="-6.98132" upper="6.98132" velocity="10.471975"/>
       <axis xyz="1 0 0"/>
-    	<dynamics damping="0.0" friction="0.0"/>
     </joint>
     <joint name="${prefix}joint6-tool0" type="fixed">
