Commit message: Update the orientation for tool 0 to match the industrial robot

File: abb_irb1600_support/urdf/irb_1600_12.urdf (robot description, URDF)
Before this commit: robot irb_1600_12, 8 links, 7 joints
Joints:
- joint joint_6-tool0: origin xyz=0 0 0 rpy=0 0 0 -> xyz=0 0 0 rpy=0 1.57079 0

File: abb_irb1600_support/urdf/irb_1600_12_macro.xacro (robot description, xacro)
@@ -292,5 +292,5 @@
 			<parent link="${prefix}link_6"/>
 			<child link="${prefix}tool0"/>
-			<origin xyz="0 0 0" rpy="0 0 0"/>
+			<origin xyz="0 0 0" rpy="0 .57079 0"/>
 		</joint>
 		<!-- end of joint list -->
