Commit message: add datasheet information to package.xml seperate model specific meshes

File: abb_irb1600_support/urdf/irb1600_6_12.urdf (robot description, URDF)
Before this commit: robot irb1600_6_12, 8 links, 7 joints
Links:
- link base_link: geometry collision mesh filename=package://abb_irb1600_support/meshes/irb1600/collision/base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; visual mesh filename=package://abb_irb1600_support/meshes/irb1600/visual/base_li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
- link link_1: geometry collision mesh filename=package://abb_irb1600_support/meshes/irb1600/collision/link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; visual mesh filename=package://abb_irb1600_support/meshes/irb1600/visual/link_1.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
- link link_3: geometry collision mesh filename=package://abb_irb1600_support/meshes/irb1600/collision/link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; visual mesh filename=package://abb_irb1600_support/meshes/irb1600/visual/link_3.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
- link link_4: geometry collision mesh filename=package://abb_irb1600_support/meshes/irb1600/collision/link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; visual mesh filename=package://abb_irb1600_support/meshes/irb1600/visual/link_4.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
- link link_5: geometry collision mesh filename=package://abb_irb1600_support/meshes/irb1600/collision/link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; visual mesh filename=package://abb_irb1600_support/meshes/irb1600/visual/link_5.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
- link link_6: geometry collision mesh filename=package://abb_irb1600_support/meshes/irb1600/collision/link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; visual mesh filename=package://abb_irb1600_support/meshes/irb1600/visual/link_6.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

File: abb_irb1600_support/urdf/irb1600_6_12_macro.xacro (robot description, xacro)
@@ -7,5 +7,5 @@
       <origin xyz="0 0 0" rpy="0 0 0"/>
       <geometry>
-        <mesh filename="package://abb_irb1600_support/meshes/irb1600_6_12/visual/base_link.stl"/>
+        <mesh filename="package://abb_irb1600_support/meshes/irb1600/visual/base_link.stl"/>
       </geometry>
       <material name="abb_orange">
@@ -15,5 +15,5 @@
     <collision>
       <geometry>
-        <mesh filename="package://abb_irb1600_support/meshes/irb1600_6_12/collision/base_link.stl"/>
+        <mesh filename="package://abb_irb1600_support/meshes/irb1600/collision/base_link.stl"/>
       </geometry>
       <material name="yellow">
@@ -26,5 +26,5 @@
       <origin xyz="0 0 0" rpy="0 0 0"/>
       <geometry>
-        <mesh filename="package://abb_irb1600_support/meshes/irb1600_6_12/visual/link_1.stl"/>
+        <mesh filename="package://abb_irb1600_support/meshes/irb1600/visual/link_1.stl"/>
       </geometry>
       <material name="abb_orange"/>
@@ -33,5 +33,5 @@
       <origin xyz="0 0 0" rpy="0 0 0"/>
       <geometry>
-        <mesh filename="package://abb_irb1600_support/meshes/irb1600_6_12/collision/link_1.stl"/>
+        <mesh filename="package://abb_irb1600_support/meshes/irb1600/collision/link_1.stl"/>
       </geometry>
       <material name="yellow"/>
@@ -58,5 +58,5 @@
       <origin xyz="0 0 0" rpy="0 0 0"/>
       <geometry>
-        <mesh filename="package://abb_irb1600_support/meshes/irb1600_6_12/visual/link_3.stl"/>
+        <mesh filename="package://abb_irb1600_support/meshes/irb1600/visual/link_3.stl"/>
       </geometry>
       <material name="abb_orange"/>
@@ -65,5 +65,5 @@
       <origin xyz="0 0 0" rpy="0 0 0"/>
       <geometry>
-        <mesh filename="package://abb_irb1600_support/meshes/irb1600_6_12/collision/link_3.stl"/>
+        <mesh filename="package://abb_irb1600_support/meshes/irb1600/collision/link_3.stl"/>
       </geometry>
       <material name="yellow"/>
@@ -74,5 +74,5 @@
       <origin xyz="0 0 0" rpy="0 0 0"/>
       <geometry>
-        <mesh filename="package://abb_irb1600_support/meshes/irb1600_6_12/visual/link_4.stl"/>
+        <mesh filename="package://abb_irb1600_support/meshes/irb1600/visual/link_4.stl"/>
       </geometry>
       <material name="abb_orange"/>
@@ -81,5 +81,5 @@
       <origin xyz="0 0 0" rpy="0 0 0"/>
       <geometry>
-        <mesh filename="package://abb_irb1600_support/meshes/irb1600_6_12/collision/link_4.stl"/>
+        <mesh filename="package://abb_irb1600_support/meshes/irb1600/collision/link_4.stl"/>
       </geometry>
       <material name="yellow"/>
@@ -90,5 +90,5 @@
       <origin xyz="0 0 0" rpy="0 0 0"/>
       <geometry>
-        <mesh filename="package://abb_irb1600_support/meshes/irb1600_6_12/visual/link_5.stl"/>
+        <mesh filename="package://abb_irb1600_support/meshes/irb1600/visual/link_5.stl"/>
       </geometry>
       <material name="abb_orange"/>
@@ -97,5 +97,5 @@
       <origin xyz="0 0 0" rpy="0 0 0"/>
       <geometry>
-        <mesh filename="package://abb_irb1600_support/meshes/irb1600_6_12/collision/link_5.stl"/>
+        <mesh filename="package://abb_irb1600_support/meshes/irb1600/collision/link_5.stl"/>
       </geometry>
       <material name="yellow"/>
@@ -106,5 +106,5 @@
       <origin xyz="0 0 0" rpy="0 0 0"/>
       <geometry>
-        <mesh filename="package://abb_irb1600_support/meshes/irb1600_6_12/visual/link_6.stl"/>
+        <mesh filename="package://abb_irb1600_support/meshes/irb1600/visual/link_6.stl"/>
       </geometry>
       <material name="abb_orange"/>
@@ -113,5 +113,5 @@
       <origin xyz="0 0 0" rpy="0 0 0"/>
       <geometry>
-        <mesh filename="package://abb_irb1600_support/meshes/irb1600_6_12/collision/link_6.stl"/>
+        <mesh filename="package://abb_irb1600_support/meshes/irb1600/collision/link_6.stl"/>
       </geometry>
       <material name="yellow"/>
