Commit message: address 2nd round questions in PR #50

File: abb_irb1600_support/urdf/irb1600_6_12_macro.xacro (robot description, xacro)
@@ -126,5 +126,5 @@
     <child link="${prefix}link_1"/>
     <axis xyz="0 0 1"/>
-    <limit lower="-3.1416" upper="3.1416" effort="0" velocity="2.618"/>
+    <limit lower="-${pi}" upper="${pi}" effort="0" velocity="2.618"/>
   </joint>
   <joint name="${prefix}joint_2" type="revolute">
@@ -166,5 +166,5 @@
     <parent link="${prefix}link_6"/>
     <child link="${prefix}tool0"/>
-    <origin xyz="0 0 0" rpy="0 1.57079 0"/>
+    <origin xyz="0 0 0" rpy="0 ${pi/2 0"/>
   </joint>
   <!-- end of joint list -->

Commit message: fix typo in irb1600_6_12_macro.xacro

File: abb_irb1600_support/urdf/irb1600_6_12_macro.xacro (robot description, xacro)
@@ -166,5 +166,5 @@
     <parent link="${prefix}link_6"/>
     <child link="${prefix}tool0"/>
-    <origin xyz="0 0 0" rpy="0 ${pi/2 0"/>
+    <origin xyz="0 0 0" rpy="0 ${pi/2} 0"/>
   </joint>
   <!-- end of joint list -->

Commit message: Added flange and base frame for irb1600

File: abb_irb1600_support/urdf/irb1600_6_12_macro.xacro (robot description, xacro)
@@ -118,5 +118,4 @@
     </collision>
   </link>
-  <link name="${prefix}tool0"/>
   <!-- end of link list -->
   <!-- joint list -->
@@ -163,10 +162,26 @@
     <limit lower="-6.9813" upper="6.9813" effort="0" velocity="7.854"/>
   </joint>
-  <joint name="${prefix}joint_6-tool0" type="fixed">
+  <!-- end of joint list -->
+  <!-- ROS-Industrial 'base' frame: base_link to ABB World Coordinates transform -->
+  <link name="${prefix}base" />
+  <joint name="${prefix}base_link-base" type="fixed">
+    <origin xyz="0 0 0" rpy="0 0 0"/>
+    <parent link="${prefix}base_link"/>
+    <child link="${prefix}base"/>
+  </joint>
+  <!-- ROS-Industrial 'flange' frame: attachment point for EEF models -->
+  <link name="${prefix}flange"/>
+  <joint type="fixed" name="${prefix}joint_6-flange">
+    <origin xyz="0 0 0" rpy="0 0 0"/>
     <parent link="${prefix}link_6"/>
-    <child link="${prefix}tool0"/>
-    <origin xyz="0 0 0" rpy="0 ${pi/2} 0"/>
+    <child link="${prefix}flange"/>
   </joint>
-  <!-- end of joint list -->
+  <!-- ROS-Industrial 'tool0' frame: all-zeros tool frame -->
+  <link name="${prefix}tool0" />
+  <joint name="${prefix}link_6-tool0" type="fixed">
+    <origin xyz="0 0 0" rpy="0 ${radians(90)} 0" />
+    <parent link="${prefix}flange" />
+    <child link="${prefix}tool0" />
+  </joint>
   </xacro:macro>
 </robot>
