Commit message: Use colours from abb_resources

File: abb_irb1600_support/urdf/irb1600_8_145_macro.xacro (robot description, xacro)
@@ -2,4 +2,5 @@
 <robot xmlns:xacro="http://ros.org/wiki/xacro" name="irb1600_8_145">
   <xacro:macro name="abb_irb1600_8_145" params="prefix">
+    <xacro:include filename="$(find abb_resources)/urdf/common_materials.xacro"/>
     <!-- link list -->
     <link name="${prefix}base_link">
@@ -9,15 +10,11 @@
           <mesh filename="package://abb_irb1600_support/meshes/irb1600/visual/base_link.stl"/>
         </geometry>
-        <material name="abb_orange">
-          <color rgba="1 0.43 0 1"/>
-        </material>
-      </visual>
+        <xacro:material_abb_orange />
+    </visual>
       <collision>
         <geometry>
           <mesh filename="package://abb_irb1600_support/meshes/irb1600/collision/base_link.stl"/>
         </geometry>
-        <material name="yellow">
-          <color rgba="0 1 1 1"/>
-        </material>
+        <xacro:material_abb_yellow />
       </collision>
     </link>
@@ -28,5 +25,5 @@
           <mesh filename="package://abb_irb1600_support/meshes/irb1600/visual/link_1.stl"/>
         </geometry>
-        <material name="abb_orange"/>
+        <xacro:material_abb_orange />
       </visual>
       <collision>
@@ -35,5 +32,5 @@
           <mesh filename="package://abb_irb1600_support/meshes/irb1600/collision/link_1.stl"/>
         </geometry>
-        <material name="yellow"/>
+        <xacro:material_abb_yellow />
       </collision>
     </link>
@@ -44,5 +41,5 @@
           <mesh filename="package://abb_irb1600_support/meshes/irb1600_8_145/visual/link_2.stl"/>
         </geometry>
-        <material name="abb_orange"/>
+        <xacro:material_abb_orange />
       </visual>
       <collision>
@@ -51,5 +48,5 @@
           <mesh filename="package://abb_irb1600_support/meshes/irb1600_8_145/collision/link_2.stl"/>
         </geometry>
-        <material name="yellow"/>
+        <xacro:material_abb_yellow />
       </collision>
     </link>
@@ -60,5 +57,5 @@
           <mesh filename="package://abb_irb1600_support/meshes/irb1600/visual/link_3.stl"/>
         </geometry>
-        <material name="abb_orange"/>
+        <xacro:material_abb_orange />
       </visual>
       <collision>
@@ -67,5 +64,5 @@
           <mesh filename="package://abb_irb1600_support/meshes/irb1600/collision/link_3.stl"/>
         </geometry>
-        <material name="yellow"/>
+        <xacro:material_abb_yellow />
       </collision>
     </link>
@@ -76,5 +73,5 @@
           <mesh filename="package://abb_irb1600_support/meshes/irb1600/visual/link_4.stl"/>
         </geometry>
-        <material name="abb_orange"/>
+        <xacro:material_abb_orange />
       </visual>
       <collision>
@@ -83,5 +80,5 @@
           <mesh filename="package://abb_irb1600_support/meshes/irb1600/collision/link_4.stl"/>
         </geometry>
-        <material name="yellow"/>
+        <xacro:material_abb_yellow />
       </collision>
     </link>
@@ -92,5 +89,5 @@
           <mesh filename="package://abb_irb1600_support/meshes/irb1600/visual/link_5.stl"/>
         </geometry>
-        <material name="abb_orange"/>
+        <xacro:material_abb_orange />
       </visual>
       <collision>
@@ -99,5 +96,5 @@
           <mesh filename="package://abb_irb1600_support/meshes/irb1600/collision/link_5.stl"/>
         </geometry>
-        <material name="yellow"/>
+        <xacro:material_abb_yellow />
       </collision>
     </link>
@@ -108,5 +105,5 @@
           <mesh filename="package://abb_irb1600_support/meshes/irb1600/visual/link_6.stl"/>
         </geometry>
-        <material name="abb_orange"/>
+        <xacro:material_abb_orange />
       </visual>
       <collision>
@@ -115,5 +112,5 @@
           <mesh filename="package://abb_irb1600_support/meshes/irb1600/collision/link_6.stl"/>
         </geometry>
-        <material name="yellow"/>
+        <xacro:material_abb_yellow />
       </collision>
     </link>
