Commit message: fix irb1600 colors, use standard colors from abb_resources

File: abb_irb1600_support/urdf/irb1600_10_145_macro.xacro (robot description, xacro)
@@ -2,4 +2,5 @@
 <robot xmlns:xacro="http://ros.org/wiki/xacro" name="irb1600_10_145">
 <xacro:macro name="abb_irb1600_10_145" params="prefix">
+  <xacro:include filename="$(find abb_resources)/urdf/common_materials.xacro"/>
   <!-- link list -->
   <link name="${prefix}base_link">
@@ -9,7 +10,5 @@
         <mesh filename="package://abb_irb1600_support/meshes/irb1600/visual/base_link.stl"/>
       </geometry>
-      <material name="abb_orange">
-        <color rgba="1 0.43 0 1"/>
-      </material>
+      <xacro:material_abb_orange/>
     </visual>
     <collision>
@@ -17,7 +16,5 @@
         <mesh filename="package://abb_irb1600_support/meshes/irb1600/collision/base_link.stl"/>
       </geometry>
-      <material name="yellow">
-        <color rgba="0 1 1 1"/>
-      </material>
+      <xacro:material_abb_yellow/>
     </collision>
   </link>
@@ -28,5 +25,5 @@
         <mesh filename="package://abb_irb1600_support/meshes/irb1600/visual/link_1.stl"/>
       </geometry>
-      <material name="abb_orange"/>
+      <xacro:material_abb_orange/>
     </visual>
     <collision>
@@ -35,5 +32,5 @@
         <mesh filename="package://abb_irb1600_support/meshes/irb1600/collision/link_1.stl"/>
       </geometry>
-      <material name="yellow"/>
+      <xacro:material_abb_yellow/>
     </collision>
   </link>
@@ -44,5 +41,5 @@
         <mesh filename="package://abb_irb1600_support/meshes/irb1600_10_145/visual/link_2.stl"/>
       </geometry>
-      <material name="abb_orange"/>
+      <xacro:material_abb_orange/>
     </visual>
     <collision>
@@ -51,5 +48,5 @@
         <mesh filename="package://abb_irb1600_support/meshes/irb1600_10_145/collision/link_2.stl"/>
       </geometry>
-      <material name="yellow"/>
+      <xacro:material_abb_yellow/>
     </collision>
   </link>
@@ -60,5 +57,5 @@
         <mesh filename="package://abb_irb1600_support/meshes/irb1600/visual/link_3.stl"/>
       </geometry>
-      <material name="abb_orange"/>
+      <xacro:material_abb_orange/>
     </visual>
     <collision>
@@ -67,5 +64,5 @@
         <mesh filename="package://abb_irb1600_support/meshes/irb1600/collision/link_3.stl"/>
       </geometry>
-      <material name="yellow"/>
+      <xacro:material_abb_yellow/>
     </collision>
   </link>
@@ -76,5 +73,5 @@
         <mesh filename="package://abb_irb1600_support/meshes/irb1600/visual/link_4.stl"/>
       </geometry>
-      <material name="abb_orange"/>
+      <xacro:material_abb_orange/>
     </visual>
     <collision>
@@ -83,5 +80,5 @@
         <mesh filename="package://abb_irb1600_support/meshes/irb1600/collision/link_4.stl"/>
       </geometry>
-      <material name="yellow"/>
+      <xacro:material_abb_yellow/>
     </collision>
   </link>
@@ -92,5 +89,5 @@
         <mesh filename="package://abb_irb1600_support/meshes/irb1600/visual/link_5.stl"/>
       </geometry>
-      <material name="abb_orange"/>
+      <xacro:material_abb_orange/>
     </visual>
     <collision>
@@ -99,5 +96,5 @@
         <mesh filename="package://abb_irb1600_support/meshes/irb1600/collision/link_5.stl"/>
       </geometry>
-      <material name="yellow"/>
+      <xacro:material_abb_yellow/>
     </collision>
   </link>
@@ -108,5 +105,5 @@
         <mesh filename="package://abb_irb1600_support/meshes/irb1600/visual/link_6.stl"/>
       </geometry>
-      <material name="abb_orange"/>
+      <xacro:material_abb_orange/>
     </visual>
     <collision>
@@ -115,5 +112,5 @@
         <mesh filename="package://abb_irb1600_support/meshes/irb1600/collision/link_6.stl"/>
       </geometry>
-      <material name="yellow"/>
+      <xacro:material_abb_yellow/>
     </collision>
   </link>

File: abb_irb1600_support/urdf/irb1600_6_12_macro.xacro (robot description, xacro)
@@ -2,4 +2,5 @@
 <robot xmlns:xacro="http://ros.org/wiki/xacro" name="irb1600_6_12">
 <xacro:macro name="abb_irb1600_6_12" params="prefix">
+  <xacro:include filename="$(find abb_resources)/urdf/common_materials.xacro"/>
   <!-- link list -->
   <link name="${prefix}base_link">
@@ -9,7 +10,5 @@
         <mesh filename="package://abb_irb1600_support/meshes/irb1600/visual/base_link.stl"/>
       </geometry>
-      <material name="abb_orange">
-        <color rgba="1 0.43 0 1"/>
-      </material>
+      <xacro:material_abb_orange/>
     </visual>
     <collision>
@@ -17,7 +16,5 @@
         <mesh filename="package://abb_irb1600_support/meshes/irb1600/collision/base_link.stl"/>
       </geometry>
-      <material name="yellow">
-        <color rgba="0 1 1 1"/>
-      </material>
+      <xacro:material_abb_yellow/>
     </collision>
   </link>
@@ -28,5 +25,5 @@
         <mesh filename="package://abb_irb1600_support/meshes/irb1600/visual/link_1.stl"/>
       </geometry>
-      <material name="abb_orange"/>
+      <xacro:material_abb_orange/>
     </visual>
     <collision>
@@ -35,5 +32,5 @@
         <mesh filename="package://abb_irb1600_support/meshes/irb1600/collision/link_1.stl"/>
       </geometry>
-      <material name="yellow"/>
+      <xacro:material_abb_yellow/>
     </collision>
   </link>
@@ -44,5 +41,5 @@
         <mesh filename="package://abb_irb1600_support/meshes/irb1600_6_12/visual/link_2.stl"/>
       </geometry>
-      <material name="abb_orange"/>
+      <xacro:material_abb_orange/>
     </visual>
     <collision>
@@ -51,5 +48,5 @@
         <mesh filename="package://abb_irb1600_support/meshes/irb1600_6_12/collision/link_2.stl"/>
       </geometry>
-      <material name="yellow"/>
+      <xacro:material_abb_yellow/>
     </collision>
   </link>
@@ -60,5 +57,5 @@
         <mesh filename="package://abb_irb1600_support/meshes/irb1600/visual/link_3.stl"/>
       </geometry>
-      <material name="abb_orange"/>
+      <xacro:material_abb_orange/>
     </visual>
     <collision>
@@ -67,5 +64,5 @@
         <mesh filename="package://abb_irb1600_support/meshes/irb1600/collision/link_3.stl"/>
       </geometry>
-      <material name="yellow"/>
+      <xacro:material_abb_yellow/>
     </collision>
   </link>
@@ -76,5 +73,5 @@
         <mesh filename="package://abb_irb1600_support/meshes/irb1600/visual/link_4.stl"/>
       </geometry>
-      <material name="abb_orange"/>
+      <xacro:material_abb_orange/>
     </visual>
     <collision>
@@ -83,5 +80,5 @@
         <mesh filename="package://abb_irb1600_support/meshes/irb1600/collision/link_4.stl"/>
       </geometry>
-      <material name="yellow"/>
+      <xacro:material_abb_yellow/>
     </collision>
   </link>
@@ -92,5 +89,5 @@
         <mesh filename="package://abb_irb1600_support/meshes/irb1600/visual/link_5.stl"/>
       </geometry>
-      <material name="abb_orange"/>
+      <xacro:material_abb_orange/>
     </visual>
     <collision>
@@ -99,5 +96,5 @@
         <mesh filename="package://abb_irb1600_support/meshes/irb1600/collision/link_5.stl"/>
       </geometry>
-      <material name="yellow"/>
+      <xacro:material_abb_yellow/>
     </collision>
   </link>
@@ -108,5 +105,5 @@
         <mesh filename="package://abb_irb1600_support/meshes/irb1600/visual/link_6.stl"/>
       </geometry>
-      <material name="abb_orange"/>
+      <xacro:material_abb_orange/>
     </visual>
     <collision>
@@ -115,5 +112,5 @@
         <mesh filename="package://abb_irb1600_support/meshes/irb1600/collision/link_6.stl"/>
       </geometry>
-      <material name="yellow"/>
+      <xacro:material_abb_yellow/>
     </collision>
   </link>

Commit message: use the same link_2 mesh for irb1600 8&10/1.45

File: abb_irb1600_support/urdf/irb1600_10_145_macro.xacro (robot description, xacro)
@@ -39,5 +39,5 @@
       <origin xyz="0 0 0" rpy="0 0 0"/>
       <geometry>
-        <mesh filename="package://abb_irb1600_support/meshes/irb1600_10_145/visual/link_2.stl"/>
+        <mesh filename="package://abb_irb1600_support/meshes/irb1600_x_145/visual/link_2.stl"/>
       </geometry>
       <xacro:material_abb_orange/>
@@ -46,5 +46,5 @@
       <origin xyz="0 0 0" rpy="0 0 0"/>
       <geometry>
-        <mesh filename="package://abb_irb1600_support/meshes/irb1600_10_145/collision/link_2.stl"/>
+        <mesh filename="package://abb_irb1600_support/meshes/irb1600_x_145/collision/link_2.stl"/>
       </geometry>
       <xacro:material_abb_yellow/>

File: abb_irb1600_support/urdf/irb1600_8_145_macro.xacro (robot description, xacro)
@@ -39,5 +39,5 @@
         <origin xyz="0 0 0" rpy="0 0 0"/>
         <geometry>
-          <mesh filename="package://abb_irb1600_support/meshes/irb1600_8_145/visual/link_2.stl"/>
+          <mesh filename="package://abb_irb1600_support/meshes/irb1600_x_145/visual/link_2.stl"/>
         </geometry>
         <xacro:material_abb_orange />
@@ -46,5 +46,5 @@
         <origin xyz="0 0 0" rpy="0 0 0"/>
         <geometry>
-          <mesh filename="package://abb_irb1600_support/meshes/irb1600_8_145/collision/link_2.stl"/>
+          <mesh filename="package://abb_irb1600_support/meshes/irb1600_x_145/collision/link_2.stl"/>
         </geometry>
         <xacro:material_abb_yellow />
