Commit message: Added missing abb colour black to abb_resource

File: abb_resources/urdf/common_colours.xacro (robot description, xacro)
@@ -12,6 +12,8 @@
   <!-- RAL 7032 pebble gray, controller -->
   <xacro:property name="colour_abb_pebble_gray" value="0.7058823 0.6901961 0.6313725 1" />
-  <!-- RAL 7012 basalt gray (abb dark gray) , robot with dark link color -->
+  <!-- RAL 7012 basalt gray (abb dark gray) , robot primer -->
   <xacro:property name="colour_abb_dark_gray" value="0.3450980 0.3647059 0.3686275 1" />
+  <!-- RAL 7021 black gray (abb black) , robot with dark link color -->
+  <xacro:property name="colour_abb_black" value="0.1882353 0.1960784 0.2039216 1" />
   <!-- Other robot colours availble, but not limited too. -->
   <!-- RAL 3001 signal red -->

File: abb_resources/urdf/common_materials.xacro (robot description, xacro)
@@ -25,4 +25,9 @@
     <material name="">
       <color rgba="${colour_abb_dark_gray}"/>
+    </material>
+  </xacro:macro>
+  <xacro:macro name="material_abb_black">
+    <material name="">
+      <color rgba="${colour_abb_black}"/>
     </material>
   </xacro:macro>
