Commit message: Various clean-up changes per Levi-Armstrong

File: abb_irb52_support/urdf/irb52_7_145_macro.xacro (robot description, xacro)
@@ -1,176 +1,176 @@
 <?xml version="1.0"?>
 <robot xmlns:xacro="http://ros.org/wiki/xacro">
-    <xacro:include filename="$(find abb_resources)/urdf/common_materials.xacro"/>
-    <xacro:macro name="abb_irb52_7_145" params="prefix">
-        <!-- link list -->
-        <link name="${prefix}base_link">
-            <visual>
-                <origin xyz="0 0 0" rpy="0 0 0"/>
-                <geometry>
-                    <mesh filename="package://abb_irb52_support/meshes/irb52/visual/base_link.stl"/>
-                </geometry>
-                <xacro:material_abb_orange />
-            </visual>
-            <collision>
-                <geometry>
-                    <mesh filename="package://abb_irb52_support/meshes/irb52/collision/base_link.stl"/>
-                </geometry>
-                <xacro:material_abb_yellow />
-            </collision>
-        </link>
-        <link name="${prefix}link_1">
-            <visual>
-                <origin xyz="0 0 0" rpy="0 0 0"/>
-                <geometry>
-                    <mesh filename="package://abb_irb52_support/meshes/irb52/visual/link_1.stl"/>
-                </geometry>
-                <xacro:material_abb_orange />
-            </visual>
-            <collision>
-                <origin xyz="0 0 0" rpy="0 0 0"/>
-                <geometry>
-                    <mesh filename="package://abb_irb52_support/meshes/irb52/collision/link_1.stl"/>
-                </geometry>
-                <xacro:material_abb_yellow />
-            </collision>
-        </link>
-        <link name="${prefix}link_2">
-            <visual>
-                <origin xyz="0 0 0" rpy="0 0 0"/>
-                <geometry>
-                    <mesh filename="package://abb_irb52_support/meshes/irb52_7_145/visual/link_2.stl"/>
-                </geometry>
-                <xacro:material_abb_orange />
-            </visual>
-            <collision>
-                <origin xyz="0 0 0" rpy="0 0 0"/>
-                <geometry>
-                    <mesh filename="package://abb_irb52_support/meshes/irb52_7_145/collision/link_2.stl"/>
-                </geometry>
-                <xacro:material_abb_yellow />
-            </collision>
-        </link>
-        <link name="${prefix}link_3">
-            <visual>
-                <origin xyz="0 0 0" rpy="0 0 0"/>
-                <geometry>
-                    <mesh filename="package://abb_irb52_support/meshes/irb52/visual/link_3.stl"/>
-                </geometry>
-                <xacro:material_abb_orange />
-            </visual>
-            <collision>
-                <origin xyz="0 0 0" rpy="0 0 0"/>
-                <geometry>
-                    <mesh filename="package://abb_irb52_support/meshes/irb52/collision/link_3.stl"/>
-                </geometry>
-                <xacro:material_abb_yellow />
-            </collision>
-        </link>
-        <link name="${prefix}link_4">
-            <visual>
-                <origin xyz="0.600 0 0" rpy="0 0 0"/>
-                <geometry>
-                    <mesh filename="package://abb_irb52_support/meshes/irb52/visual/link_4.stl"/>
-                </geometry>
-                <xacro:material_abb_orange />
-            </visual>
-            <collision>
-                <origin xyz="0.600 0 0" rpy="0 0 0"/>
-                <geometry>
-                    <mesh filename="package://abb_irb52_support/meshes/irb52/collision/link_4.stl"/>
-                </geometry>
-                <xacro:material_abb_yellow />
-            </collision>
-        </link>
-        <link name="${prefix}link_5">
-            <visual>
-                <origin xyz="0 0 0" rpy="0 0 0"/>
-                <geometry>
-                    <mesh filename="package://abb_irb52_support/meshes/irb52/visual/link_5.stl"/>
-                </geometry>
-                <xacro:material_abb_orange />
-            </visual>
-            <collision>
-                <origin xyz="0 0 0" rpy="0 0 0"/>
-                <geometry>
-                    <mesh filename="package://abb_irb52_support/meshes/irb52/collision/link_5.stl"/>
-                </geometry>
-                <xacro:material_abb_yellow />
-            </collision>
-        </link>
-        <link name="${prefix}link_6">
-            <visual>
-                <origin xyz="0 0 0" rpy="0 0 0"/>
-                <geometry>
-                    <mesh filename="package://abb_irb52_support/meshes/irb52/visual/link_6.stl"/>
-                </geometry>
-                <xacro:material_abb_black />
-            </visual>
-            <collision>
-                <origin xyz="0 0 0" rpy="0 0 0"/>
-                <geometry>
-                    <mesh filename="package://abb_irb52_support/meshes/irb52/collision/link_6.stl"/>
-                </geometry>
-                <xacro:material_abb_black />
-            </collision>
-        </link>
-        <link name="${prefix}tool0"/>
-        <!-- end of link list -->
-        <!-- joint list -->
-        <joint name="${prefix}joint_1" type="revolute">
-            <origin xyz="0 0 0" rpy="0 0 0"/>
-            <parent link="${prefix}base_link"/>
-            <child link="${prefix}link_1"/>
-            <axis xyz="0 0 1"/>
-            <limit lower="${radians(-180)}" upper="${radians(180)}" effort="0" velocity="${radians(180)}"/>
-        </joint>
-        <joint name="${prefix}joint_2" type="revolute">
-            <origin xyz="0.150 0 0.4865" rpy="0 0 0"/>
-            <parent link="${prefix}link_1"/>
-            <child link="${prefix}link_2"/>
-            <axis xyz="0 1 0"/>
-            <limit lower="${radians(-90)}" upper="${radians(120)}" effort="0" velocity="${radians(180)}"/>
-        </joint>
-        <joint name="${prefix}joint_3" type="revolute">
-            <origin xyz="0 0 0.700" rpy="0 0 0"/>
-            <parent link="${prefix}link_2"/>
-            <child link="${prefix}link_3"/>
-            <axis xyz="0 1 0"/>
-            <limit lower="${radians(-245)}" upper="${radians(65)}" effort="0" velocity="${radians(180)}"/>
-        </joint>
-        <joint name="${prefix}joint_4" type="revolute">
-            <origin xyz="0 0 0" rpy="0 0 0"/>
-            <parent link="${prefix}link_3"/>
-            <child link="${prefix}link_4"/>
-            <axis xyz="1 0 0"/>
-            <limit lower="${radians(-200)}" upper="${radians(200)}" effort="0" velocity="${radians(180)}"/>
-        </joint>
-        <joint name="${prefix}joint_5" type="revolute">
-            <origin xyz="0.600 0 0" rpy="0 0 0"/>
-            <parent link="${prefix}link_4"/>
-            <child link="${prefix}link_5"/>
-            <axis xyz="0 1 0"/>
-            <limit lower="${radians(-115)}" upper="${radians(115)}" effort="0" velocity="${radians(180)}"/>
-        </joint>
-        <joint name="${prefix}joint_6" type="revolute">
-            <origin xyz="0.065 0 0" rpy="0 0 0"/>
-            <parent link="${prefix}link_5"/>
-            <child link="${prefix}link_6"/>
-            <axis xyz="1 0 0"/>
-            <limit lower="${radians(-400)}" upper="${radians(400)}" effort="0" velocity="${radians(180)}"/>
-        </joint>
-        <joint name="${prefix}joint_6-tool0" type="fixed">
-            <origin xyz="0 0 0" rpy="0 ${radians(90)} 0"/>
-            <parent link="${prefix}link_6"/>
-            <child link="${prefix}tool0"/>
-        </joint>
-        <!-- end of joint list -->
-        <!-- ROS base_link to Robot Manufacturer World Coordinates transform -->
-        <link name="${prefix}base" />
-        <joint name="${prefix}base_link-base" type="fixed">
-            <origin xyz="0 0 0" rpy="0 0 0"/>
-            <parent link="${prefix}base_link"/>
-            <child link="${prefix}base"/>
-        </joint>
-    </xacro:macro>
+  <xacro:include filename="$(find abb_resources)/urdf/common_materials.xacro"/>
+  <xacro:macro name="abb_irb52_7_145" params="prefix">
+    <!-- link list -->
+    <link name="${prefix}base_link">
+      <visual>
+        <origin xyz="0 0 0" rpy="0 0 0"/>
+        <geometry>
+          <mesh filename="package://abb_irb52_support/meshes/irb52/visual/base_link.stl"/>
+        </geometry>
+        <xacro:material_abb_orange />
+      </visual>
+      <collision>
+        <geometry>
+          <mesh filename="package://abb_irb52_support/meshes/irb52/collision/base_link.stl"/>
+        </geometry>
+        <xacro:material_abb_yellow />
+      </collision>
+    </link>
+    <link name="${prefix}link_1">
+      <visual>
+        <origin xyz="0 0 0" rpy="0 0 0"/>
+        <geometry>
+          <mesh filename="package://abb_irb52_support/meshes/irb52/visual/link_1.stl"/>
+        </geometry>
+        <xacro:material_abb_orange />
+      </visual>
+      <collision>
+        <origin xyz="0 0 0" rpy="0 0 0"/>
+        <geometry>
+          <mesh filename="package://abb_irb52_support/meshes/irb52/collision/link_1.stl"/>
+        </geometry>
+        <xacro:material_abb_yellow />
+      </collision>
+    </link>
+    <link name="${prefix}link_2">
+      <visual>
+        <origin xyz="0 0 0" rpy="0 0 0"/>
+        <geometry>
+          <mesh filename="package://abb_irb52_support/meshes/irb52_7_145/visual/link_2.stl"/>
+        </geometry>
+        <xacro:material_abb_orange />
+      </visual>
+      <collision>
+        <origin xyz="0 0 0" rpy="0 0 0"/>
+        <geometry>
+          <mesh filename="package://abb_irb52_support/meshes/irb52_7_145/collision/link_2.stl"/>
+        </geometry>
+        <xacro:material_abb_yellow />
+      </collision>
+    </link>
+    <link name="${prefix}link_3">
+      <visual>
+        <origin xyz="0 0 0" rpy="0 0 0"/>
+        <geometry>
+          <mesh filename="package://abb_irb52_support/meshes/irb52/visual/link_3.stl"/>
+        </geometry>
+        <xacro:material_abb_orange />
+      </visual>
+      <collision>
+        <origin xyz="0 0 0" rpy="0 0 0"/>
+        <geometry>
+          <mesh filename="package://abb_irb52_support/meshes/irb52/collision/link_3.stl"/>
+        </geometry>
+        <xacro:material_abb_yellow />
+      </collision>
+    </link>
+    <link name="${prefix}link_4">
+      <visual>
+        <origin xyz="0.600 0 0" rpy="0 0 0"/>
+        <geometry>
+          <mesh filename="package://abb_irb52_support/meshes/irb52/visual/link_4.stl"/>
+        </geometry>
+        <xacro:material_abb_orange />
+      </visual>
+      <collision>
+        <origin xyz="0.600 0 0" rpy="0 0 0"/>
+        <geometry>
+          <mesh filename="package://abb_irb52_support/meshes/irb52/collision/link_4.stl"/>
+        </geometry>
+        <xacro:material_abb_yellow />
+      </collision>
+    </link>
+    <link name="${prefix}link_5">
+      <visual>
+        <origin xyz="0 0 0" rpy="0 0 0"/>
+        <geometry>
+          <mesh filename="package://abb_irb52_support/meshes/irb52/visual/link_5.stl"/>
+        </geometry>
+        <xacro:material_abb_orange />
+      </visual>
+      <collision>
+        <origin xyz="0 0 0" rpy="0 0 0"/>
+        <geometry>
+          <mesh filename="package://abb_irb52_support/meshes/irb52/collision/link_5.stl"/>
+        </geometry>
+        <xacro:material_abb_yellow />
+      </collision>
+    </link>
+    <link name="${prefix}link_6">
+      <visual>
+        <origin xyz="0 0 0" rpy="0 0 0"/>
+        <geometry>
+          <mesh filename="package://abb_irb52_support/meshes/irb52/visual/link_6.stl"/>
+        </geometry>
+        <xacro:material_abb_black />
+      </visual>
+      <collision>
+        <origin xyz="0 0 0" rpy="0 0 0"/>
+        <geometry>
+          <mesh filename="package://abb_irb52_support/meshes/irb52/collision/link_6.stl"/>
+        </geometry>
+        <xacro:material_abb_black />
+      </collision>
+    </link>
+    <link name="${prefix}tool0"/>
+    <!-- end of link list -->
+    <!-- joint list -->
+    <joint name="${prefix}joint_1" type="revolute">
+      <origin xyz="0 0 0.4865" rpy="0 0 0"/>
+      <parent link="${prefix}base_link"/>
+      <child link="${prefix}link_1"/>
+      <axis xyz="0 0 1"/>
+      <limit lower="${radians(-180)}" upper="${radians(180)}" effort="0" velocity="${radians(180)}"/>
+    </joint>
+    <joint name="${prefix}joint_2" type="revolute">
+      <origin xyz="0.150 0 0" rpy="0 0 0"/>
+      <parent link="${prefix}link_1"/>
+      <child link="${prefix}link_2"/>
+      <axis xyz="0 1 0"/>
+      <limit lower="${radians(-90)}" upper="${radians(120)}" effort="0" velocity="${radians(180)}"/>
+    </joint>
+    <joint name="${prefix}joint_3" type="revolute">
+      <origin xyz="0 0 0.700" rpy="0 0 0"/>
+      <parent link="${prefix}link_2"/>
+      <child link="${prefix}link_3"/>
+      <axis xyz="0 1 0"/>
+      <limit lower="${radians(-245)}" upper="${radians(65)}" effort="0" velocity="${radians(180)}"/>
+    </joint>
+    <joint name="${prefix}joint_4" type="revolute">
+      <origin xyz="0 0 0" rpy="0 0 0"/>
+      <parent link="${prefix}link_3"/>
+      <child link="${prefix}link_4"/>
+      <axis xyz="1 0 0"/>
+      <limit lower="${radians(-200)}" upper="${radians(200)}" effort="0" velocity="${radians(180)}"/>
+    </joint>
+    <joint name="${prefix}joint_5" type="revolute">
+      <origin xyz="0.600 0 0" rpy="0 0 0"/>
+      <parent link="${prefix}link_4"/>
+      <child link="${prefix}link_5"/>
+      <axis xyz="0 1 0"/>
+      <limit lower="${radians(-115)}" upper="${radians(115)}" effort="0" velocity="${radians(180)}"/>
+    </joint>
+    <joint name="${prefix}joint_6" type="revolute">
+      <origin xyz="0.065 0 0" rpy="0 0 0"/>
+      <parent link="${prefix}link_5"/>
+      <child link="${prefix}link_6"/>
+      <axis xyz="1 0 0"/>
+      <limit lower="${radians(-400)}" upper="${radians(400)}" effort="0" velocity="${radians(180)}"/>
+    </joint>
+    <joint name="${prefix}joint_6-tool0" type="fixed">
+      <origin xyz="0 0 0" rpy="0 ${radians(90)} 0"/>
+      <parent link="${prefix}link_6"/>
+      <child link="${prefix}tool0"/>
+    </joint>
+    <!-- end of joint list -->
+    <!-- ROS base_link to Robot Manufacturer World Coordinates transform -->
+    <link name="${prefix}base" />
+    <joint name="${prefix}base_link-base" type="fixed">
+      <origin xyz="0 0 0" rpy="0 0 0"/>
+      <parent link="${prefix}base_link"/>
+      <child link="${prefix}base"/>
+    </joint>
+  </xacro:macro>
 </robot>

Commit message: Added flange frame for irb52

File: abb_irb52_support/urdf/irb52_7_120_macro.xacro (robot description, xacro)
@@ -115,5 +115,4 @@
       </collision>
     </link>
-    <link name="${prefix}tool0"/>
     <!-- end of link list -->
     <!-- joint list -->
@@ -160,11 +159,6 @@
       <limit lower="${radians(-400)}" upper="${radians(400)}" effort="0" velocity="${radians(180)}"/>
     </joint>
-    <joint name="${prefix}joint_6-tool0" type="fixed">
-      <origin xyz="0 0 0" rpy="0 ${radians(90)} 0"/>
-      <parent link="${prefix}link_6"/>
-      <child link="${prefix}tool0"/>
-    </joint>
     <!-- end of joint list -->
-    <!-- ROS base_link to Robot Manufacturer World Coordinates transform -->
+    <!-- ROS-Industrial 'base' frame: base_link to ABB World Coordinates transform -->
     <link name="${prefix}base" />
     <joint name="${prefix}base_link-base" type="fixed">
@@ -173,4 +167,18 @@
       <child link="${prefix}base"/>
     </joint>
+    <!-- ROS-Industrial 'flange' frame: attachment point for EEF models -->
+    <link name="${prefix}flange"/>
+    <joint type="fixed" name="${prefix}joint_6-flange">
+      <origin xyz="0 0 0" rpy="0 0 0"/>
+      <parent link="${prefix}link_6"/>
+      <child link="${prefix}flange"/>
+    </joint>
+    <!-- ROS-Industrial 'tool0' frame: all-zeros tool frame -->
+    <link name="${prefix}tool0" />
+    <joint name="${prefix}link_6-tool0" type="fixed">
+      <origin xyz="0 0 0" rpy="0 ${radians(90)} 0" />
+      <parent link="${prefix}flange" />
+      <child link="${prefix}tool0" />
+    </joint>
   </xacro:macro>
 </robot>

File: abb_irb52_support/urdf/irb52_7_145_macro.xacro (robot description, xacro)
@@ -115,5 +115,4 @@
       </collision>
     </link>
-    <link name="${prefix}tool0"/>
     <!-- end of link list -->
     <!-- joint list -->
@@ -160,11 +159,6 @@
       <limit lower="${radians(-400)}" upper="${radians(400)}" effort="0" velocity="${radians(180)}"/>
     </joint>
-    <joint name="${prefix}joint_6-tool0" type="fixed">
-      <origin xyz="0 0 0" rpy="0 ${radians(90)} 0"/>
-      <parent link="${prefix}link_6"/>
-      <child link="${prefix}tool0"/>
-    </joint>
     <!-- end of joint list -->
-    <!-- ROS base_link to Robot Manufacturer World Coordinates transform -->
+    <!-- ROS-Industrial 'base' frame: base_link to ABB World Coordinates transform -->
     <link name="${prefix}base" />
     <joint name="${prefix}base_link-base" type="fixed">
@@ -173,4 +167,18 @@
       <child link="${prefix}base"/>
     </joint>
+    <!-- ROS-Industrial 'flange' frame: attachment point for EEF models -->
+    <link name="${prefix}flange"/>
+    <joint type="fixed" name="${prefix}joint_6-flange">
+      <origin xyz="0 0 0" rpy="0 0 0"/>
+      <parent link="${prefix}link_6"/>
+      <child link="${prefix}flange"/>
+    </joint>
+    <!-- ROS-Industrial 'tool0' frame: all-zeros tool frame -->
+    <link name="${prefix}tool0" />
+    <joint name="${prefix}link_6-tool0" type="fixed">
+      <origin xyz="0 0 0" rpy="0 ${radians(90)} 0" />
+      <parent link="${prefix}flange" />
+      <child link="${prefix}tool0" />
+    </joint>
   </xacro:macro>
 </robot>
