Commit message: Renamed all references to the irb120t to irb120t_3_58

File: abb_irb120_gazebo/urdf/irb120_3_58.xacro (robot description, xacro)
@@ -1,6 +1,6 @@
 <?xml version="1.0" ?>
-<robot name="abb_irb120t" xmlns:xacro="http://ros.org/wiki/xacro">
-  <xacro:include filename="$(find abb_irb120_gazebo)/urdf/irb120t_macro.xacro"/>
-  <xacro:abb_irb120t_g prefix=""/>
+<robot name="abb_irb120_3_58" xmlns:xacro="http://ros.org/wiki/xacro">
+  <xacro:include filename="$(find abb_irb120_gazebo)/urdf/irb120_3_58_macro.xacro"/>
+  <xacro:abb_irb120_3_58_g prefix=""/>
   <!-- Fix robot to Gazebo world -->
   <link name="world"/>

File: abb_irb120_gazebo/urdf/irb120_3_58_macro.xacro (robot description, xacro)
@@ -1,8 +1,8 @@
 <?xml version="1.0"?>
 <robot xmlns:xacro="http://ros.org/wiki/xacro">
-<xacro:include filename="$(find abb_irb120_support)/urdf/irb120_macro.xacro"/>
-<xacro:macro name="abb_irb120_g" params="prefix">
+<xacro:include filename="$(find abb_irb120_support)/urdf/irb120_3_58_macro.xacro"/>
+<xacro:macro name="abb_irb120_3_58_g" params="prefix">
   <!-- get base ABB IRB120 model -->
-  <xacro:abb_irb120 prefix="${prefix}" />
+  <xacro:abb_irb120_3_58 prefix="${prefix}" />
   <!-- transmission list -->
   <transmission name="${prefix}tran1">

File: abb_irb120_gazebo/urdf/irb120t_3_58.xacro (robot description, xacro)
@@ -1,6 +1,6 @@
 <?xml version="1.0" ?>
-<robot name="abb_irb120" xmlns:xacro="http://ros.org/wiki/xacro">
-  <xacro:include filename="$(find abb_irb120_gazebo)/urdf/irb120_macro.xacro"/>
-  <xacro:abb_irb120_g prefix=""/>
+<robot name="abb_irb120t_3_58" xmlns:xacro="http://ros.org/wiki/xacro">
+  <xacro:include filename="$(find abb_irb120_gazebo)/urdf/irb120t_3_58_macro.xacro"/>
+  <xacro:abb_irb120t_3_58_g prefix=""/>
   <!-- Fix robot to Gazebo world -->
   <link name="world"/>

File: abb_irb120_gazebo/urdf/irb120t_3_58_macro.xacro (robot description, xacro)
@@ -1,8 +1,8 @@
 <?xml version="1.0"?>
 <robot xmlns:xacro="http://ros.org/wiki/xacro">
-<xacro:include filename="$(find abb_irb120_support)/urdf/irb120t_macro.xacro"/>
-<xacro:macro name="abb_irb120t_g" params="prefix">
+<xacro:include filename="$(find abb_irb120_support)/urdf/irb120t_3_58_macro.xacro"/>
+<xacro:macro name="abb_irb120t_3_58_g" params="prefix">
   <!-- get base ABB IRB120T model -->
-  <xacro:abb_irb120t prefix="${prefix}" />
+  <xacro:abb_irb120t_3_58 prefix="${prefix}" />
   <!-- transmission list -->
   <transmission name="${prefix}tran1">

File: abb_irb120_support/urdf/irb120_3_58.urdf (robot description, URDF)
Before this commit: robot abb_irb120, 9 links, 8 joints
Links:
- link base_link: geometry collision mesh filename=package://abb_irb120_support/meshes/irb120_3_58/collision/b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; visual mesh filename=package://abb_irb120_support/meshes/irb120_3_58/visual/base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
- link link_1: geometry collision mesh filename=package://abb_irb120_support/meshes/irb120_3_58/collision/l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; visual mesh filename=package://abb_irb120_support/meshes/irb120_3_58/visual/link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
- link link_2: geometry collision mesh filename=package://abb_irb120_support/meshes/irb120_3_58/collision/l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; visual mesh filename=package://abb_irb120_support/meshes/irb120_3_58/visual/link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
- link link_3: geometry collision mesh filename=package://abb_irb120_support/meshes/irb120_3_58/collision/l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; visual mesh filename=package://abb_irb120_support/meshes/irb120_3_58/visual/link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
- link link_4: geometry collision mesh filename=package://abb_irb120_support/meshes/irb120_3_58/collision/l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; visual mesh filename=package://abb_irb120_support/meshes/irb120_3_58/visual/link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
- link link_5: geometry collision mesh filename=package://abb_irb120_support/meshes/irb120_3_58/collision/l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; visual mesh filename=package://abb_irb120_support/meshes/irb120_3_58/visual/link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
- link link_6: geometry collision mesh filename=package://abb_irb120_support/meshes/irb120_3_58/collision/l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; visual mesh filename=package://abb_irb120_support/meshes/irb120_3_58/visual/link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

File: abb_irb120_support/urdf/irb120_3_58_macro.xacro (robot description, xacro)
@@ -2,23 +2,23 @@
 <robot xmlns:xacro="http://ros.org/wiki/xacro">
   <xacro:include filename="$(find abb_resources)/urdf/common_materials.xacro"/>
-  <xacro:macro name="abb_irb120t" params="prefix">
+  <xacro:macro name="abb_irb120_3_58" params="prefix">
     <!-- link list -->
     <link name="${prefix}base_link">
-    	<inertial>
-    	  <mass value="6.215"/>
-    	  <origin xyz="-0.04204 8.01E-05 0.07964" rpy="0 0 0"/>
-    	  <inertia ixx="0.0247272" ixy="-8.0784E-05" ixz="0.00130902" iyy="0.0491285" iyz="-8.0419E-06" izz="0.0472376"/>
-    	</inertial>
-      <visual>
-        <origin xyz="0 0 0" rpy="0 0 0"/>
-        <geometry>
-          <mesh filename="package://abb_irb120_support/meshes/irb120/visual/base_link.stl"/>
-        </geometry>
-        <xacro:material_abb_orange />
-      </visual>
-      <collision>
-        <origin xyz="0 0 0" rpy="0 0 0"/>
-        <geometry>
-          <mesh filename="package://abb_irb120_support/meshes/irb120/collision/base_link.stl"/>
+      <inertial>
+        <mass value="6.215"/>
+        <origin xyz="-0.04204 8.01E-05 0.07964" rpy="0 0 0"/>
+        <inertia ixx="0.0247272" ixy="-8.0784E-05" ixz="0.00130902" iyy="0.0491285" iyz="-8.0419E-06" izz="0.0472376"/>
+      </inertial>
+      <visual>
+        <origin xyz="0 0 0" rpy="0 0 0"/>
+        <geometry>
+          <mesh filename="package://abb_irb120_support/meshes/irb120_3_58/visual/base_link.stl"/>
+        </geometry>
+        <xacro:material_abb_orange />
+      </visual>
+      <collision>
+        <origin xyz="0 0 0" rpy="0 0 0"/>
+        <geometry>
+          <mesh filename="package://abb_irb120_support/meshes/irb120_3_58/collision/base_link.stl"/>
         </geometry>
         <xacro:material_abb_yellow />
@@ -26,20 +26,20 @@
     </link>
     <link name="${prefix}link_1">
-    	<inertial>
-    	  <mass value="3.067" />
-    	  <origin xyz="9.77E-05 -0.00012 0.23841" rpy="0 0 0"/>
-    	  <inertia ixx="0.0142175" ixy="-1.28579E-05" ixz="-2.31364E-05" iyy="0.0144041" iyz="1.93404E-05" izz="0.0104533"/>
-    	</inertial>
-      <visual>
-        <origin xyz="0 0 0" rpy="0 0 0"/>
-        <geometry>
-          <mesh filename="package://abb_irb120_support/meshes/irb120/visual/link_1.stl"/>
-        </geometry>
-        <xacro:material_abb_orange />
-      </visual>
-      <collision>
-        <origin xyz="0 0 0" rpy="0 0 0"/>
-        <geometry>
-          <mesh filename="package://abb_irb120_support/meshes/irb120/collision/link_1.stl"/>
+      <inertial>
+        <mass value="3.067" />
+        <origin xyz="9.77E-05 -0.00012 0.23841" rpy="0 0 0"/>
+        <inertia ixx="0.0142175" ixy="-1.28579E-05" ixz="-2.31364E-05" iyy="0.0144041" iyz="1.93404E-05" izz="0.0104533"/>
+      </inertial>
+      <visual>
+        <origin xyz="0 0 0" rpy="0 0 0"/>
+        <geometry>
+          <mesh filename="package://abb_irb120_support/meshes/irb120_3_58/visual/link_1.stl"/>
+        </geometry>
+        <xacro:material_abb_orange />
+      </visual>
+      <collision>
+        <origin xyz="0 0 0" rpy="0 0 0"/>
+        <geometry>
+          <mesh filename="package://abb_irb120_support/meshes/irb120_3_58/collision/link_1.stl"/>
         </geometry>
         <xacro:material_abb_yellow />
@@ -47,20 +47,20 @@
     </link>
     <link name="${prefix}link_2">
-    	<inertial>
-    	  <mass value="3.909"/>
-    	  <origin xyz="0.00078 -0.00212 0.10124" rpy="0 0 0"/>
-    	  <inertia ixx="0.0603111" ixy="9.83431E-06" ixz="5.72407E-05" iyy="0.041569" iyz="-0.00050497" izz="0.0259548"/>
-    	</inertial>
-      <visual>
-        <origin xyz="0 0 0" rpy="0 0 0"/>
-        <geometry>
-          <mesh filename="package://abb_irb120_support/meshes/irb120/visual/link_2.stl"/>
-        </geometry>
-        <xacro:material_abb_orange />
-      </visual>
-      <collision>
-        <origin xyz="0 0 0" rpy="0 0 0"/>
-        <geometry>
-          <mesh filename="package://abb_irb120_support/meshes/irb120/collision/link_2.stl"/>
+      <inertial>
+        <mass value="3.909"/>
+        <origin xyz="0.00078 -0.00212 0.10124" rpy="0 0 0"/>
+        <inertia ixx="0.0603111" ixy="9.83431E-06" ixz="5.72407E-05" iyy="0.041569" iyz="-0.00050497" izz="0.0259548"/>
+      </inertial>
+      <visual>
+        <origin xyz="0 0 0" rpy="0 0 0"/>
+        <geometry>
+          <mesh filename="package://abb_irb120_support/meshes/irb120_3_58/visual/link_2.stl"/>
+        </geometry>
+        <xacro:material_abb_orange />
+      </visual>
+      <collision>
+        <origin xyz="0 0 0" rpy="0 0 0"/>
+        <geometry>
+          <mesh filename="package://abb_irb120_support/meshes/irb120_3_58/collision/link_2.stl"/>
         </geometry>
         <xacro:material_abb_yellow />
@@ -68,20 +68,20 @@
     </link>
     <link name="${prefix}link_3">
-    	<inertial>
-    	  <mass value="2.944"/>
-    	  <origin xyz="0.02281 0.00106 0.05791" rpy="0 0 0"/>
-    	  <inertia ixx="0.00835606" ixy="-8.01545E-05" ixz="0.00142884" iyy="0.016713" iyz="-0.000182227" izz="0.0126984"/>
-    	</inertial>
-      <visual>
-        <origin xyz="0 0 0" rpy="0 0 0"/>
-        <geometry>
-          <mesh filename="package://abb_irb120_support/meshes/irb120/visual/link_3.stl"/>
-        </geometry>
-        <xacro:material_abb_orange />
-      </visual>
-      <collision>
-        <origin xyz="0 0 0" rpy="0 0 0"/>
-        <geometry>
-          <mesh filename="package://abb_irb120_support/meshes/irb120/collision/link_3.stl"/>
+      <inertial>
+        <mass value="2.944"/>
+        <origin xyz="0.02281 0.00106 0.05791" rpy="0 0 0"/>
+        <inertia ixx="0.00835606" ixy="-8.01545E-05" ixz="0.00142884" iyy="0.016713" iyz="-0.000182227" izz="0.0126984"/>
+      </inertial>
+      <visual>
+        <origin xyz="0 0 0" rpy="0 0 0"/>
+        <geometry>
+          <mesh filename="package://abb_irb120_support/meshes/irb120_3_58/visual/link_3.stl"/>
+        </geometry>
+        <xacro:material_abb_orange />
+      </visual>
+      <collision>
+        <origin xyz="0 0 0" rpy="0 0 0"/>
+        <geometry>
+          <mesh filename="package://abb_irb120_support/meshes/irb120_3_58/collision/link_3.stl"/>
         </geometry>
         <xacro:material_abb_yellow />
@@ -89,20 +89,20 @@
     </link>
     <link name="${prefix}link_4">
-    	<inertial>
-    	  <mass value="1.328"/>
-    	  <origin xyz="0.2247 0.00015 0.00041" rpy="0 0 0"/>
-    	  <inertia ixx="0.00284661" ixy="-2.12765E-05" ixz="-1.6435E-05" iyy="0.00401346" iyz="1.31336E-05" izz="0.0052535"/>
-    	</inertial>
-      <visual>
-        <origin xyz="0 0 0" rpy="0 0 0"/>
-        <geometry>
-          <mesh filename="package://abb_irb120_support/meshes/irb120/visual/link_4.stl"/>
-        </geometry>
-        <xacro:material_abb_orange />
-      </visual>
-      <collision>
-        <origin xyz="0 0 0" rpy="0 0 0"/>
-        <geometry>
-          <mesh filename="package://abb_irb120_support/meshes/irb120/collision/link_4.stl"/>
+      <inertial>
+        <mass value="1.328"/>
+        <origin xyz="0.2247 0.00015 0.00041" rpy="0 0 0"/>
+        <inertia ixx="0.00284661" ixy="-2.12765E-05" ixz="-1.6435E-05" iyy="0.00401346" iyz="1.31336E-05" izz="0.0052535"/>
+      </inertial>
+      <visual>
+        <origin xyz="0 0 0" rpy="0 0 0"/>
+        <geometry>
+          <mesh filename="package://abb_irb120_support/meshes/irb120_3_58/visual/link_4.stl"/>
+        </geometry>
+        <xacro:material_abb_orange />
+      </visual>
+      <collision>
+        <origin xyz="0 0 0" rpy="0 0 0"/>
+        <geometry>
+          <mesh filename="package://abb_irb120_support/meshes/irb120_3_58/collision/link_4.stl"/>
         </geometry>
         <xacro:material_abb_yellow />
@@ -110,20 +110,20 @@
     </link>
     <link name="${prefix}link_5">
-    	<inertial>
-    	  <mass value="0.546"/>
-    	  <origin xyz="-0.00109 3.68E-05 6.22E-05" rpy="0 0 0"/>
-    	  <inertia ixx="0.000404891" ixy="1.61943E-06" ixz="8.46805E-07" iyy="0.000892825" iyz="-1.51792E-08" izz="0.000815468"/>
-    	</inertial>
-      <visual>
-        <origin xyz="0 0 0" rpy="0 0 0"/>
-        <geometry>
-          <mesh filename="package://abb_irb120_support/meshes/irb120/visual/link_5.stl"/>
-        </geometry>
-        <xacro:material_abb_orange />
-      </visual>
-      <collision>
-        <origin xyz="0 0 0" rpy="0 0 0"/>
-        <geometry>
-          <mesh filename="package://abb_irb120_support/meshes/irb120/collision/link_5.stl"/>
+      <inertial>
+        <mass value="0.546"/>
+        <origin xyz="-0.00109 3.68E-05 6.22E-05" rpy="0 0 0"/>
+        <inertia ixx="0.000404891" ixy="1.61943E-06" ixz="8.46805E-07" iyy="0.000892825" iyz="-1.51792E-08" izz="0.000815468"/>
+      </inertial>
+      <visual>
+        <origin xyz="0 0 0" rpy="0 0 0"/>
+        <geometry>
+          <mesh filename="package://abb_irb120_support/meshes/irb120_3_58/visual/link_5.stl"/>
+        </geometry>
+        <xacro:material_abb_orange />
+      </visual>
+      <collision>
+        <origin xyz="0 0 0" rpy="0 0 0"/>
+        <geometry>
+          <mesh filename="package://abb_irb120_support/meshes/irb120_3_58/collision/link_5.stl"/>
         </geometry>
         <xacro:material_abb_yellow />
@@ -131,13 +131,13 @@
     </link>
     <link name="${prefix}link_6">
-    	<inertial>
-    	  <mass value="0.137"/>
-    	  <origin xyz="-0.00706 -0.00017 -1.32E-06" rpy="0 0 0"/>
-    	  <inertia ixx="0.001" ixy="0" ixz="0" iyy="0.001" iyz="0" izz="0.001"/>
-    	</inertial>
-      <visual>
-        <origin xyz="0 0 0" rpy="0 0 0"/>
-        <geometry>
-          <mesh filename="package://abb_irb120_support/meshes/irb120/visual/link_6.stl"/>
+      <inertial>
+        <mass value="0.137"/>
+        <origin xyz="-0.00706 -0.00017 -1.32E-06" rpy="0 0 0"/>
+        <inertia ixx="0.001" ixy="0" ixz="0" iyy="0.001" iyz="0" izz="0.001"/>
+      </inertial>
+      <visual>
+        <origin xyz="0 0 0" rpy="0 0 0"/>
+        <geometry>
+          <mesh filename="package://abb_irb120_support/meshes/irb120_3_58/visual/link_6.stl"/>
         </geometry>
         <xacro:material_abb_black />
@@ -146,5 +146,5 @@
         <origin xyz="0 0 0" rpy="0 0 0"/>
         <geometry>
-          <mesh filename="package://abb_irb120_support/meshes/irb120/collision/link_6.stl"/>
+          <mesh filename="package://abb_irb120_support/meshes/irb120_3_58/collision/link_6.stl"/>
         </geometry>
         <xacro:material_abb_yellow />
@@ -160,5 +160,5 @@
       <limit effort="0" lower="-2.87979" upper="2.87979" velocity="4.36332"/>
       <axis xyz="0 0 1"/>
-    	<dynamics damping="0.0" friction="0.0"/>
+      <dynamics damping="0.0" friction="0.0"/>
     </joint>
     <joint name="${prefix}joint_2" type="revolute">
@@ -168,5 +168,5 @@
       <limit effort="0" lower="-1.91986" upper="1.91986" velocity="4.36332"/>
       <axis xyz="0 1 0"/>
-    	<dynamics damping="0.0" friction="0.0"/>
+      <dynamics damping="0.0" friction="0.0"/>
     </joint>
     <joint name="${prefix}joint_3" type="revolute">
@@ -176,5 +176,5 @@
       <limit effort="0" lower="-1.91986" upper="1.22173" velocity="4.36332"/>
       <axis xyz="0 1 0"/>
-    	<dynamics damping="0.0" friction="0.0"/>
+      <dynamics damping="0.0" friction="0.0"/>
     </joint>
     <joint name="${prefix}joint_4" type="revolute">
@@ -182,7 +182,7 @@
       <parent link="${prefix}link_3"/>
       <child link="${prefix}link_4"/>
-      <limit effort="0" lower="-2.79253" upper="2.79253" velocity="7.33038"/>
+      <limit effort="0" lower="-2.79253" upper="2.79253" velocity="5.58505"/>
       <axis xyz="1 0 0"/>
-    	<dynamics damping="0.0" friction="0.0"/>
+      <dynamics damping="0.0" friction="0.0"/>
     </joint>
     <joint name="${prefix}joint_5" type="revolute">
@@ -190,7 +190,7 @@
       <parent link="${prefix}link_4"/>
       <child link="${prefix}link_5"/>
-      <limit effort="0" lower="-2.094395" upper="2.094395" velocity="10.29744"/>
+      <limit effort="0" lower="-2.094395" upper="2.094395" velocity="5.58505"/>
       <axis xyz="0 1 0"/>
-    	<dynamics damping="0.0" friction="0.0"/>
+      <dynamics damping="0.0" friction="0.0"/>
     </joint>
     <joint name="${prefix}joint_6" type="revolute">
@@ -198,7 +198,7 @@
       <parent link="${prefix}link_5"/>
       <child link="${prefix}link_6"/>
-      <limit effort="0" lower="-6.98132" upper="6.98132" velocity="10.471975"/>
+      <limit effort="0" lower="-6.98132" upper="6.98132" velocity="7.33038"/>
       <axis xyz="1 0 0"/>
-    	<dynamics damping="0.0" friction="0.0"/>
+      <dynamics damping="0.0" friction="0.0"/>
     </joint>
     <joint name="${prefix}joint6-tool0" type="fixed">

File: abb_irb120_support/urdf/irb120t_3_58.urdf (robot description, URDF)
Before this commit: robot abb_irb120t, 9 links, 8 joints
Links:
- link base_link: geometry collision mesh filename=package://abb_irb120_support/meshes/irb120_3_58/collision/b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; visual mesh filename=package://abb_irb120_support/meshes/irb120_3_58/visual/base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
- link link_1: geometry collision mesh filename=package://abb_irb120_support/meshes/irb120_3_58/collision/l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; visual mesh filename=package://abb_irb120_support/meshes/irb120_3_58/visual/link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
- link link_2: geometry collision mesh filename=package://abb_irb120_support/meshes/irb120_3_58/collision/l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; visual mesh filename=package://abb_irb120_support/meshes/irb120_3_58/visual/link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
- link link_3: geometry collision mesh filename=package://abb_irb120_support/meshes/irb120_3_58/collision/l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; visual mesh filename=package://abb_irb120_support/meshes/irb120_3_58/visual/link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
- link link_4: geometry collision mesh filename=package://abb_irb120_support/meshes/irb120_3_58/collision/l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; visual mesh filename=package://abb_irb120_support/meshes/irb120_3_58/visual/link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
- link link_5: geometry collision mesh filename=package://abb_irb120_support/meshes/irb120_3_58/collision/l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; visual mesh filename=package://abb_irb120_support/meshes/irb120_3_58/visual/link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
- link link_6: geometry collision mesh filename=package://abb_irb120_support/meshes/irb120_3_58/collision/l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; visual mesh filename=package://abb_irb120_support/meshes/irb120_3_58/visual/link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
