Commit message: irb1200_7_70: fix mesh origins, scaling and normals.

File: abb_irb1200_support/urdf/irb1200_7_70_macro.xacro (robot description, xacro)
@@ -6,5 +6,5 @@
       <collision name="collision">
         <geometry>
-          <mesh filename="package://abb_irb1200_support/meshes/irb1200_7_70/collision/base_link.stl" scale="0.001 0.001 0.001" />
+          <mesh filename="package://abb_irb1200_support/meshes/irb1200_7_70/collision/base_link.stl" />
         </geometry>
         <material name="yellow">
@@ -14,5 +14,5 @@
       <visual name="visual">
         <geometry>
-          <mesh filename="package://abb_irb1200_support/meshes/irb1200_7_70/visual/base_link.stl" scale="0.001 0.001 0.001" />
+          <mesh filename="package://abb_irb1200_support/meshes/irb1200_7_70/visual/base_link.stl" />
         </geometry>
         <material name="graphite_white">
@@ -24,5 +24,5 @@
       <collision name="collision">
         <geometry>
-          <mesh filename="package://abb_irb1200_support/meshes/irb1200_7_70/collision/link_1.stl" scale="0.001 0.001 0.001" />
+          <mesh filename="package://abb_irb1200_support/meshes/irb1200_7_70/collision/link_1.stl" />
         </geometry>
         <material name="yellow"/>
@@ -30,5 +30,5 @@
       <visual name="visual">
         <geometry>
-          <mesh filename="package://abb_irb1200_support/meshes/irb1200_7_70/visual/link_1.stl" scale="0.001 0.001 0.001" />
+          <mesh filename="package://abb_irb1200_support/meshes/irb1200_7_70/visual/link_1.stl" />
         </geometry>
         <material name="graphite_white"/>
@@ -38,14 +38,12 @@
       <collision name="collision">
         <geometry>
-          <mesh filename="package://abb_irb1200_support/meshes/irb1200_7_70/collision/link_2.stl" scale="0.001 0.001 0.001" />
+          <mesh filename="package://abb_irb1200_support/meshes/irb1200_7_70/collision/link_2.stl" />
         </geometry>
-        <origin xyz="0 0 -0.399" />
         <material name="yellow"/>
       </collision>
       <visual name="visual">
         <geometry>
-          <mesh filename="package://abb_irb1200_support/meshes/irb1200_7_70/visual/link_2.stl" scale="0.001 0.001 0.001" />
+          <mesh filename="package://abb_irb1200_support/meshes/irb1200_7_70/visual/link_2.stl" />
         </geometry>
-        <origin xyz="0 0 -0.399" />
         <material name="graphite_white"/>
       </visual>
@@ -54,14 +52,12 @@
       <collision name="graphite_white">
         <geometry>
-          <mesh filename="package://abb_irb1200_support/meshes/irb1200_7_70/collision/link_3.stl" scale="0.001 0.001 0.001" />
+          <mesh filename="package://abb_irb1200_support/meshes/irb1200_7_70/collision/link_3.stl" />
         </geometry>
-        <origin xyz="0 0 -0.749" />
         <material name="yellow"/>
       </collision>
       <visual name="visual">
         <geometry>
-          <mesh filename="package://abb_irb1200_support/meshes/irb1200_7_70/visual/link_3.stl" scale="0.001 0.001 0.001" />
+          <mesh filename="package://abb_irb1200_support/meshes/irb1200_7_70/visual/link_3.stl" />
         </geometry>
-        <origin xyz="0 0 -0.749" />
         <material name="graphite_white"/>
       </visual>
@@ -70,14 +66,12 @@
       <collision name="collision">
         <geometry>
-          <mesh filename="package://abb_irb1200_support/meshes/irb1200_7_70/collision/link_4.stl" scale="0.001 0.001 0.001" />
+          <mesh filename="package://abb_irb1200_support/meshes/irb1200_7_70/collision/link_4.stl" />
         </geometry>
-        <origin xyz="0 0 ${-0.749 - 0.042}" />
         <material name="yellow"/>
       </collision>
       <visual name="visual">
         <geometry>
-          <mesh filename="package://abb_irb1200_support/meshes/irb1200_7_70/visual/link_4.stl" scale="0.001 0.001 0.001" />
+          <mesh filename="package://abb_irb1200_support/meshes/irb1200_7_70/visual/link_4.stl" />
         </geometry>
-        <origin xyz="0 0 ${-0.749 - 0.042}" />
         <material name="graphite_white"/>
       </visual>
@@ -86,14 +80,12 @@
       <collision name="collision">
         <geometry>
-          <mesh filename="package://abb_irb1200_support/meshes/irb1200_7_70/collision/link_5.stl" scale="0.001 0.001 0.001" />
+          <mesh filename="package://abb_irb1200_support/meshes/irb1200_7_70/collision/link_5.stl" />
         </geometry>
-        <origin xyz="-0.351 0 ${-0.749 - 0.042}" />
         <material name="yellow"/>
       </collision>
       <visual name="visual">
         <geometry>
-          <mesh filename="package://abb_irb1200_support/meshes/irb1200_7_70/visual/link_5.stl" scale="0.001 0.001 0.001" />
+          <mesh filename="package://abb_irb1200_support/meshes/irb1200_7_70/visual/link_5.stl" />
         </geometry>
-        <origin xyz="-0.351 0 ${-0.749 - 0.042}" />
         <material name="graphite_white"/>
       </visual>
@@ -102,14 +94,12 @@
       <collision name="collision">
         <geometry>
-          <mesh filename="package://abb_irb1200_support/meshes/irb1200_7_70/collision/link_6.stl" scale="0.001 0.001 0.001" />
+          <mesh filename="package://abb_irb1200_support/meshes/irb1200_7_70/collision/link_6.stl" />
         </geometry>
-        <origin xyz="${-0.351 - 0.082} 0 ${-0.749 - 0.042}" />
         <material name="yellow"/>
       </collision>
       <visual name="visual">
         <geometry>
-          <mesh filename="package://abb_irb1200_support/meshes/irb1200_7_70/visual/link_6.stl" scale="0.001 0.001 0.001" />
+          <mesh filename="package://abb_irb1200_support/meshes/irb1200_7_70/visual/link_6.stl" />
         </geometry>
-        <origin xyz="${-0.351 - 0.082} 0 ${-0.749 - 0.042}" />
         <material name="graphite_white"/>
       </visual>
@@ -119,5 +109,5 @@
     <!-- joint list -->
     <joint type="revolute" name="${prefix}joint_1">
-      <origin xyz="0 0 0" rpy="0 0 0"/>
+      <origin xyz="0 0 0.3991" rpy="0 0 0"/>
       <axis xyz="0 0 1"/>
       <parent link="${prefix}base_link"/>
@@ -126,5 +116,5 @@
     </joint>
     <joint type="revolute" name="${prefix}joint_2">
-      <origin xyz="0 0 0.399" rpy="0 0 0"/>
+      <origin xyz="0 0 0" rpy="0 0 0"/>
       <axis xyz="0 1 0"/>
       <parent link="${prefix}link_1"/>

Commit message: irb1200_7_70: use xacro pi.

File: abb_irb1200_support/urdf/irb1200_7_70_macro.xacro (robot description, xacro)
@@ -153,5 +153,5 @@
       <parent link="${prefix}link_6"/>
       <child link="${prefix}tool0"/>
-      <origin xyz="0 0 0" rpy="0 1.57079632679 0"/>
+      <origin xyz="0 0 0" rpy="0 ${pi/2.0} 0"/>
     </joint>
     <!-- end of joint list -->

Commit message: Add all collada meshes

File: abb_irb1200_support/urdf/irb1200_7_70_macro.xacro (robot description, xacro)
@@ -14,5 +14,6 @@
       <visual name="visual">
         <geometry>
-          <mesh filename="package://abb_irb1200_support/meshes/irb1200_7_70/visual/base_link.stl" />
+	        <!-- reference irb1200_5_90 package since mesh is shared-->
+          <mesh filename="package://abb_irb1200_support/meshes/irb1200_5_90/visual/base_link.dae"  />
         </geometry>
         <material name="graphite_white">
@@ -30,5 +31,6 @@
       <visual name="visual">
         <geometry>
-          <mesh filename="package://abb_irb1200_support/meshes/irb1200_7_70/visual/link_1.stl" />
+	        <!-- reference irb1200_5_90 package since mesh is shared-->
+          <mesh filename="package://abb_irb1200_support/meshes/irb1200_5_90/visual/link_1.dae" />
         </geometry>
         <material name="graphite_white"/>
@@ -44,5 +46,5 @@
       <visual name="visual">
         <geometry>
-          <mesh filename="package://abb_irb1200_support/meshes/irb1200_7_70/visual/link_2.stl" />
+          <mesh filename="package://abb_irb1200_support/meshes/irb1200_7_70/visual/link_2.dae" />
         </geometry>
         <material name="graphite_white"/>
@@ -58,5 +60,5 @@
       <visual name="visual">
         <geometry>
-          <mesh filename="package://abb_irb1200_support/meshes/irb1200_7_70/visual/link_3.stl" />
+          <mesh filename="package://abb_irb1200_support/meshes/irb1200_7_70/visual/link_3.dae" />
         </geometry>
         <material name="graphite_white"/>
@@ -72,5 +74,6 @@
       <visual name="visual">
         <geometry>
-          <mesh filename="package://abb_irb1200_support/meshes/irb1200_7_70/visual/link_4.stl" />
+	        <!-- reference irb1200_5_90 package since mesh is shared-->
+          <mesh filename="package://abb_irb1200_support/meshes/irb1200_7_70/visual/link_4.dae" />
         </geometry>
         <material name="graphite_white"/>
@@ -86,5 +89,6 @@
       <visual name="visual">
         <geometry>
-          <mesh filename="package://abb_irb1200_support/meshes/irb1200_7_70/visual/link_5.stl" />
+	        <!-- reference irb1200_5_90 package since mesh is shared-->
+          <mesh filename="package://abb_irb1200_support/meshes/irb1200_5_90/visual/link_5.dae" />
         </geometry>
         <material name="graphite_white"/>
@@ -100,5 +104,6 @@
       <visual name="visual">
         <geometry>
-          <mesh filename="package://abb_irb1200_support/meshes/irb1200_7_70/visual/link_6.stl" />
+	        <!-- reference irb1200_5_90 package since mesh is shared-->
+          <mesh filename="package://abb_irb1200_support/meshes/irb1200_5_90/visual/link_6.dae" />
         </geometry>
         <material name="graphite_white"/>

Commit message: irb1200_7_70: share even more meshes.
Updated collision meshes to match new visuals.

Reuse link_4 from 5_90 with a small (0.1m) offset in x.

File: abb_irb1200_support/urdf/irb1200_7_70_macro.xacro (robot description, xacro)
@@ -6,5 +6,5 @@
       <collision name="collision">
         <geometry>
-          <mesh filename="package://abb_irb1200_support/meshes/irb1200_7_70/collision/base_link.stl" />
+          <mesh filename="package://abb_irb1200_support/meshes/irb1200_5_90/collision/base_link.stl" />
         </geometry>
         <material name="yellow">
@@ -14,5 +14,4 @@
       <visual name="visual">
         <geometry>
-	        <!-- reference irb1200_5_90 package since mesh is shared-->
           <mesh filename="package://abb_irb1200_support/meshes/irb1200_5_90/visual/base_link.dae"  />
         </geometry>
@@ -25,5 +24,5 @@
       <collision name="collision">
         <geometry>
-          <mesh filename="package://abb_irb1200_support/meshes/irb1200_7_70/collision/link_1.stl" />
+          <mesh filename="package://abb_irb1200_support/meshes/irb1200_5_90/collision/link_1.stl" />
         </geometry>
         <material name="yellow"/>
@@ -31,5 +30,4 @@
       <visual name="visual">
         <geometry>
-	        <!-- reference irb1200_5_90 package since mesh is shared-->
           <mesh filename="package://abb_irb1200_support/meshes/irb1200_5_90/visual/link_1.dae" />
         </geometry>
@@ -67,13 +65,16 @@
     <link name="${prefix}link_4">
       <collision name="collision">
+        <!-- offset purely to allow reuse of meshes -->
+        <origin xyz="-0.1 0 0" rpy="0 0 0"/>
         <geometry>
-          <mesh filename="package://abb_irb1200_support/meshes/irb1200_7_70/collision/link_4.stl" />
+          <mesh filename="package://abb_irb1200_support/meshes/irb1200_5_90/collision/link_4.stl" />
         </geometry>
         <material name="yellow"/>
       </collision>
       <visual name="visual">
+        <!-- offset purely to allow reuse of meshes -->
+        <origin xyz="-0.1 0 0" rpy="0 0 0"/>
         <geometry>
-	        <!-- reference irb1200_5_90 package since mesh is shared-->
-          <mesh filename="package://abb_irb1200_support/meshes/irb1200_7_70/visual/link_4.dae" />
+          <mesh filename="package://abb_irb1200_support/meshes/irb1200_5_90/visual/link_4.dae" />
         </geometry>
         <material name="graphite_white"/>
@@ -83,5 +84,5 @@
       <collision name="collision">
         <geometry>
-          <mesh filename="package://abb_irb1200_support/meshes/irb1200_7_70/collision/link_5.stl" />
+          <mesh filename="package://abb_irb1200_support/meshes/irb1200_5_90/collision/link_5.stl" />
         </geometry>
         <material name="yellow"/>
@@ -89,5 +90,4 @@
       <visual name="visual">
         <geometry>
-	        <!-- reference irb1200_5_90 package since mesh is shared-->
           <mesh filename="package://abb_irb1200_support/meshes/irb1200_5_90/visual/link_5.dae" />
         </geometry>
@@ -98,5 +98,5 @@
       <collision name="collision">
         <geometry>
-          <mesh filename="package://abb_irb1200_support/meshes/irb1200_7_70/collision/link_6.stl" />
+          <mesh filename="package://abb_irb1200_support/meshes/irb1200_5_90/collision/link_6.stl" />
         </geometry>
         <material name="yellow"/>
@@ -104,5 +104,4 @@
       <visual name="visual">
         <geometry>
-	        <!-- reference irb1200_5_90 package since mesh is shared-->
           <mesh filename="package://abb_irb1200_support/meshes/irb1200_5_90/visual/link_6.dae" />
         </geometry>

Commit message: IRB 1200 updates and experimental (MoveIt) support for 7/0.7 variant (#85)
This commit is the result of squashing a range of commits that introduced:

 - support for the 7/0.7 variant of the IRB 1200
 - MoveIt configurations for both the 5/0.9 and the 7/0.7

The range of commits was squashed to prevent repository bloat (due to overly complex and detailed meshes that received numerous edits and saw numerous revisions).

The following people contributed to these updates to the IRB 1200 support in ROS-Industrial:

 - Andrew Short (@ajshort): initial PR and support for 7/0.7 and MoveIt
 - Stephan Wirth (@stwirth): joints update in support pkg
 - Bianca Homberg (@bhomberg): Collada meshes for 7/0.7
 - Jonathan Binney (@jonbinney): fixes to Collada meshes

Squashed commits:

* Add ABB IRB 1200 moveit package
* IRB1200 moveit controllers and execution
* Add IRB1200 7-70 model
* Create IRB1200 7-70 moveit package
* Add IRB1200 7-70 moveit controllers
* Simplify collision models
* Correct reference to launch file
* Correct joint names file reference
* Decouple joint_names_irb1200.yaml for both robot variants.
* irb1200_support: be explicit about which variants are supported exactly.
* irb1200_support: refer to ABB doc ID.
* irb1200_7_70: fix mesh origins, scaling and normals.
* irb1200_7_70: use xacro pi.
* irb1200_7_70: subsample meshes.
* irb1200_moveit_cfg: make RRTConnect the default planner.
* irb1200_moveit_cfg: use standardised 'all_zero' name for all-zeros home pos.
* irb1200_moveit_cfg: fixup moveit_planning_execution launch file.
* irb1200_moveit_cfg: fixup package manifests.
* irb1200_moveit_cfg: use a more sane default RViz config.
* irb1200_moveit_cfg: use Trac IK as default IK plugin.
* irb1200_5_90: use xacro pi.
* Add all collada meshes
* irb1200_7_70: share even more meshes.
* irb1200: set yellow material on collision geometry.

File: abb_irb1200_support/urdf/irb1200_7_70_macro.xacro (robot description, xacro)
@@ -2,15 +2,15 @@
 <robot xmlns:xacro="http://ros.org/wiki/xacro">
   <xacro:include filename="$(find abb_resources)/urdf/common_materials.xacro"/>
-  <xacro:macro name="abb_irb1200_5_90" params="prefix">
+  <xacro:macro name="abb_irb1200_7_70" params="prefix">
     <!-- link list -->
     <link name="${prefix}base_link">
       <collision name="collision">
         <geometry>
-          <mesh filename="package://abb_irb1200_support/meshes/irb1200_5_90/collision/base_link.stl"/>
+          <mesh filename="package://abb_irb1200_support/meshes/irb1200_5_90/collision/base_link.stl" />
         </geometry>
       </collision>
       <visual name="visual">
         <geometry>
-          <mesh filename="package://abb_irb1200_support/meshes/irb1200_5_90/visual/base_link.dae"/>
+          <mesh filename="package://abb_irb1200_support/meshes/irb1200_5_90/visual/base_link.dae"  />
         </geometry>
         <xacro:material_abb_yellow />
@@ -20,10 +20,10 @@
       <collision name="collision">
         <geometry>
-          <mesh filename="package://abb_irb1200_support/meshes/irb1200_5_90/collision/link_1.stl"/>
+          <mesh filename="package://abb_irb1200_support/meshes/irb1200_5_90/collision/link_1.stl" />
         </geometry>
       </collision>
       <visual name="visual">
         <geometry>
-          <mesh filename="package://abb_irb1200_support/meshes/irb1200_5_90/visual/link_1.dae"/>
+          <mesh filename="package://abb_irb1200_support/meshes/irb1200_5_90/visual/link_1.dae" />
         </geometry>
         <xacro:material_abb_yellow />
@@ -33,10 +33,10 @@
       <collision name="collision">
         <geometry>
-          <mesh filename="package://abb_irb1200_support/meshes/irb1200_5_90/collision/link_2.stl"/>
+          <mesh filename="package://abb_irb1200_support/meshes/irb1200_7_70/collision/link_2.stl" />
         </geometry>
       </collision>
       <visual name="visual">
         <geometry>
-          <mesh filename="package://abb_irb1200_support/meshes/irb1200_5_90/visual/link_2.dae"/>
+          <mesh filename="package://abb_irb1200_support/meshes/irb1200_7_70/visual/link_2.dae" />
         </geometry>
         <xacro:material_abb_yellow />
@@ -44,12 +44,12 @@
     </link>
     <link name="${prefix}link_3">
-      <collision name="collision">
+      <collision name="graphite_white">
         <geometry>
-          <mesh filename="package://abb_irb1200_support/meshes/irb1200_5_90/collision/link_3.stl"/>
+          <mesh filename="package://abb_irb1200_support/meshes/irb1200_7_70/collision/link_3.stl" />
         </geometry>
       </collision>
       <visual name="visual">
         <geometry>
-          <mesh filename="package://abb_irb1200_support/meshes/irb1200_5_90/visual/link_3.dae"/>
+          <mesh filename="package://abb_irb1200_support/meshes/irb1200_7_70/visual/link_3.dae" />
         </geometry>
         <xacro:material_abb_yellow />
@@ -58,11 +58,15 @@
     <link name="${prefix}link_4">
       <collision name="collision">
+        <!-- offset purely to allow reuse of meshes -->
+        <origin xyz="-0.1 0 0" rpy="0 0 0"/>
         <geometry>
-          <mesh filename="package://abb_irb1200_support/meshes/irb1200_5_90/collision/link_4.stl"/>
+          <mesh filename="package://abb_irb1200_support/meshes/irb1200_5_90/collision/link_4.stl" />
         </geometry>
       </collision>
       <visual name="visual">
+        <!-- offset purely to allow reuse of meshes -->
+        <origin xyz="-0.1 0 0" rpy="0 0 0"/>
         <geometry>
-          <mesh filename="package://abb_irb1200_support/meshes/irb1200_5_90/visual/link_4.dae"/>
+          <mesh filename="package://abb_irb1200_support/meshes/irb1200_5_90/visual/link_4.dae" />
         </geometry>
         <xacro:material_abb_yellow />
@@ -72,10 +76,10 @@
       <collision name="collision">
         <geometry>
-          <mesh filename="package://abb_irb1200_support/meshes/irb1200_5_90/collision/link_5.stl"/>
+          <mesh filename="package://abb_irb1200_support/meshes/irb1200_5_90/collision/link_5.stl" />
         </geometry>
       </collision>
       <visual name="visual">
         <geometry>
-          <mesh filename="package://abb_irb1200_support/meshes/irb1200_5_90/visual/link_5.dae"/>
+          <mesh filename="package://abb_irb1200_support/meshes/irb1200_5_90/visual/link_5.dae" />
         </geometry>
         <xacro:material_abb_yellow />
@@ -85,10 +89,10 @@
       <collision name="collision">
         <geometry>
-          <mesh filename="package://abb_irb1200_support/meshes/irb1200_5_90/collision/link_6.stl"/>
+          <mesh filename="package://abb_irb1200_support/meshes/irb1200_5_90/collision/link_6.stl" />
         </geometry>
       </collision>
       <visual name="visual">
         <geometry>
-          <mesh filename="package://abb_irb1200_support/meshes/irb1200_5_90/visual/link_6.dae"/>
+          <mesh filename="package://abb_irb1200_support/meshes/irb1200_5_90/visual/link_6.dae" />
         </geometry>
         <xacro:material_abb_yellow />
@@ -110,8 +114,8 @@
       <parent link="${prefix}link_1"/>
       <child link="${prefix}link_2"/>
-      <limit effort="0" lower="-1.745" upper="2.269" velocity="4.189"/>
+      <limit effort="0" lower="-1.745" upper="2.356" velocity="4.189"/>
     </joint>
     <joint type="revolute" name="${prefix}joint_3">
-      <origin xyz="0 0 0.448" rpy="0 0 0"/>
+      <origin xyz="0 0 0.350" rpy="0 0 0"/>
       <axis xyz="0 1 0"/>
       <parent link="${prefix}link_2"/>
@@ -127,5 +131,5 @@
     </joint>
     <joint type="revolute" name="${prefix}joint_5">
-      <origin xyz="0.451 0 0" rpy="0 0 0"/>
+      <origin xyz="0.351 0 0 " rpy="0 0 0"/>
       <axis xyz="0 1 0"/>
       <parent link="${prefix}link_4"/>
@@ -134,5 +138,5 @@
     </joint>
     <joint type="revolute" name="${prefix}joint_6">
-      <origin xyz="0.082 0 0" rpy="0 0 0"/>
+      <origin xyz="0.082 0 0 " rpy="0 0 0"/>
       <axis xyz="1 0 0"/>
       <parent link="${prefix}link_5"/>
