Commit message: irb1200_5_90: use xacro pi.

File: abb_irb1200_support/urdf/irb1200_5_90_macro.xacro (robot description, xacro)
@@ -128,5 +128,5 @@
     </joint>
     <joint type="revolute" name="${prefix}joint_5">
-      <origin xyz="0.451 0 0 " rpy="0 0 0"/>
+      <origin xyz="0.451 0 0" rpy="0 0 0"/>
       <axis xyz="0 1 0"/>
       <parent link="${prefix}link_4"/>
@@ -135,5 +135,5 @@
     </joint>
     <joint type="revolute" name="${prefix}joint_6">
-      <origin xyz="0.082 0 0 " rpy="0 0 0"/>
+      <origin xyz="0.082 0 0" rpy="0 0 0"/>
       <axis xyz="1 0 0"/>
       <parent link="${prefix}link_5"/>
@@ -144,5 +144,5 @@
       <parent link="${prefix}link_6"/>
       <child link="${prefix}tool0"/>
-      <origin xyz="0 0 0" rpy="0 1.57079632679 0"/>
+      <origin xyz="0 0 0" rpy="0 ${pi/2.0} 0"/>
     </joint>
     <!-- end of joint list -->

Commit message: irb1200_5_90: fix base_link->link_1 transform. Fix #82.
Docs (3HAC046982-001, rev. G) spec a 0.3991m translation in Z direction, while
xacro had it at 0.399m.

File: abb_irb1200_support/urdf/irb1200_5_90_macro.xacro (robot description, xacro)
@@ -100,5 +100,5 @@
     <!-- joint list -->
     <joint type="revolute" name="${prefix}joint_1">
-      <origin xyz="0 0 0" rpy="0 0 0"/>
+      <origin xyz="0 0 0.3991" rpy="0 0 0"/>
       <axis xyz="0 0 1"/>
       <parent link="${prefix}base_link"/>
@@ -107,5 +107,5 @@
     </joint>
     <joint type="revolute" name="${prefix}joint_2">
-      <origin xyz="0 0 0.399" rpy="0 0 0"/>
+      <origin xyz="0 0 0" rpy="0 0 0"/>
       <axis xyz="0 1 0"/>
       <parent link="${prefix}link_1"/>

Commit message: irb1200: set yellow material on collision geometry.
More in-line with other support packages.

File: abb_irb1200_support/urdf/irb1200_5_90_macro.xacro (robot description, xacro)
@@ -1,4 +1,5 @@
 <?xml version="1.0"?>
 <robot xmlns:xacro="http://ros.org/wiki/xacro">
+  <xacro:include filename="$(find abb_resources)/urdf/common_materials.xacro"/>
   <xacro:macro name="abb_irb1200_5_90" params="prefix">
     <!-- link list -->
@@ -13,7 +14,5 @@
           <mesh filename="package://abb_irb1200_support/meshes/irb1200_5_90/visual/base_link.dae"/>
         </geometry>
-        <material name="yellow">
-          <color rgba="1 1 0 1"/>
-        </material>
+        <xacro:material_abb_yellow />
       </visual>
     </link>
@@ -28,5 +27,5 @@
           <mesh filename="package://abb_irb1200_support/meshes/irb1200_5_90/visual/link_1.dae"/>
         </geometry>
-        <material name="yellow"/>
+        <xacro:material_abb_yellow />
       </visual>
     </link>
@@ -41,5 +40,5 @@
           <mesh filename="package://abb_irb1200_support/meshes/irb1200_5_90/visual/link_2.dae"/>
         </geometry>
-        <material name="yellow"/>
+        <xacro:material_abb_yellow />
       </visual>
     </link>
@@ -54,5 +53,5 @@
           <mesh filename="package://abb_irb1200_support/meshes/irb1200_5_90/visual/link_3.dae"/>
         </geometry>
-        <material name="yellow"/>
+        <xacro:material_abb_yellow />
       </visual>
     </link>
@@ -67,5 +66,5 @@
           <mesh filename="package://abb_irb1200_support/meshes/irb1200_5_90/visual/link_4.dae"/>
         </geometry>
-        <material name="yellow"/>
+        <xacro:material_abb_yellow />
       </visual>
     </link>
@@ -80,5 +79,5 @@
           <mesh filename="package://abb_irb1200_support/meshes/irb1200_5_90/visual/link_5.dae"/>
         </geometry>
-        <material name="yellow"/>
+        <xacro:material_abb_yellow />
       </visual>
     </link>
@@ -93,5 +92,5 @@
           <mesh filename="package://abb_irb1200_support/meshes/irb1200_5_90/visual/link_6.dae"/>
         </geometry>
-        <material name="yellow"/>
+        <xacro:material_abb_yellow />
       </visual>
     </link>

File: abb_irb1200_support/urdf/irb1200_7_70_macro.xacro (robot description, xacro)
@@ -1,4 +1,5 @@
 <?xml version="1.0"?>
 <robot xmlns:xacro="http://ros.org/wiki/xacro">
+  <xacro:include filename="$(find abb_resources)/urdf/common_materials.xacro"/>
   <xacro:macro name="abb_irb1200_7_70" params="prefix">
     <!-- link list -->
@@ -8,7 +9,4 @@
           <mesh filename="package://abb_irb1200_support/meshes/irb1200_5_90/collision/base_link.stl" />
         </geometry>
-        <material name="yellow">
-          <color rgba="1 1 0 1"/>
-        </material>
       </collision>
       <visual name="visual">
@@ -16,7 +14,5 @@
           <mesh filename="package://abb_irb1200_support/meshes/irb1200_5_90/visual/base_link.dae"  />
         </geometry>
-        <material name="graphite_white">
-          <color rgba="0.9 0.9 0.9 1"/>
-        </material>
+        <xacro:material_abb_yellow />
       </visual>
     </link>
@@ -26,5 +22,4 @@
           <mesh filename="package://abb_irb1200_support/meshes/irb1200_5_90/collision/link_1.stl" />
         </geometry>
-        <material name="yellow"/>
       </collision>
       <visual name="visual">
@@ -32,5 +27,5 @@
           <mesh filename="package://abb_irb1200_support/meshes/irb1200_5_90/visual/link_1.dae" />
         </geometry>
-        <material name="graphite_white"/>
+        <xacro:material_abb_yellow />
       </visual>
     </link>
@@ -40,5 +35,4 @@
           <mesh filename="package://abb_irb1200_support/meshes/irb1200_7_70/collision/link_2.stl" />
         </geometry>
-        <material name="yellow"/>
       </collision>
       <visual name="visual">
@@ -46,5 +40,5 @@
           <mesh filename="package://abb_irb1200_support/meshes/irb1200_7_70/visual/link_2.dae" />
         </geometry>
-        <material name="graphite_white"/>
+        <xacro:material_abb_yellow />
       </visual>
     </link>
@@ -54,5 +48,4 @@
           <mesh filename="package://abb_irb1200_support/meshes/irb1200_7_70/collision/link_3.stl" />
         </geometry>
-        <material name="yellow"/>
       </collision>
       <visual name="visual">
@@ -60,5 +53,5 @@
           <mesh filename="package://abb_irb1200_support/meshes/irb1200_7_70/visual/link_3.dae" />
         </geometry>
-        <material name="graphite_white"/>
+        <xacro:material_abb_yellow />
       </visual>
     </link>
@@ -70,5 +63,4 @@
           <mesh filename="package://abb_irb1200_support/meshes/irb1200_5_90/collision/link_4.stl" />
         </geometry>
-        <material name="yellow"/>
       </collision>
       <visual name="visual">
@@ -78,5 +70,5 @@
           <mesh filename="package://abb_irb1200_support/meshes/irb1200_5_90/visual/link_4.dae" />
         </geometry>
-        <material name="graphite_white"/>
+        <xacro:material_abb_yellow />
       </visual>
     </link>
@@ -86,5 +78,4 @@
           <mesh filename="package://abb_irb1200_support/meshes/irb1200_5_90/collision/link_5.stl" />
         </geometry>
-        <material name="yellow"/>
       </collision>
       <visual name="visual">
@@ -92,5 +83,5 @@
           <mesh filename="package://abb_irb1200_support/meshes/irb1200_5_90/visual/link_5.dae" />
         </geometry>
-        <material name="graphite_white"/>
+        <xacro:material_abb_yellow />
       </visual>
     </link>
@@ -100,5 +91,4 @@
           <mesh filename="package://abb_irb1200_support/meshes/irb1200_5_90/collision/link_6.stl" />
         </geometry>
-        <material name="yellow"/>
       </collision>
       <visual name="visual">
@@ -106,5 +96,5 @@
           <mesh filename="package://abb_irb1200_support/meshes/irb1200_5_90/visual/link_6.dae" />
         </geometry>
-        <material name="graphite_white"/>
+        <xacro:material_abb_yellow />
       </visual>
     </link>

Commit message: Gazebo support for irb1200_5_90

File: abb_irb1200_support/urdf/irb1200_5_90_macro.xacro (robot description, xacro)
@@ -5,4 +5,9 @@
     <!-- link list -->
     <link name="${prefix}base_link">
+      <inertial>
+        <mass value="6.215"/>
+        <origin xyz="-0.04204 8.01E-05 0.07964" rpy="0 0 0"/>
+        <inertia ixx="0.0247272" ixy="-8.0784E-05" ixz="0.00130902" iyy="0.0491285" iyz="-8.0419E-06" izz="0.0472376"/>
+      </inertial>
       <collision name="collision">
         <geometry>
@@ -18,4 +23,9 @@
     </link>
     <link name="${prefix}link_1">
+      <inertial>
+        <mass value="3.067" />
+        <origin xyz="9.77E-05 -0.00012 0.23841" rpy="0 0 0"/>
+        <inertia ixx="0.0142175" ixy="-1.28579E-05" ixz="-2.31364E-05" iyy="0.0144041" iyz="1.93404E-05" izz="0.0104533"/>
+      </inertial>
       <collision name="collision">
         <geometry>
@@ -31,4 +41,9 @@
     </link>
     <link name="${prefix}link_2">
+      <inertial>
+        <mass value="3.909"/>
+        <origin xyz="0.00078 -0.00212 0.10124" rpy="0 0 0"/>
+        <inertia ixx="0.0603111" ixy="9.83431E-06" ixz="5.72407E-05" iyy="0.041569" iyz="-0.00050497" izz="0.0259548"/>
+      </inertial>
       <collision name="collision">
         <geometry>
@@ -44,4 +59,9 @@
     </link>
     <link name="${prefix}link_3">
+      <inertial>
+        <mass value="2.944"/>
+        <origin xyz="0.02281 0.00106 0.05791" rpy="0 0 0"/>
+        <inertia ixx="0.00835606" ixy="-8.01545E-05" ixz="0.00142884" iyy="0.016713" iyz="-0.000182227" izz="0.0126984"/>
+      </inertial>
       <collision name="collision">
         <geometry>
@@ -57,4 +77,9 @@
     </link>
     <link name="${prefix}link_4">
+      <inertial>
+        <mass value="1.328"/>
+        <origin xyz="0.2247 0.00015 0.00041" rpy="0 0 0"/>
+        <inertia ixx="0.00284661" ixy="-2.12765E-05" ixz="-1.6435E-05" iyy="0.00401346" iyz="1.31336E-05" izz="0.0052535"/>
+      </inertial>
       <collision name="collision">
         <geometry>
@@ -70,4 +95,9 @@
     </link>
     <link name="${prefix}link_5">
+      <inertial>
+        <mass value="0.546"/>
+        <origin xyz="-0.00109 3.68E-05 6.22E-05" rpy="0 0 0"/>
+        <inertia ixx="0.000404891" ixy="1.61943E-06" ixz="8.46805E-07" iyy="0.000892825" iyz="-1.51792E-08" izz="0.000815468"/>
+      </inertial>
       <collision name="collision">
         <geometry>
@@ -83,4 +113,9 @@
     </link>
     <link name="${prefix}link_6">
+      <inertial>
+        <mass value="0.137"/>
+        <origin xyz="-0.00706 -0.00017 -1.32E-06" rpy="0 0 0"/>
+        <inertia ixx="0.001" ixy="0" ixz="0" iyy="0.001" iyz="0" izz="0.001"/>
+      </inertial>
       <collision name="collision">
         <geometry>

Commit message: Add gazebo support for IRB1200 5/90 variant
* Adds inertial values to abb_irb1200_support irb1200_5_90 xacro file
* Adds the irb1200_gazebo package with support for the 5 90 variant
using effort controllers.

This is built upon the initial work of @stwirth
(https://github.com/ros-industrial/abb_experimental/pull/98) and
@jonbinnie.

File: abb_irb1200_support/urdf/irb1200_5_90_macro.xacro (robot description, xacro)
@@ -5,4 +5,9 @@
     <!-- link list -->
     <link name="${prefix}base_link">
+      <inertial>
+        <mass value="13.7742"/>
+        <origin xyz="-0.028986 0.000596 0.11273"/>
+        <inertia ixx="0.101998" ixy="0.000495482" ixz="0.000311158" iyy="0.13969" iyz="-0.000245375" izz="0.130433"/>
+      </inertial>
       <collision name="collision">
         <geometry>
@@ -18,4 +23,9 @@
     </link>
     <link name="${prefix}link_1">
+      <inertial>
+        <mass value="11.8419"/>
+        <origin xyz="0.000877 -0.000631 -0.062883"/>
+        <inertia ixx="0.11194" ixy="-4.54988e-05" ixz="0.000280961" iyy="0.0915159" iyz="-0.000109905" izz="0.0876456"/>
+      </inertial>
       <collision name="collision">
         <geometry>
@@ -31,4 +41,9 @@
     </link>
     <link name="${prefix}link_2">
+      <inertial>
+        <mass value="17.5394"/>
+        <origin xyz="-0.000928 -0.000497 0.250051"/>
+        <inertia ixx="0.493558" ixy="1.32136e-05" ixz="0.000209024" iyy="0.462939" iyz="-0.00179901" izz="0.0894214"/>
+      </inertial>
       <collision name="collision">
         <geometry>
@@ -44,4 +59,9 @@
     </link>
     <link name="${prefix}link_3">
+      <inertial>
+        <mass value="7.46365"/>
+        <origin xyz="0.099588 0.001143 0.032333"/>
+        <inertia ixx="0.0252424" ixy="0.000142737" ixz="-0.00565542" iyy="0.0906438" iyz="0.000142213" izz="0.0825079"/>
+      </inertial>
       <collision name="collision">
         <geometry>
@@ -57,4 +77,9 @@
     </link>
     <link name="${prefix}link_4">
+      <inertial>
+        <mass value="2.74436"/>
+        <origin xyz="0.381678 0.001261 0.005168"/>
+        <inertia ixx="0.00573099" ixy="-0.000131119" ixz="0.000380232" iyy="0.0118352" iyz="-2.26565e-05" izz="0.0114428"/>
+      </inertial>
       <collision name="collision">
         <geometry>
@@ -70,4 +95,9 @@
     </link>
     <link name="${prefix}link_5">
+      <inertial>
+        <mass value="0.62953"/>
+        <origin xyz="0.011197 -0.001056 0.000109"/>
+        <inertia ixx="0.000502815" ixy="-1.03173e-05" ixz="-8.74347e-08" iyy="0.00108856" iyz="2.07657e-07" izz="0.000918873"/>
+      </inertial>
       <collision name="collision">
         <geometry>
@@ -83,4 +113,15 @@
     </link>
     <link name="${prefix}link_6">
+      <inertial>
+        <mass value="0.137"/>
+        <origin xyz="-0.00706 -0.00017 -1.32E-06" rpy="0 0 0"/>
+        <inertia ixx="0.001" ixy="0" ixz="0" iyy="0.001" iyz="0" izz="0.001"/>
+      </inertial>
+      <!-- Meshlab calculated values (below) make gazebo crash when rotating this joint. -->
+      <!-- <inertial>
+        <mass value="0.00686711"/>
+        <origin xyz="-0.00250976 -1.89e-06 0.00010218"/>
+        <inertia ixx="1.3517e-06" ixy="-1.21316e-11" ixz="9.18065e-12" iyy="6.89813e-07" iyz="-1.21534e-10" izz="6.90097e-07"/>
+      </inertial> -->
       <collision name="collision">
         <geometry>
@@ -103,5 +144,6 @@
       <parent link="${prefix}base_link"/>
       <child link="${prefix}link_1"/>
-      <limit effort="0" lower="-2.967" upper="2.967" velocity="5.027"/>
+      <limit effort="1000" lower="-2.967" upper="2.967" velocity="5.027"/>
+      <dynamics damping="50.0" friction="1.0"/>
     </joint>
     <joint type="revolute" name="${prefix}joint_2">
@@ -110,5 +152,6 @@
       <parent link="${prefix}link_1"/>
       <child link="${prefix}link_2"/>
-      <limit effort="0" lower="-1.745" upper="2.269" velocity="4.189"/>
+      <limit effort="1000" lower="-1.745" upper="2.269" velocity="4.189"/>
+      <dynamics damping="50.0" friction="1.0"/>
     </joint>
     <joint type="revolute" name="${prefix}joint_3">
@@ -117,5 +160,6 @@
       <parent link="${prefix}link_2"/>
       <child link="${prefix}link_3"/>
-      <limit effort="0" lower="-3.491" upper="1.222" velocity="5.236"/>
+      <limit effort="1000" lower="-3.491" upper="1.222" velocity="5.236"/>
+      <dynamics damping="10.0" friction="1.0"/>
     </joint>
     <joint type="revolute" name="${prefix}joint_4">
@@ -124,5 +168,6 @@
       <parent link="${prefix}link_3"/>
       <child link="${prefix}link_4"/>
-      <limit effort="0" lower="-4.712" upper="4.712" velocity="6.981"/>
+      <limit effort="1000" lower="-4.712" upper="4.712" velocity="6.981"/>
+      <dynamics damping="5.0" friction="1.0"/>
     </joint>
     <joint type="revolute" name="${prefix}joint_5">
@@ -131,5 +176,6 @@
       <parent link="${prefix}link_4"/>
       <child link="${prefix}link_5"/>
-      <limit effort="0" lower="-2.269" upper="2.269" velocity="7.069"/>
+      <limit effort="1000" lower="-2.269" upper="2.269" velocity="7.069"/>
+      <dynamics damping="2.0" friction="1.0"/>
     </joint>
     <joint type="revolute" name="${prefix}joint_6">
@@ -138,5 +184,6 @@
       <parent link="${prefix}link_5"/>
       <child link="${prefix}link_6"/>
-      <limit effort="0" lower="-6.283" upper="6.283" velocity="10.472"/>
+      <limit effort="1000" lower="-6.283" upper="6.283" velocity="10.472"/>
+      <dynamics damping="1.0" friction="1.0"/>
     </joint>
     <joint type="fixed" name="${prefix}joint_6-tool0">

Commit message: Add gazebo support for IRB1200 5/90 variant (#110)
Squashed commits:

* Add gazebo support for IRB1200 5/90 variant
* Adds inertial values to abb_irb1200_support irb1200_5_90 xacro file
* Adds the irb1200_gazebo package with support for the 5 90 variant using effort controllers.
  This is built upon the initial work of @stwirth (#98) and @jonbinnie.

* Re-arrange abb_irb1200 xacros
* Document how the values were obtained
* irb1200: clarify where inertial, dynamics and effort values came from.
* irb1200_gazebo: update gazebo pkg manifest.
* irb1200_gazebo: don't depend on metapackages.

File: abb_irb1200_support/urdf/irb1200_5_90_macro.xacro (robot description, xacro)
@@ -5,4 +5,10 @@
     <!-- link list -->
     <link name="${prefix}base_link">
+      <!-- See note 1 in package.xml about the inertial and mass values -->
+      <inertial>
+        <mass value="13.7742"/>
+        <origin xyz="-0.028986 0.000596 0.11273"/>
+        <inertia ixx="0.101998" ixy="0.000495482" ixz="0.000311158" iyy="0.13969" iyz="-0.000245375" izz="0.130433"/>
+      </inertial>
       <collision name="collision">
         <geometry>
@@ -18,4 +24,10 @@
     </link>
     <link name="${prefix}link_1">
+      <!-- See note 1 in package.xml about the inertial and mass values -->
+      <inertial>
+        <mass value="11.8419"/>
+        <origin xyz="0.000877 -0.000631 -0.062883"/>
+        <inertia ixx="0.11194" ixy="-4.54988e-05" ixz="0.000280961" iyy="0.0915159" iyz="-0.000109905" izz="0.0876456"/>
+      </inertial>
       <collision name="collision">
         <geometry>
@@ -31,4 +43,10 @@
     </link>
     <link name="${prefix}link_2">
+      <!-- See note 1 in package.xml about the inertial and mass values -->
+      <inertial>
+        <mass value="17.5394"/>
+        <origin xyz="-0.000928 -0.000497 0.250051"/>
+        <inertia ixx="0.493558" ixy="1.32136e-05" ixz="0.000209024" iyy="0.462939" iyz="-0.00179901" izz="0.0894214"/>
+      </inertial>
       <collision name="collision">
         <geometry>
@@ -44,4 +62,10 @@
     </link>
     <link name="${prefix}link_3">
+      <!-- See note 1 in package.xml about the inertial and mass values -->
+      <inertial>
+        <mass value="7.46365"/>
+        <origin xyz="0.099588 0.001143 0.032333"/>
+        <inertia ixx="0.0252424" ixy="0.000142737" ixz="-0.00565542" iyy="0.0906438" iyz="0.000142213" izz="0.0825079"/>
+      </inertial>
       <collision name="collision">
         <geometry>
@@ -57,4 +81,10 @@
     </link>
     <link name="${prefix}link_4">
+      <!-- See note 1 in package.xml about the inertial and mass values -->
+      <inertial>
+        <mass value="2.74436"/>
+        <origin xyz="0.381678 0.001261 0.005168"/>
+        <inertia ixx="0.00573099" ixy="-0.000131119" ixz="0.000380232" iyy="0.0118352" iyz="-2.26565e-05" izz="0.0114428"/>
+      </inertial>
       <collision name="collision">
         <geometry>
@@ -70,4 +100,10 @@
     </link>
     <link name="${prefix}link_5">
+      <!-- See note 1 in package.xml about the inertial and mass values -->
+      <inertial>
+        <mass value="0.62953"/>
+        <origin xyz="0.011197 -0.001056 0.000109"/>
+        <inertia ixx="0.000502815" ixy="-1.03173e-05" ixz="-8.74347e-08" iyy="0.00108856" iyz="2.07657e-07" izz="0.000918873"/>
+      </inertial>
       <collision name="collision">
         <geometry>
@@ -83,4 +119,16 @@
     </link>
     <link name="${prefix}link_6">
+      <!-- See note 1 in package.xml about the inertial and mass values -->
+      <inertial>
+        <mass value="0.137"/>
+        <origin xyz="-0.00706 -0.00017 -1.32E-06" rpy="0 0 0"/>
+        <inertia ixx="0.001" ixy="0" ixz="0" iyy="0.001" iyz="0" izz="0.001"/>
+      </inertial>
+      <!-- Meshlab calculated values (below) make gazebo crash when rotating this joint. -->
+      <!-- <inertial>
+        <mass value="0.00686711"/>
+        <origin xyz="-0.00250976 -1.89e-06 0.00010218"/>
+        <inertia ixx="1.3517e-06" ixy="-1.21316e-11" ixz="9.18065e-12" iyy="6.89813e-07" iyz="-1.21534e-10" izz="6.90097e-07"/>
+      </inertial> -->
       <collision name="collision">
         <geometry>
@@ -103,5 +151,7 @@
       <parent link="${prefix}base_link"/>
       <child link="${prefix}link_1"/>
-      <limit effort="0" lower="-2.967" upper="2.967" velocity="5.027"/>
+      <!-- See note 2 in package.xml about effort limits and dynamics values -->
+      <limit effort="1000" lower="-2.967" upper="2.967" velocity="5.027"/>
+      <dynamics damping="50.0" friction="1.0"/>
     </joint>
     <joint type="revolute" name="${prefix}joint_2">
@@ -110,5 +160,7 @@
       <parent link="${prefix}link_1"/>
       <child link="${prefix}link_2"/>
-      <limit effort="0" lower="-1.745" upper="2.269" velocity="4.189"/>
+      <!-- See note 2 in package.xml about effort limits and dynamics values -->
+      <limit effort="1000" lower="-1.745" upper="2.269" velocity="4.189"/>
+      <dynamics damping="50.0" friction="1.0"/>
     </joint>
     <joint type="revolute" name="${prefix}joint_3">
@@ -117,5 +169,7 @@
       <parent link="${prefix}link_2"/>
       <child link="${prefix}link_3"/>
-      <limit effort="0" lower="-3.491" upper="1.222" velocity="5.236"/>
+      <!-- See note 2 in package.xml about effort limits and dynamics values -->
+      <limit effort="1000" lower="-3.491" upper="1.222" velocity="5.236"/>
+      <dynamics damping="10.0" friction="1.0"/>
     </joint>
     <joint type="revolute" name="${prefix}joint_4">
@@ -124,5 +178,7 @@
       <parent link="${prefix}link_3"/>
       <child link="${prefix}link_4"/>
-      <limit effort="0" lower="-4.712" upper="4.712" velocity="6.981"/>
+      <!-- See note 2 in package.xml about effort limits and dynamics values -->
+      <limit effort="1000" lower="-4.712" upper="4.712" velocity="6.981"/>
+      <dynamics damping="5.0" friction="1.0"/>
     </joint>
     <joint type="revolute" name="${prefix}joint_5">
@@ -131,5 +187,7 @@
       <parent link="${prefix}link_4"/>
       <child link="${prefix}link_5"/>
-      <limit effort="0" lower="-2.269" upper="2.269" velocity="7.069"/>
+      <!-- See note 2 in package.xml about effort limits and dynamics values -->
+      <limit effort="1000" lower="-2.269" upper="2.269" velocity="7.069"/>
+      <dynamics damping="2.0" friction="1.0"/>
     </joint>
     <joint type="revolute" name="${prefix}joint_6">
@@ -138,5 +196,7 @@
       <parent link="${prefix}link_5"/>
       <child link="${prefix}link_6"/>
-      <limit effort="0" lower="-6.283" upper="6.283" velocity="10.472"/>
+      <!-- See note 2 in package.xml about effort limits and dynamics values -->
+      <limit effort="1000" lower="-6.283" upper="6.283" velocity="10.472"/>
+      <dynamics damping="1.0" friction="1.0"/>
     </joint>
     <joint type="fixed" name="${prefix}joint_6-tool0">
