Commit message: adjusted some joints to accomodate the shorter links lengths of the 20 kg model

File: abb_irb4600_support/urdf/irb4600_20_250.xacro (robot description, xacro)
@@ -1,6 +1,5 @@
 <?xml version="1.0" ?>
 <robot name="abb_irb4600_20_250" xmlns:xacro="http://ros.org/wiki/xacro">
-  <xacro:include filename="$(find abb_irb4600_support)/urdf/irb4600_20_250
-_macro.xacro"/>
-  <xacro:abb_irb4600_40_255 prefix=""/>
+  <xacro:include filename="$(find abb_irb4600_support)/urdf/irb4600_20_250_macro.xacro"/>
+  <xacro:abb_irb4600_20_250 prefix=""/>
 </robot>

File: abb_irb4600_support/urdf/irb4600_20_250_macro.xacro (robot description, xacro)
@@ -143,5 +143,5 @@
     </joint>
     <joint type="revolute" name="${prefix}joint_5">
-      <origin xyz="0.960 0 0 " rpy="0 0 0"/>
+      <origin xyz="0.900 0 0 " rpy="0 0 0"/>
       <axis xyz="0 1 0"/>
       <parent link="${prefix}link_4"/>
@@ -150,5 +150,5 @@
     </joint>
     <joint type="revolute" name="${prefix}joint_6">
-      <origin xyz="0.135 0 0 " rpy="0 0 0"/>
+      <origin xyz="0.085 0 0 " rpy="0 0 0"/>
       <axis xyz="1 0 0"/>
       <parent link="${prefix}link_5"/>
