Commit message: updated transform between link3 and link4

File: abb_irb4600_support/urdf/irb4600_40_255_macro.xacro (robot description, xacro)
@@ -136,5 +136,5 @@
     </joint>
     <joint type="revolute" name="${prefix}joint_4">
-      <origin xyz="0 0 0.175" rpy="0 0 0"/>
+      <origin xyz="0.33 0 0.175" rpy="0 0 0"/>
       <axis xyz="1 0 0"/>
       <parent link="${prefix}link_3"/>

Commit message: replaced all radian axis limit values to degrees with a conversion to follow (new) ros convention

File: abb_irb4600_support/urdf/irb4600_40_255_macro.xacro (robot description, xacro)
@@ -119,5 +119,5 @@
       <parent link="${prefix}base_link"/>
       <child link="${prefix}link_1"/>
-      <limit effort="0" lower="-3.141" upper="3.141" velocity="3.054"/>
+      <limit effort="0" lower="${radians(-180)}" upper="${radians(180)}" velocity="3.054"/>
     </joint>
     <joint type="revolute" name="${prefix}joint_2">
@@ -126,5 +126,5 @@
       <parent link="${prefix}link_1"/>
       <child link="${prefix}link_2"/>
-      <limit effort="0" lower="-1.570" upper="2.617" velocity="3.054"/>
+      <limit effort="0" lower="${radians(-90)}" upper="${radians(150)}" velocity="3.054"/>
     </joint>
     <joint type="revolute" name="${prefix}joint_3">
@@ -133,5 +133,5 @@
       <parent link="${prefix}link_2"/>
       <child link="${prefix}link_3"/>
-      <limit effort="0" lower="-3.141" upper="1.308" velocity="3.054"/>
+      <limit effort="0" lower="${radians(-180)}" upper="${radians(75)}" velocity="3.054"/>
     </joint>
     <joint type="revolute" name="${prefix}joint_4">
@@ -140,5 +140,5 @@
       <parent link="${prefix}link_3"/>
       <child link="${prefix}link_4"/>
-      <limit effort="0" lower="-6.981" upper="6.981" velocity="4.363"/>
+      <limit effort="0" lower="${radians(-400)}" upper="${radians(400)}" velocity="4.363"/>
     </joint>
     <joint type="revolute" name="${prefix}joint_5">
@@ -147,5 +147,5 @@
       <parent link="${prefix}link_4"/>
       <child link="${prefix}link_5"/>
-      <limit effort="0" lower="-2.181" upper="2.094" velocity="4.363"/>
+      <limit effort="0" lower="${radians(-125)}" upper="${radians(120)}" velocity="4.363"/>
     </joint>
     <joint type="revolute" name="${prefix}joint_6">
@@ -154,5 +154,5 @@
       <parent link="${prefix}link_5"/>
       <child link="${prefix}link_6"/>
-      <limit effort="0" lower="-6.981" upper="6.981" velocity="6.283"/>
+      <limit effort="0" lower="${radians(-400)}" upper="${radians(400)}" velocity="6.283"/>
     </joint>
     <joint type="fixed" name="${prefix}joint_6-tool0">

File: abb_irb4600_support/urdf/irb4600_60_205_macro.xacro (robot description, xacro)
@@ -104,5 +104,5 @@
       <parent link="${prefix}base_link"/>
       <child link="${prefix}link_1"/>
-      <limit effort="0" lower="-3.141" upper="3.141" velocity="3.054"/>
+      <limit effort="0" lower="${radians(-180)}" upper="${radians(180)}" velocity="3.054"/>
     </joint>
     <joint type="revolute" name="${prefix}joint_2">
@@ -111,5 +111,5 @@
       <parent link="${prefix}link_1"/>
       <child link="${prefix}link_2"/>
-      <limit effort="0" lower="-1.570" upper="2.617" velocity="3.054"/>
+      <limit effort="0" lower="${radians(-90)}" upper="${radians(150)}" velocity="3.054"/>
     </joint>
     <joint type="revolute" name="${prefix}joint_3">
@@ -118,5 +118,5 @@
       <parent link="${prefix}link_2"/>
       <child link="${prefix}link_3"/>
-      <limit effort="0" lower="-3.141" upper="1.308" velocity="3.054"/>
+      <limit effort="0" lower="${radians(-180)}" upper="${radians(75)}" velocity="3.054"/>
     </joint>
     <joint type="revolute" name="${prefix}joint_4">
@@ -125,5 +125,5 @@
       <parent link="${prefix}link_3"/>
       <child link="${prefix}link_4"/>
-      <limit effort="0" lower="-6.981" upper="6.981" velocity="4.363"/>
+      <limit effort="0" lower="${radians(-400)}" upper="${radians(400)}" velocity="4.363"/>
     </joint>
     <joint type="revolute" name="${prefix}joint_5">
@@ -132,5 +132,5 @@
       <parent link="${prefix}link_4"/>
       <child link="${prefix}link_5"/>
-      <limit effort="0" lower="-2.181" upper="2.094" velocity="4.363"/>
+      <limit effort="0" lower="${radians(-125)}" upper="${radians(120)}" velocity="4.363"/>
     </joint>
     <joint type="revolute" name="${prefix}joint_6">
@@ -139,5 +139,5 @@
       <parent link="${prefix}link_5"/>
       <child link="${prefix}link_6"/>
-      <limit effort="0" lower="-6.981" upper="6.981" velocity="6.283"/>
+      <limit effort="0" lower="${radians(-400)}" upper="${radians(400)}" velocity="6.283"/>
     </joint>
     <joint type="fixed" name="${prefix}joint_6-tool0">

Commit message: irb4600: variants share base_link and link_1.

File: abb_irb4600_support/urdf/irb4600_40_255_macro.xacro (robot description, xacro)
@@ -7,5 +7,5 @@
       <collision name="collision">
         <geometry>
-          <mesh filename="package://abb_irb4600_support/meshes/irb4600_60_205/collision/base_link.stl"/>
+          <mesh filename="package://abb_irb4600_support/meshes/irb4600/collision/base_link.stl"/>
         </geometry>
         <xacro:material_abb_white/>
@@ -13,5 +13,5 @@
       <visual name="visual">
         <geometry>
-          <mesh filename="package://abb_irb4600_support/meshes/irb4600_60_205/visual/base_link.stl"/>
+          <mesh filename="package://abb_irb4600_support/meshes/irb4600/visual/base_link.stl"/>
         </geometry>
         <xacro:material_abb_white/>
@@ -24,5 +24,5 @@
       <collision name="collision">
         <geometry>
-          <mesh filename="package://abb_irb4600_support/meshes/irb4600_60_205/collision/link_1.stl"/>
+          <mesh filename="package://abb_irb4600_support/meshes/irb4600/collision/link_1.stl"/>
         </geometry>
         <xacro:material_abb_white/>
@@ -30,5 +30,5 @@
       <visual name="visual">
         <geometry>
-          <mesh filename="package://abb_irb4600_support/meshes/irb4600_60_205/visual/link_1.stl"/>
+          <mesh filename="package://abb_irb4600_support/meshes/irb4600/visual/link_1.stl"/>
         </geometry>
         <xacro:material_abb_white/>

File: abb_irb4600_support/urdf/irb4600_60_205_macro.xacro (robot description, xacro)
@@ -6,10 +6,10 @@
       <collision name="collision">
         <geometry>
-          <mesh filename="package://abb_irb4600_support/meshes/irb4600_60_205/collision/base_link.stl"/>
+          <mesh filename="package://abb_irb4600_support/meshes/irb4600/collision/base_link.stl"/>
         </geometry>
       </collision>
       <visual name="visual">
         <geometry>
-          <mesh filename="package://abb_irb4600_support/meshes/irb4600_60_205/visual/base_link.stl"/>
+          <mesh filename="package://abb_irb4600_support/meshes/irb4600/visual/base_link.stl"/>
         </geometry>
         <material name="yellow">
@@ -21,10 +21,10 @@
       <collision name="collision">
         <geometry>
-          <mesh filename="package://abb_irb4600_support/meshes/irb4600_60_205/collision/link_1.stl"/>
+          <mesh filename="package://abb_irb4600_support/meshes/irb4600/collision/link_1.stl"/>
         </geometry>
       </collision>
       <visual name="visual">
         <geometry>
-          <mesh filename="package://abb_irb4600_support/meshes/irb4600_60_205/visual/link_1.stl"/>
+          <mesh filename="package://abb_irb4600_support/meshes/irb4600/visual/link_1.stl"/>
         </geometry>
         <material name="yellow"/>

Commit message: irb4600: convert common meshes to Collada.
Only for the visual meshes.

File: abb_irb4600_support/urdf/irb4600_40_255_macro.xacro (robot description, xacro)
@@ -13,5 +13,5 @@
       <visual name="visual">
         <geometry>
-          <mesh filename="package://abb_irb4600_support/meshes/irb4600/visual/base_link.stl"/>
+          <mesh filename="package://abb_irb4600_support/meshes/irb4600/visual/base_link.dae"/>
         </geometry>
         <xacro:material_abb_white/>
@@ -30,5 +30,5 @@
       <visual name="visual">
         <geometry>
-          <mesh filename="package://abb_irb4600_support/meshes/irb4600/visual/link_1.stl"/>
+          <mesh filename="package://abb_irb4600_support/meshes/irb4600/visual/link_1.dae"/>
         </geometry>
         <xacro:material_abb_white/>

File: abb_irb4600_support/urdf/irb4600_60_205_macro.xacro (robot description, xacro)
@@ -11,5 +11,5 @@
       <visual name="visual">
         <geometry>
-          <mesh filename="package://abb_irb4600_support/meshes/irb4600/visual/base_link.stl"/>
+          <mesh filename="package://abb_irb4600_support/meshes/irb4600/visual/base_link.dae"/>
         </geometry>
         <material name="yellow">
@@ -26,5 +26,5 @@
       <visual name="visual">
         <geometry>
-          <mesh filename="package://abb_irb4600_support/meshes/irb4600/visual/link_1.stl"/>
+          <mesh filename="package://abb_irb4600_support/meshes/irb4600/visual/link_1.dae"/>
         </geometry>
         <material name="yellow"/>
