Commit message: irb4600: convert 60/2.05 to Collada.
Visual meshes only again.

File: abb_irb4600_support/urdf/irb4600_60_205_macro.xacro (robot description, xacro)
@@ -39,5 +39,5 @@
       <visual name="visual">
         <geometry>
-          <mesh filename="package://abb_irb4600_support/meshes/irb4600_60_205/visual/link_2.stl"/>
+          <mesh filename="package://abb_irb4600_support/meshes/irb4600_60_205/visual/link_2.dae"/>
         </geometry>
         <material name="yellow"/>
@@ -52,5 +52,5 @@
       <visual name="visual">
         <geometry>
-          <mesh filename="package://abb_irb4600_support/meshes/irb4600_60_205/visual/link_3.stl"/>
+          <mesh filename="package://abb_irb4600_support/meshes/irb4600_60_205/visual/link_3.dae"/>
         </geometry>
         <material name="yellow"/>
@@ -65,5 +65,5 @@
       <visual name="visual">
         <geometry>
-          <mesh filename="package://abb_irb4600_support/meshes/irb4600_60_205/visual/link_4.stl"/>
+          <mesh filename="package://abb_irb4600_support/meshes/irb4600_60_205/visual/link_4.dae"/>
         </geometry>
         <material name="yellow"/>
@@ -78,5 +78,5 @@
       <visual name="visual">
         <geometry>
-          <mesh filename="package://abb_irb4600_support/meshes/irb4600_60_205/visual/link_5.stl"/>
+          <mesh filename="package://abb_irb4600_support/meshes/irb4600_60_205/visual/link_5.dae"/>
         </geometry>
         <material name="yellow"/>
@@ -91,5 +91,5 @@
       <visual name="visual">
         <geometry>
-          <mesh filename="package://abb_irb4600_support/meshes/irb4600_60_205/visual/link_6.stl"/>
+          <mesh filename="package://abb_irb4600_support/meshes/irb4600_60_205/visual/link_6.dae"/>
         </geometry>
         <material name="yellow"/>
