Commit message: base_links for all irb4600s are equal

File: abb_irb4600_support/urdf/irb4600_20_250_macro.xacro (robot description, xacro)
@@ -7,5 +7,5 @@
       <collision name="collision">
         <geometry>
-          <mesh filename="package://abb_irb4600_support/meshes/irb4600_20_250/collision/base_link.stl"/>
+          <mesh filename="package://abb_irb4600_support/meshes/irb4600_common/collision/base_link.stl"/>
         </geometry>
         <xacro:material_abb_white/>
@@ -13,5 +13,5 @@
       <visual name="visual">
         <geometry>
-          <mesh filename="package://abb_irb4600_support/meshes/irb4600_20_250/visual/base_link.stl"/>
+          <mesh filename="package://abb_irb4600_support/meshes/irb4600_common/visual/base_link.stl"/>
         </geometry>
         <xacro:material_abb_white/>

File: abb_irb4600_support/urdf/irb4600_40_255_macro.xacro (robot description, xacro)
@@ -7,5 +7,5 @@
       <collision name="collision">
         <geometry>
-          <mesh filename="package://abb_irb4600_support/meshes/irb4600_40_255/collision/base_link.stl"/>
+          <mesh filename="package://abb_irb4600_support/meshes/irb4600_common/collision/base_link.stl"/>
         </geometry>
         <xacro:material_abb_white/>
@@ -13,5 +13,5 @@
       <visual name="visual">
         <geometry>
-          <mesh filename="package://abb_irb4600_support/meshes/irb4600_40_255/visual/base_link.stl"/>
+          <mesh filename="package://abb_irb4600_support/meshes/irb4600_common/visual/base_link.stl"/>
         </geometry>
         <xacro:material_abb_white/>

File: abb_irb4600_support/urdf/irb4600_60_205_macro.xacro (robot description, xacro)
@@ -6,10 +6,10 @@
       <collision name="collision">
         <geometry>
-          <mesh filename="package://abb_irb4600_support/meshes/irb4600_60_205/collision/base_link.stl"/>
+          <mesh filename="package://abb_irb4600_support/meshes/irb4600_common/collision/base_link.stl"/>
         </geometry>
       </collision>
       <visual name="visual">
         <geometry>
-          <mesh filename="package://abb_irb4600_support/meshes/irb4600_60_205/visual/base_link.stl"/>
+          <mesh filename="package://abb_irb4600_support/meshes/irb4600_common/visual/base_link.stl"/>
         </geometry>
         <material name="yellow">

Commit message: link_1 in all models is the same

File: abb_irb4600_support/urdf/irb4600_20_250_macro.xacro (robot description, xacro)
@@ -24,5 +24,5 @@
       <collision name="collision">
         <geometry>
-          <mesh filename="package://abb_irb4600_support/meshes/irb4600_20_250/collision/link_1.stl"/>
+          <mesh filename="package://abb_irb4600_support/meshes/irb4600_common/collision/link_1.stl"/>
         </geometry>
         <xacro:material_abb_white/>
@@ -30,5 +30,5 @@
       <visual name="visual">
         <geometry>
-          <mesh filename="package://abb_irb4600_support/meshes/irb4600_20_250/visual/link_1.stl"/>
+          <mesh filename="package://abb_irb4600_support/meshes/irb4600_common/visual/link_1.stl"/>
         </geometry>
         <xacro:material_abb_white/>

File: abb_irb4600_support/urdf/irb4600_40_255_macro.xacro (robot description, xacro)
@@ -24,5 +24,5 @@
       <collision name="collision">
         <geometry>
-          <mesh filename="package://abb_irb4600_support/meshes/irb4600_40_255/collision/link_1.stl"/>
+          <mesh filename="package://abb_irb4600_support/meshes/irb4600_common/collision/link_1.stl"/>
         </geometry>
         <xacro:material_abb_white/>
@@ -30,5 +30,5 @@
       <visual name="visual">
         <geometry>
-          <mesh filename="package://abb_irb4600_support/meshes/irb4600_40_255/visual/link_1.stl"/>
+          <mesh filename="package://abb_irb4600_support/meshes/irb4600_common/visual/link_1.stl"/>
         </geometry>
         <xacro:material_abb_white/>

File: abb_irb4600_support/urdf/irb4600_60_205_macro.xacro (robot description, xacro)
@@ -21,10 +21,10 @@
       <collision name="collision">
         <geometry>
-          <mesh filename="package://abb_irb4600_support/meshes/irb4600_60_205/collision/link_1.stl"/>
+          <mesh filename="package://abb_irb4600_support/meshes/irb4600_common/collision/link_1.stl"/>
         </geometry>
       </collision>
       <visual name="visual">
         <geometry>
-          <mesh filename="package://abb_irb4600_support/meshes/irb4600_60_205/visual/link_1.stl"/>
+          <mesh filename="package://abb_irb4600_support/meshes/irb4600_common/visual/link_1.stl"/>
         </geometry>
         <material name="yellow"/>

Commit message: seperated parts into a common and specific mesh folders

File: abb_irb4600_support/urdf/irb4600_20_250_macro.xacro (robot description, xacro)
@@ -129,5 +129,5 @@
     </joint>
     <joint type="revolute" name="${prefix}joint_3">
-      <origin xyz="0 0 0.9" rpy="0 0 0"/>
+      <origin xyz="0 0 1.095" rpy="0 0 0"/>
       <axis xyz="0 1 0"/>
       <parent link="${prefix}link_2"/>

File: abb_irb4600_support/urdf/irb4600_40_255_macro.xacro (robot description, xacro)
@@ -129,5 +129,5 @@
     </joint>
     <joint type="revolute" name="${prefix}joint_3">
-      <origin xyz="0 0 0.9" rpy="0 0 0"/>
+      <origin xyz="0 0 1.095" rpy="0 0 0"/>
       <axis xyz="0 1 0"/>
       <parent link="${prefix}link_2"/>

Commit message: Update abb_irb4600_support/urdf/irb4600_20_250_macro.xacro
Co-Authored-By: rtonnaer <r.tonnaer@tudelft.nl>

File: abb_irb4600_support/urdf/irb4600_20_250_macro.xacro (robot description, xacro)
@@ -159,5 +159,5 @@
       <parent link="${prefix}link_6"/>
       <child link="${prefix}tool0"/>
-      <origin xyz="0 0 0" rpy="0 1.57079632679 0"/>
+      <origin xyz="0 0 0" rpy="0 ${pi/2.0} 0"/>
     </joint>
     <!-- end of joint list -->

Commit message: updated axes limits to degrees with a radians conversion

File: abb_irb4600_support/urdf/irb4600_20_250_macro.xacro (robot description, xacro)
@@ -119,5 +119,5 @@
       <parent link="${prefix}base_link"/>
       <child link="${prefix}link_1"/>
-      <limit effort="0" lower="-3.141" upper="3.141" velocity="3.054"/>
+      <limit effort="0" lower="${radians(-180)}" upper="${radians(180)}" velocity="3.054"/>
     </joint>
     <joint type="revolute" name="${prefix}joint_2">
@@ -126,5 +126,5 @@
       <parent link="${prefix}link_1"/>
       <child link="${prefix}link_2"/>
-      <limit effort="0" lower="-1.570" upper="2.617" velocity="3.054"/>
+      <limit effort="0" lower="${radians(-90)}" upper="${radians(150)}" velocity="3.054"/>
     </joint>
     <joint type="revolute" name="${prefix}joint_3">
@@ -133,5 +133,5 @@
       <parent link="${prefix}link_2"/>
       <child link="${prefix}link_3"/>
-      <limit effort="0" lower="-3.141" upper="1.308" velocity="3.054"/>
+      <limit effort="0" lower="${radians(-180)}" upper="${radians(75)}" velocity="3.054"/>
     </joint>
     <joint type="revolute" name="${prefix}joint_4">
@@ -140,5 +140,5 @@
       <parent link="${prefix}link_3"/>
       <child link="${prefix}link_4"/>
-      <limit effort="0" lower="-6.981" upper="6.981" velocity="4.363"/>
+      <limit effort="0" lower="${radians(-400)}" upper="${radians(400)}" velocity="4.363"/>
     </joint>
     <joint type="revolute" name="${prefix}joint_5">
@@ -147,5 +147,5 @@
       <parent link="${prefix}link_4"/>
       <child link="${prefix}link_5"/>
-      <limit effort="0" lower="-2.181" upper="2.094" velocity="4.363"/>
+      <limit effort="0" lower="${radians(-125)}" upper="${radians(120)}" velocity="4.363"/>
     </joint>
     <joint type="revolute" name="${prefix}joint_6">
@@ -154,5 +154,5 @@
       <parent link="${prefix}link_5"/>
       <child link="${prefix}link_6"/>
-      <limit effort="0" lower="-6.981" upper="6.981" velocity="6.283"/>
+      <limit effort="0" lower="${radians(-400)}" upper="${radians(400)}" velocity="6.283"/>
     </joint>
     <joint type="fixed" name="${prefix}joint_6-tool0">

Commit message: irb4600: add 20/2.50 and 40/2.55 variants

File: abb_irb4600_support/urdf/irb4600_20_250_macro.xacro (robot description, xacro)
@@ -1,5 +1,6 @@
 <?xml version="1.0"?>
 <robot xmlns:xacro="http://ros.org/wiki/xacro">
-  <xacro:macro name="abb_irb4600_60_205" params="prefix">
+<xacro:include filename="$(find abb_resources)/urdf/common_materials.xacro"/>
+  <xacro:macro name="abb_irb4600_20_250" params="prefix">
     <!-- link list -->
     <link name="${prefix}base_link">
@@ -8,4 +9,5 @@
           <mesh filename="package://abb_irb4600_support/meshes/irb4600_common/collision/base_link.stl"/>
         </geometry>
+        <xacro:material_abb_white/>
       </collision>
       <visual name="visual">
@@ -13,4 +15,5 @@
           <mesh filename="package://abb_irb4600_support/meshes/irb4600_common/visual/base_link.stl"/>
         </geometry>
+        <xacro:material_abb_white/>
         <material name="yellow">
           <color rgba="1 1 0 1"/>
@@ -23,4 +26,5 @@
           <mesh filename="package://abb_irb4600_support/meshes/irb4600_common/collision/link_1.stl"/>
         </geometry>
+        <xacro:material_abb_white/>
       </collision>
       <visual name="visual">
@@ -28,4 +32,5 @@
           <mesh filename="package://abb_irb4600_support/meshes/irb4600_common/visual/link_1.stl"/>
         </geometry>
+        <xacro:material_abb_white/>
         <material name="yellow"/>
       </visual>
@@ -34,11 +39,13 @@
       <collision name="collision">
         <geometry>
-          <mesh filename="package://abb_irb4600_support/meshes/irb4600_60_205/collision/link_2.stl"/>
+          <mesh filename="package://abb_irb4600_support/meshes/irb4600_20_250/collision/link_2.stl"/>
         </geometry>
+        <xacro:material_abb_white/>
       </collision>
       <visual name="visual">
         <geometry>
-          <mesh filename="package://abb_irb4600_support/meshes/irb4600_60_205/visual/link_2.stl"/>
+          <mesh filename="package://abb_irb4600_support/meshes/irb4600_20_250/visual/link_2.stl"/>
         </geometry>
+        <xacro:material_abb_white/>
         <material name="yellow"/>
       </visual>
@@ -47,11 +54,13 @@
       <collision name="collision">
         <geometry>
-          <mesh filename="package://abb_irb4600_support/meshes/irb4600_60_205/collision/link_3.stl"/>
+          <mesh filename="package://abb_irb4600_support/meshes/irb4600_20_250/collision/link_3.stl"/>
         </geometry>
+        <xacro:material_abb_white/>
       </collision>
       <visual name="visual">
         <geometry>
-          <mesh filename="package://abb_irb4600_support/meshes/irb4600_60_205/visual/link_3.stl"/>
+          <mesh filename="package://abb_irb4600_support/meshes/irb4600_20_250/visual/link_3.stl"/>
         </geometry>
+        <xacro:material_abb_white/>
         <material name="yellow"/>
       </visual>
@@ -60,11 +69,13 @@
       <collision name="collision">
         <geometry>
-          <mesh filename="package://abb_irb4600_support/meshes/irb4600_60_205/collision/link_4.stl"/>
+          <mesh filename="package://abb_irb4600_support/meshes/irb4600_20_250/collision/link_4.stl"/>
         </geometry>
+        <xacro:material_abb_white/>
       </collision>
       <visual name="visual">
         <geometry>
-          <mesh filename="package://abb_irb4600_support/meshes/irb4600_60_205/visual/link_4.stl"/>
+          <mesh filename="package://abb_irb4600_support/meshes/irb4600_20_250/visual/link_4.stl"/>
         </geometry>
+        <xacro:material_abb_white/>
         <material name="yellow"/>
       </visual>
@@ -73,11 +84,13 @@
       <collision name="collision">
         <geometry>
-          <mesh filename="package://abb_irb4600_support/meshes/irb4600_60_205/collision/link_5.stl"/>
+          <mesh filename="package://abb_irb4600_support/meshes/irb4600_20_250/collision/link_5.stl"/>
         </geometry>
+        <xacro:material_abb_white/>
       </collision>
       <visual name="visual">
         <geometry>
-          <mesh filename="package://abb_irb4600_support/meshes/irb4600_60_205/visual/link_5.stl"/>
+          <mesh filename="package://abb_irb4600_support/meshes/irb4600_20_250/visual/link_5.stl"/>
         </geometry>
+        <xacro:material_abb_white/>
         <material name="yellow"/>
       </visual>
@@ -86,11 +99,13 @@
       <collision name="collision">
         <geometry>
-          <mesh filename="package://abb_irb4600_support/meshes/irb4600_60_205/collision/link_6.stl"/>
+          <mesh filename="package://abb_irb4600_support/meshes/irb4600_20_250/collision/link_6.stl"/>
         </geometry>
+        <xacro:material_abb_white/>
       </collision>
       <visual name="visual">
         <geometry>
-          <mesh filename="package://abb_irb4600_support/meshes/irb4600_60_205/visual/link_6.stl"/>
+          <mesh filename="package://abb_irb4600_support/meshes/irb4600_20_250/visual/link_6.stl"/>
         </geometry>
+        <xacro:material_abb_white/>
         <material name="yellow"/>
       </visual>
@@ -114,5 +129,5 @@
     </joint>
     <joint type="revolute" name="${prefix}joint_3">
-      <origin xyz="0 0 0.9" rpy="0 0 0"/>
+      <origin xyz="0 0 1.095" rpy="0 0 0"/>
       <axis xyz="0 1 0"/>
       <parent link="${prefix}link_2"/>
@@ -128,5 +143,5 @@
     </joint>
     <joint type="revolute" name="${prefix}joint_5">
-      <origin xyz="0.960 0 0 " rpy="0 0 0"/>
+      <origin xyz="1.2305 0 0 " rpy="0 0 0"/>
       <axis xyz="0 1 0"/>
       <parent link="${prefix}link_4"/>
@@ -135,5 +150,5 @@
     </joint>
     <joint type="revolute" name="${prefix}joint_6">
-      <origin xyz="0.135 0 0 " rpy="0 0 0"/>
+      <origin xyz="0.085 0 0 " rpy="0 0 0"/>
       <axis xyz="1 0 0"/>
       <parent link="${prefix}link_5"/>
@@ -144,5 +159,5 @@
       <parent link="${prefix}link_6"/>
       <child link="${prefix}tool0"/>
-      <origin xyz="0 0 0" rpy="0 1.57079632679 0"/>
+      <origin xyz="0 0 0" rpy="0 ${pi/2.0} 0"/>
     </joint>
     <!-- end of joint list -->

File: abb_irb4600_support/urdf/irb4600_40_255_macro.xacro (robot description, xacro)
@@ -1,5 +1,6 @@
 <?xml version="1.0"?>
 <robot xmlns:xacro="http://ros.org/wiki/xacro">
-  <xacro:macro name="abb_irb4600_60_205" params="prefix">
+<xacro:include filename="$(find abb_resources)/urdf/common_materials.xacro"/>
+  <xacro:macro name="abb_irb4600_40_255" params="prefix">
     <!-- link list -->
     <link name="${prefix}base_link">
@@ -8,4 +9,5 @@
           <mesh filename="package://abb_irb4600_support/meshes/irb4600_common/collision/base_link.stl"/>
         </geometry>
+        <xacro:material_abb_white/>
       </collision>
       <visual name="visual">
@@ -13,4 +15,5 @@
           <mesh filename="package://abb_irb4600_support/meshes/irb4600_common/visual/base_link.stl"/>
         </geometry>
+        <xacro:material_abb_white/>
         <material name="yellow">
           <color rgba="1 1 0 1"/>
@@ -23,4 +26,5 @@
           <mesh filename="package://abb_irb4600_support/meshes/irb4600_common/collision/link_1.stl"/>
         </geometry>
+        <xacro:material_abb_white/>
       </collision>
       <visual name="visual">
@@ -28,4 +32,5 @@
           <mesh filename="package://abb_irb4600_support/meshes/irb4600_common/visual/link_1.stl"/>
         </geometry>
+        <xacro:material_abb_white/>
         <material name="yellow"/>
       </visual>
@@ -34,11 +39,13 @@
       <collision name="collision">
         <geometry>
-          <mesh filename="package://abb_irb4600_support/meshes/irb4600_60_205/collision/link_2.stl"/>
+          <mesh filename="package://abb_irb4600_support/meshes/irb4600_40_255/collision/link_2.stl"/>
         </geometry>
+        <xacro:material_abb_white/>
       </collision>
       <visual name="visual">
         <geometry>
-          <mesh filename="package://abb_irb4600_support/meshes/irb4600_60_205/visual/link_2.stl"/>
+          <mesh filename="package://abb_irb4600_support/meshes/irb4600_40_255/visual/link_2.stl"/>
         </geometry>
+        <xacro:material_abb_white/>
         <material name="yellow"/>
       </visual>
@@ -47,11 +54,13 @@
       <collision name="collision">
         <geometry>
-          <mesh filename="package://abb_irb4600_support/meshes/irb4600_60_205/collision/link_3.stl"/>
+          <mesh filename="package://abb_irb4600_support/meshes/irb4600_40_255/collision/link_3.stl"/>
         </geometry>
+        <xacro:material_abb_white/>
       </collision>
       <visual name="visual">
         <geometry>
-          <mesh filename="package://abb_irb4600_support/meshes/irb4600_60_205/visual/link_3.stl"/>
+          <mesh filename="package://abb_irb4600_support/meshes/irb4600_40_255/visual/link_3.stl"/>
         </geometry>
+        <xacro:material_abb_white/>
         <material name="yellow"/>
       </visual>
@@ -60,11 +69,13 @@
       <collision name="collision">
         <geometry>
-          <mesh filename="package://abb_irb4600_support/meshes/irb4600_60_205/collision/link_4.stl"/>
+          <mesh filename="package://abb_irb4600_support/meshes/irb4600_40_255/collision/link_4.stl"/>
         </geometry>
+        <xacro:material_abb_white/>
       </collision>
       <visual name="visual">
         <geometry>
-          <mesh filename="package://abb_irb4600_support/meshes/irb4600_60_205/visual/link_4.stl"/>
+          <mesh filename="package://abb_irb4600_support/meshes/irb4600_40_255/visual/link_4.stl"/>
         </geometry>
+        <xacro:material_abb_white/>
         <material name="yellow"/>
       </visual>
@@ -73,11 +84,13 @@
       <collision name="collision">
         <geometry>
-          <mesh filename="package://abb_irb4600_support/meshes/irb4600_60_205/collision/link_5.stl"/>
+          <mesh filename="package://abb_irb4600_support/meshes/irb4600_40_255/collision/link_5.stl"/>
         </geometry>
+        <xacro:material_abb_white/>
       </collision>
       <visual name="visual">
         <geometry>
-          <mesh filename="package://abb_irb4600_support/meshes/irb4600_60_205/visual/link_5.stl"/>
+          <mesh filename="package://abb_irb4600_support/meshes/irb4600_40_255/visual/link_5.stl"/>
         </geometry>
+        <xacro:material_abb_white/>
         <material name="yellow"/>
       </visual>
@@ -86,11 +99,13 @@
       <collision name="collision">
         <geometry>
-          <mesh filename="package://abb_irb4600_support/meshes/irb4600_60_205/collision/link_6.stl"/>
+          <mesh filename="package://abb_irb4600_support/meshes/irb4600_40_255/collision/link_6.stl"/>
         </geometry>
+        <xacro:material_abb_white/>
       </collision>
       <visual name="visual">
         <geometry>
-          <mesh filename="package://abb_irb4600_support/meshes/irb4600_60_205/visual/link_6.stl"/>
+          <mesh filename="package://abb_irb4600_support/meshes/irb4600_40_255/visual/link_6.stl"/>
         </geometry>
+        <xacro:material_abb_white/>
         <material name="yellow"/>
       </visual>
@@ -114,5 +129,5 @@
     </joint>
     <joint type="revolute" name="${prefix}joint_3">
-      <origin xyz="0 0 0.9" rpy="0 0 0"/>
+      <origin xyz="0 0 1.095" rpy="0 0 0"/>
       <axis xyz="0 1 0"/>
       <parent link="${prefix}link_2"/>
@@ -128,5 +143,5 @@
     </joint>
     <joint type="revolute" name="${prefix}joint_5">
-      <origin xyz="0.960 0 0 " rpy="0 0 0"/>
+      <origin xyz="1.270 0 0 " rpy="0 0 0"/>
       <axis xyz="0 1 0"/>
       <parent link="${prefix}link_4"/>
@@ -144,5 +159,5 @@
       <parent link="${prefix}link_6"/>
       <child link="${prefix}tool0"/>
-      <origin xyz="0 0 0" rpy="0 1.57079632679 0"/>
+      <origin xyz="0 0 0" rpy="0 ${pi/2.0} 0"/>
     </joint>
     <!-- end of joint list -->
