Commit message: converted meshes to dae and used meshlab to reduce mesh sizes. IRB4600 meshes reduced from 14.4 mb to 8.5 mb

File: abb_irb4600_support/urdf/irb4600_20_250_macro.xacro (robot description, xacro)
@@ -13,5 +13,5 @@
       <visual name="visual">
         <geometry>
-          <mesh filename="package://abb_irb4600_support/meshes/irb4600_common/visual/base_link.stl"/>
+          <mesh filename="package://abb_irb4600_support/meshes/irb4600_common/visual/base_link.dae"/>
         </geometry>
         <xacro:material_abb_white/>
@@ -30,5 +30,5 @@
       <visual name="visual">
         <geometry>
-          <mesh filename="package://abb_irb4600_support/meshes/irb4600_common/visual/link_1.stl"/>
+          <mesh filename="package://abb_irb4600_support/meshes/irb4600_common/visual/link_1.dae"/>
         </geometry>
         <xacro:material_abb_white/>
@@ -45,5 +45,5 @@
       <visual name="visual">
         <geometry>
-          <mesh filename="package://abb_irb4600_support/meshes/irb4600_20_250/visual/link_2.stl"/>
+          <mesh filename="package://abb_irb4600_support/meshes/irb4600_20_250/visual/link_2.dae"/>
         </geometry>
         <xacro:material_abb_white/>
@@ -60,5 +60,5 @@
       <visual name="visual">
         <geometry>
-          <mesh filename="package://abb_irb4600_support/meshes/irb4600_20_250/visual/link_3.stl"/>
+          <mesh filename="package://abb_irb4600_support/meshes/irb4600_20_250/visual/link_3.dae"/>
         </geometry>
         <xacro:material_abb_white/>
@@ -75,5 +75,5 @@
       <visual name="visual">
         <geometry>
-          <mesh filename="package://abb_irb4600_support/meshes/irb4600_20_250/visual/link_4.stl"/>
+          <mesh filename="package://abb_irb4600_support/meshes/irb4600_20_250/visual/link_4.dae"/>
         </geometry>
         <xacro:material_abb_white/>
@@ -90,5 +90,5 @@
       <visual name="visual">
         <geometry>
-          <mesh filename="package://abb_irb4600_support/meshes/irb4600_20_250/visual/link_5.stl"/>
+          <mesh filename="package://abb_irb4600_support/meshes/irb4600_20_250/visual/link_5.dae"/>
         </geometry>
         <xacro:material_abb_white/>
@@ -105,5 +105,5 @@
       <visual name="visual">
         <geometry>
-          <mesh filename="package://abb_irb4600_support/meshes/irb4600_20_250/visual/link_6.stl"/>
+          <mesh filename="package://abb_irb4600_support/meshes/irb4600_20_250/visual/link_6.dae"/>
         </geometry>
         <xacro:material_abb_white/>

File: abb_irb4600_support/urdf/irb4600_40_255_macro.xacro (robot description, xacro)
@@ -13,5 +13,5 @@
       <visual name="visual">
         <geometry>
-          <mesh filename="package://abb_irb4600_support/meshes/irb4600_common/visual/base_link.stl"/>
+          <mesh filename="package://abb_irb4600_support/meshes/irb4600_common/visual/base_link.dae"/>
         </geometry>
         <xacro:material_abb_white/>
@@ -30,5 +30,5 @@
       <visual name="visual">
         <geometry>
-          <mesh filename="package://abb_irb4600_support/meshes/irb4600_common/visual/link_1.stl"/>
+          <mesh filename="package://abb_irb4600_support/meshes/irb4600_common/visual/link_1.dae"/>
         </geometry>
         <xacro:material_abb_white/>
@@ -45,5 +45,5 @@
       <visual name="visual">
         <geometry>
-          <mesh filename="package://abb_irb4600_support/meshes/irb4600_40_255/visual/link_2.stl"/>
+          <mesh filename="package://abb_irb4600_support/meshes/irb4600_40_255/visual/link_2.dae"/>
         </geometry>
         <xacro:material_abb_white/>
@@ -60,5 +60,5 @@
       <visual name="visual">
         <geometry>
-          <mesh filename="package://abb_irb4600_support/meshes/irb4600_40_255/visual/link_3.stl"/>
+          <mesh filename="package://abb_irb4600_support/meshes/irb4600_40_255/visual/link_3.dae"/>
         </geometry>
         <xacro:material_abb_white/>
@@ -75,5 +75,5 @@
       <visual name="visual">
         <geometry>
-          <mesh filename="package://abb_irb4600_support/meshes/irb4600_40_255/visual/link_4.stl"/>
+          <mesh filename="package://abb_irb4600_support/meshes/irb4600_40_255/visual/link_4.dae"/>
         </geometry>
         <xacro:material_abb_white/>
@@ -90,5 +90,5 @@
       <visual name="visual">
         <geometry>
-          <mesh filename="package://abb_irb4600_support/meshes/irb4600_40_255/visual/link_5.stl"/>
+          <mesh filename="package://abb_irb4600_support/meshes/irb4600_40_255/visual/link_5.dae"/>
         </geometry>
         <xacro:material_abb_white/>
@@ -105,5 +105,5 @@
       <visual name="visual">
         <geometry>
-          <mesh filename="package://abb_irb4600_support/meshes/irb4600_40_255/visual/link_6.stl"/>
+          <mesh filename="package://abb_irb4600_support/meshes/irb4600_40_255/visual/link_6.dae"/>
         </geometry>
         <xacro:material_abb_white/>

File: abb_irb4600_support/urdf/irb4600_60_205_macro.xacro (robot description, xacro)
@@ -11,5 +11,5 @@
       <visual name="visual">
         <geometry>
-          <mesh filename="package://abb_irb4600_support/meshes/irb4600_common/visual/base_link.stl"/>
+          <mesh filename="package://abb_irb4600_support/meshes/irb4600_common/visual/base_link.dae"/>
         </geometry>
         <material name="yellow">
@@ -26,5 +26,5 @@
       <visual name="visual">
         <geometry>
-          <mesh filename="package://abb_irb4600_support/meshes/irb4600_common/visual/link_1.stl"/>
+          <mesh filename="package://abb_irb4600_support/meshes/irb4600_common/visual/link_1.dae"/>
         </geometry>
         <material name="yellow"/>
@@ -39,5 +39,5 @@
       <visual name="visual">
         <geometry>
-          <mesh filename="package://abb_irb4600_support/meshes/irb4600_60_205/visual/link_2.stl"/>
+          <mesh filename="package://abb_irb4600_support/meshes/irb4600_60_205/visual/link_2.dae"/>
         </geometry>
         <material name="yellow"/>
@@ -52,5 +52,5 @@
       <visual name="visual">
         <geometry>
-          <mesh filename="package://abb_irb4600_support/meshes/irb4600_60_205/visual/link_3.stl"/>
+          <mesh filename="package://abb_irb4600_support/meshes/irb4600_60_205/visual/link_3.dae"/>
         </geometry>
         <material name="yellow"/>
@@ -65,5 +65,5 @@
       <visual name="visual">
         <geometry>
-          <mesh filename="package://abb_irb4600_support/meshes/irb4600_60_205/visual/link_4.stl"/>
+          <mesh filename="package://abb_irb4600_support/meshes/irb4600_60_205/visual/link_4.dae"/>
         </geometry>
         <material name="yellow"/>
@@ -78,5 +78,5 @@
       <visual name="visual">
         <geometry>
-          <mesh filename="package://abb_irb4600_support/meshes/irb4600_60_205/visual/link_5.stl"/>
+          <mesh filename="package://abb_irb4600_support/meshes/irb4600_60_205/visual/link_5.dae"/>
         </geometry>
         <material name="yellow"/>
@@ -91,5 +91,5 @@
       <visual name="visual">
         <geometry>
-          <mesh filename="package://abb_irb4600_support/meshes/irb4600_60_205/visual/link_6.stl"/>
+          <mesh filename="package://abb_irb4600_support/meshes/irb4600_60_205/visual/link_6.dae"/>
         </geometry>
         <material name="yellow"/>

Commit message: Added flange frame for irb4600

File: abb_irb4600_support/urdf/irb4600_20_250_macro.xacro (robot description, xacro)
@@ -156,11 +156,5 @@
     </joint>
     <!-- end of joint list -->
-    <link name="${prefix}tool0"/>
-    <joint type="fixed" name="${prefix}joint_6-tool0">
-      <parent link="${prefix}link_6"/>
-      <child link="${prefix}tool0"/>
-      <origin xyz="0 0 0" rpy="0 ${pi/2.0} 0"/>
-    </joint>
-    <!-- ROS base_link to ABB World Coordinates transform -->
+    <!-- ROS-Industrial 'base' frame: base_link to ABB World Coordinates transform -->
     <link name="${prefix}base" />
     <joint name="${prefix}base_link-base" type="fixed">
@@ -169,4 +163,18 @@
       <child link="${prefix}base"/>
     </joint>
+    <!-- ROS-Industrial 'flange' frame: attachment point for EEF models -->
+    <link name="${prefix}flange"/>
+    <joint type="fixed" name="${prefix}joint_6-flange">
+      <origin xyz="0 0 0" rpy="0 0 0"/>
+      <parent link="${prefix}link_6"/>
+      <child link="${prefix}flange"/>
+    </joint>
+    <!-- ROS-Industrial 'tool0' frame: all-zeros tool frame -->
+    <link name="${prefix}tool0" />
+    <joint name="${prefix}link_6-tool0" type="fixed">
+      <origin xyz="0 0 0" rpy="0 ${pi/2.0} 0" />
+      <parent link="${prefix}flange" />
+      <child link="${prefix}tool0" />
+    </joint>
   </xacro:macro>
 </robot>

File: abb_irb4600_support/urdf/irb4600_40_255_macro.xacro (robot description, xacro)
@@ -156,11 +156,5 @@
     </joint>
     <!-- end of joint list -->
-    <link name="${prefix}tool0"/>
-    <joint type="fixed" name="${prefix}joint_6-tool0">
-      <parent link="${prefix}link_6"/>
-      <child link="${prefix}tool0"/>
-      <origin xyz="0 0 0" rpy="0 ${pi/2.0} 0"/>
-    </joint>
-    <!-- ROS base_link to ABB World Coordinates transform -->
+    <!-- ROS-Industrial 'base' frame: base_link to ABB World Coordinates transform -->
     <link name="${prefix}base" />
     <joint name="${prefix}base_link-base" type="fixed">
@@ -169,4 +163,18 @@
       <child link="${prefix}base"/>
     </joint>
+    <!-- ROS-Industrial 'flange' frame: attachment point for EEF models -->
+    <link name="${prefix}flange"/>
+    <joint type="fixed" name="${prefix}joint_6-flange">
+      <origin xyz="0 0 0" rpy="0 0 0"/>
+      <parent link="${prefix}link_6"/>
+      <child link="${prefix}flange"/>
+    </joint>
+    <!-- ROS-Industrial 'tool0' frame: all-zeros tool frame -->
+    <link name="${prefix}tool0" />
+    <joint name="${prefix}link_6-tool0" type="fixed">
+      <origin xyz="0 0 0" rpy="0 ${pi/2.0} 0" />
+      <parent link="${prefix}flange" />
+      <child link="${prefix}tool0" />
+    </joint>
   </xacro:macro>
 </robot>

File: abb_irb4600_support/urdf/irb4600_60_205_macro.xacro (robot description, xacro)
@@ -96,5 +96,4 @@
       </visual>
     </link>
-    <link name="${prefix}tool0"/>
     <!-- end of link list -->
     <!-- joint list -->
@@ -141,11 +140,6 @@
       <limit effort="0" lower="-6.981" upper="6.981" velocity="6.283"/>
     </joint>
-    <joint type="fixed" name="${prefix}joint_6-tool0">
-      <parent link="${prefix}link_6"/>
-      <child link="${prefix}tool0"/>
-      <origin xyz="0 0 0" rpy="0 1.57079632679 0"/>
-    </joint>
     <!-- end of joint list -->
-    <!-- ROS base_link to ABB World Coordinates transform -->
+    <!-- ROS-Industrial 'base' frame: base_link to ABB World Coordinates transform -->
     <link name="${prefix}base" />
     <joint name="${prefix}base_link-base" type="fixed">
@@ -154,4 +148,18 @@
       <child link="${prefix}base"/>
     </joint>
+    <!-- ROS-Industrial 'flange' frame: attachment point for EEF models -->
+    <link name="${prefix}flange"/>
+    <joint type="fixed" name="${prefix}joint_6-flange">
+      <origin xyz="0 0 0" rpy="0 0 0"/>
+      <parent link="${prefix}link_6"/>
+      <child link="${prefix}flange"/>
+    </joint>
+    <!-- ROS-Industrial 'tool0' frame: all-zeros tool frame -->
+    <link name="${prefix}tool0" />
+    <joint name="${prefix}link_6-tool0" type="fixed">
+      <origin xyz="0 0 0" rpy="0 ${pi/2.0} 0" />
+      <parent link="${prefix}flange" />
+      <child link="${prefix}tool0" />
+    </joint>
   </xacro:macro>
 </robot>

Commit message: Use radians() for consistency

File: abb_irb4600_support/urdf/irb4600_20_250_macro.xacro (robot description, xacro)
@@ -173,5 +173,5 @@
     <link name="${prefix}tool0" />
     <joint name="${prefix}link_6-tool0" type="fixed">
-      <origin xyz="0 0 0" rpy="0 ${pi/2.0} 0" />
+      <origin xyz="0 0 0" rpy="0 ${radians(90)} 0" />
       <parent link="${prefix}flange" />
       <child link="${prefix}tool0" />

File: abb_irb4600_support/urdf/irb4600_40_255_macro.xacro (robot description, xacro)
@@ -173,5 +173,5 @@
     <link name="${prefix}tool0" />
     <joint name="${prefix}link_6-tool0" type="fixed">
-      <origin xyz="0 0 0" rpy="0 ${pi/2.0} 0" />
+      <origin xyz="0 0 0" rpy="0 ${radians(90)} 0" />
       <parent link="${prefix}flange" />
       <child link="${prefix}tool0" />

File: abb_irb4600_support/urdf/irb4600_60_205_macro.xacro (robot description, xacro)
@@ -158,5 +158,5 @@
     <link name="${prefix}tool0" />
     <joint name="${prefix}link_6-tool0" type="fixed">
-      <origin xyz="0 0 0" rpy="0 ${pi/2.0} 0" />
+      <origin xyz="0 0 0" rpy="0 ${radians(90)} 0" />
       <parent link="${prefix}flange" />
       <child link="${prefix}tool0" />

File: abb_irb7600_support/urdf/irb7600_150_350_macro.xacro (robot description, xacro)
@@ -205,5 +205,5 @@
     <link name="${prefix}tool0" />
     <joint name="${prefix}link_6-tool0" type="fixed">
-      <origin xyz="0 0 0" rpy="0 ${pi/2.0} 0" />
+      <origin xyz="0 0 0" rpy="0 ${radians(90)} 0" />
       <parent link="${prefix}flange" />
       <child link="${prefix}tool0" />

Commit message: Fix length of link5 in IRB4600-20/2.50
based on Product specification - IRB 4600 3HAC032885-001 Revision: Z

File: abb_irb4600_support/urdf/irb4600_20_250_macro.xacro (robot description, xacro)
@@ -142,5 +142,5 @@
     </joint>
     <joint type="revolute" name="${prefix}joint_5">
-      <origin xyz="1.235 0 0" rpy="0 0 0"/>
+      <origin xyz="1.2305 0 0" rpy="0 0 0"/>
       <axis xyz="0 1 0"/>
       <parent link="${prefix}link_4"/>
