Commit message: Added flange frame for irb6700

File: abb_irb6700_support/urdf/irb6700_200_260_macro.xacro (robot description, xacro)
@@ -148,5 +148,4 @@
       </collision>
     </link>
-    <link name="${prefix}tool0"/>
     <joint name="${prefix}joint_1" type="revolute">
       <origin xyz="0 0 0.78" rpy="0 0 0" />
@@ -191,10 +190,4 @@
       <limit lower="-${radians(360)}" upper="${radians(360)}" effort="0" velocity="${radians(190)}" />
     </joint>
-    <joint name="${prefix}joint_6_tool0" type="fixed">
-      <origin xyz="0 0 0" rpy="0 ${radians(90)} 0" />
-      <parent link="${prefix}link_6" />
-      <child link="${prefix}tool0" />
-      <axis xyz="0 0 0" />
-    </joint>
     <joint name="${prefix}cylinder_joint" type="revolute">
       <origin xyz="-0.349 -0.194 -0.142" rpy="0 0 0" />
@@ -213,11 +206,25 @@
       <limit lower="-0.25" upper="0.25" effort="0" velocity="100" />
     </joint>
-    <!-- ROS base_link to ABB World Coordinates transform -->
-    <link name="${prefix}base"/>
-    <joint name="${prefix}base_link_base" type="fixed">
+    <!-- ROS-Industrial 'base' frame: base_link to ABB World Coordinates transform -->
+    <link name="${prefix}base" />
+    <joint name="${prefix}base_link-base" type="fixed">
       <origin xyz="0 0 0" rpy="0 0 0"/>
       <parent link="${prefix}base_link"/>
       <child link="${prefix}base"/>
     </joint>
+    <!-- ROS-Industrial 'flange' frame: attachment point for EEF models -->
+    <link name="${prefix}flange"/>
+    <joint type="fixed" name="${prefix}joint_6-flange">
+      <origin xyz="0 0 0" rpy="0 0 0"/>
+      <parent link="${prefix}link_6"/>
+      <child link="${prefix}flange"/>
+    </joint>
+    <!-- ROS-Industrial 'tool0' frame: all-zeros tool frame -->
+    <link name="${prefix}tool0" />
+    <joint name="${prefix}link_6-tool0" type="fixed">
+      <origin xyz="0 0 0" rpy="0 ${radians(90)} 0" />
+      <parent link="${prefix}flange" />
+      <child link="${prefix}tool0" />
+    </joint>
   </xacro:macro>
 </robot>

File: abb_irb6700_support/urdf/irb6700_235_265_macro.xacro (robot description, xacro)
@@ -148,5 +148,4 @@
       </collision>
     </link>
-    <link name="${prefix}tool0"/>
     <joint name="${prefix}joint_1" type="revolute">
       <origin xyz="0 0 0.78" rpy="0 0 0" />
@@ -191,10 +190,4 @@
       <limit lower="-${radians(360)}" upper="${radians(360)}" effort="0" velocity="${radians(190)}" />
     </joint>
-    <joint name="${prefix}joint_6_tool0" type="fixed">
-      <origin xyz="0 0 0" rpy="0 ${radians(90)} 0" />
-      <parent link="${prefix}link_6" />
-      <child link="${prefix}tool0" />
-      <axis xyz="0 0 0" />
-    </joint>
     <joint name="${prefix}cylinder_joint" type="revolute">
       <origin xyz="-0.349 -0.194 -0.142" rpy="0 0 0" />
@@ -213,11 +206,25 @@
       <limit lower="-0.25" upper="0.25" effort="0" velocity="100" />
     </joint>
-    <!-- ROS base_link to ABB World Coordinates transform -->
-    <link name="${prefix}base"/>
-    <joint name="${prefix}base_link_base" type="fixed">
+    <!-- ROS-Industrial 'base' frame: base_link to ABB World Coordinates transform -->
+    <link name="${prefix}base" />
+    <joint name="${prefix}base_link-base" type="fixed">
       <origin xyz="0 0 0" rpy="0 0 0"/>
       <parent link="${prefix}base_link"/>
       <child link="${prefix}base"/>
     </joint>
+    <!-- ROS-Industrial 'flange' frame: attachment point for EEF models -->
+    <link name="${prefix}flange"/>
+    <joint type="fixed" name="${prefix}joint_6-flange">
+      <origin xyz="0 0 0" rpy="0 0 0"/>
+      <parent link="${prefix}link_6"/>
+      <child link="${prefix}flange"/>
+    </joint>
+    <!-- ROS-Industrial 'tool0' frame: all-zeros tool frame -->
+    <link name="${prefix}tool0" />
+    <joint name="${prefix}link_6-tool0" type="fixed">
+      <origin xyz="0 0 0" rpy="0 ${radians(90)} 0" />
+      <parent link="${prefix}flange" />
+      <child link="${prefix}tool0" />
+    </joint>
   </xacro:macro>
 </robot>

Commit message: Updated joint velocities for IRB6700-200/2.6

File: abb_irb6700_support/urdf/irb6700_200_260_macro.xacro (robot description, xacro)
@@ -153,5 +153,5 @@
       <child link="${prefix}link_1" />
       <axis xyz="0 0 1" />
-      <limit lower="-${radians(170)}" upper="${radians(170)}" effort="0" velocity="${radians(100)}" />
+      <limit lower="-${radians(170)}" upper="${radians(170)}" effort="0" velocity="${radians(110)}" />
     </joint>
     <joint name="${prefix}joint_2" type="revolute">
@@ -160,5 +160,5 @@
       <child link="${prefix}link_2" />
       <axis xyz="0 1 0" />
-      <limit lower="-${radians(65)}" upper="${radians(85)}" effort="0" velocity="${radians(90)}" />
+      <limit lower="-${radians(65)}" upper="${radians(85)}" effort="0" velocity="${radians(110)}" />
     </joint>
     <joint name="${prefix}joint_3" type="revolute">
@@ -167,5 +167,5 @@
       <child link="${prefix}link_3" />
       <axis xyz="0 1 0" />
-      <limit lower="-${radians(180)}" upper="${radians(70)}" effort="0" velocity="${radians(90)}" />
+      <limit lower="-${radians(180)}" upper="${radians(70)}" effort="0" velocity="${radians(110)}" />
     </joint>
     <joint name="${prefix}joint_4" type="revolute">
@@ -174,5 +174,5 @@
       <child link="${prefix}link_4" />
       <axis xyz="1 0 0" />
-      <limit lower="-${radians(300)}" upper="${radians(300)}" effort="0" velocity="${radians(170)}" />
+      <limit lower="-${radians(300)}" upper="${radians(300)}" effort="0" velocity="${radians(190)}" />
     </joint>
     <joint name="${prefix}joint_5" type="revolute">
@@ -181,5 +181,5 @@
       <child link="${prefix}link_5" />
       <axis xyz="0 1 0" />
-      <limit lower="-${radians(130)}" upper="${radians(130)}" effort="0" velocity="${radians(120)}" />
+      <limit lower="-${radians(130)}" upper="${radians(130)}" effort="0" velocity="${radians(150)}" />
     </joint>
     <joint name="${prefix}joint_6" type="revolute">
@@ -188,5 +188,5 @@
       <child link="${prefix}link_6" />
       <axis xyz="1 0 0" />
-      <limit lower="-${radians(360)}" upper="${radians(360)}" effort="0" velocity="${radians(190)}" />
+      <limit lower="-${radians(360)}" upper="${radians(360)}" effort="0" velocity="${radians(210)}" />
     </joint>
     <joint name="${prefix}cylinder_joint" type="revolute">
