Commit message: Update irb6660_100_330_macro.xacro
Update link list and joint list parameter to matched ABB IRB6660_100_330 data

File: abb_irb6660_support/urdf/irb6660_100_330_macro.xacro (robot description, xacro)
@@ -39,5 +39,5 @@
         <origin xyz="0 0 0" rpy="0 0 0"/>
         <geometry>
-          <mesh filename="package://abb_irb6660_support/meshes/irb6660/visual/link_2.stl"/>
+          <mesh filename="package://abb_irb6660_support/meshes/irb6660_100_330/visual/link_2.stl"/>
         </geometry>
         <xacro:material_abb_orange />
@@ -46,5 +46,5 @@
         <origin xyz="0 0 0" rpy="0 0 0"/>
         <geometry>
-          <mesh filename="package://abb_irb6660_support/meshes/irb6660/collision/link_2.stl"/>
+          <mesh filename="package://abb_irb6660_support/meshes/irb6660_100_330/collision/link_2.stl"/>
         </geometry>
         <xacro:material_abb_yellow />
@@ -85,14 +85,14 @@
     <link name="${prefix}link_5">
       <visual>
-        <origin xyz="0 0 0" rpy="0 0 0"/>
+        <origin xyz="-0.15 0 0" rpy="0 0 0"/>
         <geometry>
-          <mesh filename="package://abb_irb6660_support/meshes/irb6660/visual/link_5.stl"/>
+          <mesh filename="package://abb_irb6660_support/meshes/irb6660_100_330/visual/link_5.stl"/>
         </geometry>
         <xacro:material_abb_orange />
       </visual>
       <collision>
-        <origin xyz="0 0 0" rpy="0 0 0"/>
+        <origin xyz="-0.15 0 0" rpy="0 0 0"/>
         <geometry>
-          <mesh filename="package://abb_irb6660_support/meshes/irb6660/collision/link_5.stl"/>
+          <mesh filename="package://abb_irb6660_support/meshes/irb6660_100_330/collision/link_5.stl"/>
         </geometry>
         <xacro:material_abb_yellow />
@@ -101,5 +101,5 @@
     <link name="${prefix}link_6">
       <visual>
-        <origin xyz="0 0 0" rpy="0 0 0"/>
+        <origin xyz="-0.15 0 0" rpy="0 0 0"/>
         <geometry>
           <mesh filename="package://abb_irb6660_support/meshes/irb6660/visual/link_6.stl"/>
@@ -108,5 +108,5 @@
       </visual>
       <collision>
-        <origin xyz="0 0 0" rpy="0 0 0"/>
+        <origin xyz="-0.15 0 0" rpy="0 0 0"/>
         <geometry>
           <mesh filename="package://abb_irb6660_support/meshes/irb6660/collision/link_6.stl"/>
@@ -119,16 +119,16 @@
     <!-- joint list -->
     <joint name="${prefix}joint_1" type="revolute">
-      <origin xyz="0 0 0.630" rpy="0 0 0"/>
+      <origin xyz="0 0 0.8145" rpy="0 0 0"/>
       <parent link="${prefix}base_link"/>
       <child link="${prefix}link_1"/>
       <axis xyz="0 0 1"/>
-      <limit lower="-${radians(180)}" upper="${radians(180)}" effort="0" velocity="${radians(100)}"/>
+      <limit lower="-${radians(180)}" upper="${radians(180)}" effort="0" velocity="${radians(110)}"/>
       </joint>
     <joint name="${prefix}joint_2" type="revolute">
-      <origin xyz="0.600 0 0" rpy="0 0 0"/>
+      <origin xyz="0.300 0 0" rpy="0 0 0"/>
       <parent link="${prefix}link_1"/>
       <child link="${prefix}link_2"/>
       <axis xyz="0 1 0"/>
-      <limit lower="-${radians(40)}" upper="${radians(160)}" effort="0" velocity="${radians(90)}"/>
+      <limit lower="-${radians(42)}" upper="${radians(85)}" effort="0" velocity="${radians(130)}"/>
     </joint>
     <joint name="${prefix}joint_3" type="revolute">
@@ -137,8 +137,8 @@
       <child link="${prefix}link_3"/>
       <axis xyz="0 1 0"/>
-      <limit lower="-${radians(180)}" upper="${radians(70)}" effort="0" velocity="${radians(90)}"/>
+      <limit lower="-${radians(20)}" upper="${radians(120)}" effort="0" velocity="${radians(130)}"/>
     </joint>
     <joint name="${prefix}joint_4" type="revolute">
-      <origin xyz="0 0 0.200" rpy="0 0 0"/>
+      <origin xyz="0 0 0.280" rpy="0 0 0"/>
       <parent link="${prefix}link_3"/>
       <child link="${prefix}link_4"/>
@@ -147,5 +147,5 @@
     </joint>
     <joint name="${prefix}joint_5" type="revolute">
-      <origin xyz="2.042 0 0" rpy="0 0 0"/>
+      <origin xyz="1.7555 0 0" rpy="0 0 0"/>
       <parent link="${prefix}link_4"/>
       <child link="${prefix}link_5"/>
@@ -158,5 +158,5 @@
       <child link="${prefix}link_6"/>
       <axis xyz="1 0 0"/>
-      <limit lower="-${radians(360)}" upper="${radians(360)}" effort="0" velocity="${radians(235)}"/>
+      <limit lower="-${radians(360)}" upper="${radians(360)}" effort="0" velocity="${radians(240)}"/>
     </joint>
     <joint name="${prefix}joint_6-tool0" type="fixed">
