Commit message: Update abb_irb6660_100_330 and abb_irb6660_130_310 urdf's, meshes. Upload all 3 vairiances moveit config

File: abb_irb6660_support/urdf/irb6660_130_310_macro.xacro (robot description, xacro)
@@ -39,5 +39,5 @@
         <origin xyz="0 0 0" rpy="0 0 0"/>
         <geometry>
-          <mesh filename="package://abb_irb6660_support/meshes/irb6660/visual/link_2.stl"/>
+          <mesh filename="package://abb_irb6660_support/meshes/irb6660_130_310/visual/link_2.stl"/>
         </geometry>
         <xacro:material_abb_orange />
@@ -46,5 +46,5 @@
         <origin xyz="0 0 0" rpy="0 0 0"/>
         <geometry>
-          <mesh filename="package://abb_irb6660_support/meshes/irb6660/collision/link_2.stl"/>
+          <mesh filename="package://abb_irb6660_support/meshes/irb6660_130_310/collision/link_2.stl"/>
         </geometry>
         <xacro:material_abb_yellow />
@@ -69,5 +69,5 @@
     <link name="${prefix}link_4">
       <visual>
-        <origin xyz="-0.600 0 0" rpy="0 0 0"/>
+        <origin xyz="0 0 0" rpy="0 0 0"/>
         <geometry>
           <mesh filename="package://abb_irb6660_support/meshes/irb6660_130_310/visual/link_4.stl"/>
@@ -76,5 +76,5 @@
       </visual>
       <collision>
-        <origin xyz="-0.600 0 0" rpy="0 0 0"/>
+        <origin xyz="0 0 0" rpy="0 0 0"/>
         <geometry>
             <mesh filename="package://abb_irb6660_support/meshes/irb6660_130_310/collision/link_4.stl"/>
@@ -85,5 +85,5 @@
     <link name="${prefix}link_5">
       <visual>
-        <origin xyz="0 0 0" rpy="0 0 0"/>
+        <origin xyz="-0.15 0 0" rpy="0 0 0"/>
         <geometry>
           <mesh filename="package://abb_irb6660_support/meshes/irb6660/visual/link_5.stl"/>
@@ -92,5 +92,5 @@
       </visual>
       <collision>
-        <origin xyz="0 0 0" rpy="0 0 0"/>
+        <origin xyz="-0.15 0 0" rpy="0 0 0"/>
         <geometry>
           <mesh filename="package://abb_irb6660_support/meshes/irb6660/collision/link_5.stl"/>
@@ -101,5 +101,5 @@
     <link name="${prefix}link_6">
       <visual>
-        <origin xyz="0 0 0" rpy="0 0 0"/>
+        <origin xyz="-0.15 0 0" rpy="0 0 0"/>
         <geometry>
           <mesh filename="package://abb_irb6660_support/meshes/irb6660/visual/link_6.stl"/>
@@ -108,5 +108,5 @@
       </visual>
       <collision>
-        <origin xyz="0 0 0" rpy="0 0 0"/>
+        <origin xyz="-0.15 0 0" rpy="0 0 0"/>
         <geometry>
           <mesh filename="package://abb_irb6660_support/meshes/irb6660/collision/link_6.stl"/>
@@ -130,12 +130,12 @@
       <child link="${prefix}link_2"/>
       <axis xyz="0 1 0"/>
-      <limit lower="-${radians(40)}" upper="${radians(160)}" effort="0" velocity="${radians(90)}"/>
+      <limit lower="-${radians(42)}" upper="${radians(85)}" effort="0" velocity="${radians(130)}"/>
     </joint>
     <joint name="${prefix}joint_3" type="revolute">
-      <origin xyz="0 0 0.700" rpy="0 0 0"/>
+      <origin xyz="0 0 1.280" rpy="0 0 0"/>
       <parent link="${prefix}link_2"/>
       <child link="${prefix}link_3"/>
       <axis xyz="0 1 0"/>
-      <limit lower="-${radians(180)}" upper="${radians(70)}" effort="0" velocity="${radians(90)}"/>
+      <limit lower="-${radians(20)}" upper="${radians(120)}" effort="0" velocity="${radians(130)}"/>
     </joint>
     <joint name="${prefix}joint_4" type="revolute">
@@ -147,5 +147,5 @@
     </joint>
     <joint name="${prefix}joint_5" type="revolute">
-      <origin xyz="0.893 0 0" rpy="0 0 0"/>
+      <origin xyz="1.5055 0 0" rpy="0 0 0"/>
       <parent link="${prefix}link_4"/>
       <child link="${prefix}link_5"/>
@@ -158,5 +158,5 @@
       <child link="${prefix}link_6"/>
       <axis xyz="1 0 0"/>
-      <limit lower="-${radians(360)}" upper="${radians(360)}" effort="0" velocity="${radians(235)}"/>
+      <limit lower="-${radians(360)}" upper="${radians(360)}" effort="0" velocity="${radians(240)}"/>
     </joint>
     <joint name="${prefix}joint_6-tool0" type="fixed">

File: abb_irb6660_support/urdf/irb6660_205_190_macro.xacro (robot description, xacro)
@@ -123,5 +123,5 @@
       <child link="${prefix}link_1"/>
       <axis xyz="0 0 1"/>
-      <limit lower="-${radians(180)}" upper="${radians(180)}" effort="0" velocity="${radians(110)}"/>
+      <limit lower="-${radians(180)}" upper="${radians(180)}" effort="0" velocity="${radians(130)}"/>
     </joint>
     <joint name="${prefix}joint_2" type="revolute">
@@ -130,5 +130,5 @@
       <child link="${prefix}link_2"/>
       <axis xyz="0 1 0"/>
-      <limit lower="-${radians(40)}" upper="${radians(160)}" effort="0" velocity="${radians(90)}"/>
+      <limit lower="-${radians(42)}" upper="${radians(85)}" effort="0" velocity="${radians(130)}"/>
     </joint>
     <joint name="${prefix}joint_3" type="revolute">
@@ -137,5 +137,5 @@
       <child link="${prefix}link_3"/>
       <axis xyz="0 1 0"/>
-      <limit lower="-${radians(180)}" upper="${radians(70)}" effort="0" velocity="${radians(90)}"/>
+      <limit lower="-${radians(20)}" upper="${radians(120)}" effort="0" velocity="${radians(130)}"/>
     </joint>
     <joint name="${prefix}joint_4" type="revolute">
@@ -158,5 +158,5 @@
       <child link="${prefix}link_6"/>
       <axis xyz="1 0 0"/>
-      <limit lower="-${radians(360)}" upper="${radians(360)}" effort="0" velocity="${radians(235)}"/>
+      <limit lower="-${radians(360)}" upper="${radians(360)}" effort="0" velocity="${radians(190)}"/>
     </joint>
     <joint name="${prefix}joint_6-tool0" type="fixed">
