Commit message: adding updated joint limits for joint 3 (dynamic axis causes problems)

File: abb_irb6660_support/urdf/irb6660_205_190_macro.xacro (robot description, xacro)
@@ -137,5 +137,5 @@
       <child link="${prefix}link_3"/>
       <axis xyz="0 1 0"/>
-      <limit lower="-${radians(20)}" upper="${radians(120)}" effort="0" velocity="${radians(130)}"/>
+      <limit lower="-${radians(70)}" upper="${radians(70)}" effort="0" velocity="${radians(130)}"/>
     </joint>
     <joint name="${prefix}joint_4" type="revolute">
