Commit message: Re-arrange abb_irb1200 xacros

File: abb_irb1200_gazebo/urdf/irb1200_5_90.xacro (robot description, xacro)
@@ -2,9 +2,5 @@
 <robot name="abb_irb1200_5_90" xmlns:xacro="http://ros.org/wiki/xacro">
   <xacro:include filename="$(find abb_irb1200_gazebo)/urdf/irb1200_5_90_macro.xacro" />
-  <xacro:include filename="$(find abb_irb1200_support)/urdf/irb1200_5_90_macro.xacro" />
-  <!-- get base ABB IRB1200 model -->
-  <xacro:abb_irb1200_5_90 prefix="" />
-  <!-- get gazebo add-ons -->
-  <xacro:abb_irb1200_5_90_gazebo_spec prefix="" />
+  <xacro:abb_irb1200_5_90_gazebo prefix="" />
   <!-- connect robot with world -->
   <link name="world" />

File: abb_irb1200_gazebo/urdf/irb1200_5_90_macro.xacro (robot description, xacro)
@@ -1,5 +1,8 @@
 <?xml version="1.0"?>
 <robot xmlns:xacro="http://ros.org/wiki/xacro">
-  <xacro:macro name="abb_irb1200_5_90_gazebo_spec" params="prefix">
+  <xacro:include filename="$(find abb_irb1200_support)/urdf/irb1200_5_90_macro.xacro" />
+  <xacro:macro name="abb_irb1200_5_90_gazebo" params="prefix">
+    <!-- get base ABB IRB1200 model -->
+    <xacro:abb_irb1200_5_90 prefix="${prefix}" />
     <!-- transmission list -->
     <transmission name="${prefix}tran1">
