Commit message: Added flange frame for irb2600

File: abb_irb2600_support/urdf/irb2600_12_165_macro.xacro (robot description, xacro)
@@ -111,5 +111,4 @@
       </collision>
     </link>
-    <link name="${prefix}tool0" />
     <!-- Joints -->
     <joint name="${prefix}joint_1" type="revolute">
@@ -155,15 +154,24 @@
       <limit lower="-6.981" upper="6.981" effort="0" velocity="8.727" />
     </joint>
-    <joint name="${prefix}joint6-tool0" type="fixed">
-      <origin xyz="0 0 0" rpy="0 1.5707963267948966 0" />
-      <parent link="${prefix}link_6" />
-      <child link="${prefix}tool0" />
-    </joint>
-    <!-- ROS base_link to ABB World Coordinates transform -->
+    <!-- ROS-Industrial 'base' frame: base_link to ABB World Coordinates transform -->
     <link name="${prefix}base" />
     <joint name="${prefix}base_link-base" type="fixed">
-      <origin xyz="0 0 0" rpy="0 0 0" />
-      <parent link="${prefix}base_link" />
-      <child link="${prefix}base" />
+      <origin xyz="0 0 0" rpy="0 0 0"/>
+      <parent link="${prefix}base_link"/>
+      <child link="${prefix}base"/>
+    </joint>
+    <!-- ROS-Industrial 'flange' frame: attachment point for EEF models -->
+    <link name="${prefix}flange"/>
+    <joint type="fixed" name="${prefix}joint_6-flange">
+      <origin xyz="0 0 0" rpy="0 0 0"/>
+      <parent link="${prefix}link_6"/>
+      <child link="${prefix}flange"/>
+    </joint>
+    <!-- ROS-Industrial 'tool0' frame: all-zeros tool frame -->
+    <link name="${prefix}tool0" />
+    <joint name="${prefix}link_6-tool0" type="fixed">
+      <origin xyz="0 0 0" rpy="0 ${radians(90)} 0" />
+      <parent link="${prefix}flange" />
+      <child link="${prefix}tool0" />
     </joint>
   </xacro:macro>
