Commit message: changes to urdf and mesh of link 2

File: abb_irb2600_support/urdf/irb2600_12_185_macro.xacro (robot description, xacro)
@@ -36,5 +36,5 @@
     <link name="${prefix}link_2">
       <visual>
-        <origin xyz="0 0 0" rpy="0 0 0" />
+        <origin xyz="-0.15 0 -0.445" rpy="0 0 0" />
         <geometry>
           <mesh filename="package://abb_irb2600_support/meshes/irb2600_12_185/visual/link_2.stl" />
@@ -127,5 +127,5 @@
     </joint>
     <joint name="${prefix}joint_3" type="revolute">
-      <origin xyz="0 0 0.7" rpy="0 0 0" />
+      <origin xyz="0 0 0.9" rpy="0 0 0" />
       <parent link="${prefix}link_2" />
       <child link="${prefix}link_3" />

Commit message: correct position of collision stl

File: abb_irb2600_support/urdf/irb2600_12_185_macro.xacro (robot description, xacro)
@@ -43,5 +43,5 @@
       </visual>
       <collision>
-        <origin xyz="0 0 0" rpy="0 0 0" />
+        <origin xyz="-0.15 0 -0.445" rpy="0 0 0" />
         <geometry>
           <mesh filename="package://abb_irb2600_support/meshes/irb2600_12_185/collision/link_2.stl" />
