Commit message: Added support for CRB 15000-12

File: abb_crb15000_support/urdf/crb15000_12_127_macro.xacro (robot description, xacro)
@@ -46,10 +46,10 @@
       <collision>
         <geometry>
-          <mesh filename="package://abb_crb15000_support/meshes/crb15000_12_127/collision/link_3.stl"/>
+          <mesh filename="package://abb_crb15000_support/meshes/crb15000_5_95/collision/link_3.stl"/>
         </geometry>
       </collision>
       <visual>
         <geometry>
-          <mesh filename="package://abb_crb15000_support/meshes/crb15000_12_127/visual/link_3.stl"/>
+          <mesh filename="package://abb_crb15000_support/meshes/crb15000_5_95/visual/link_3.stl"/>
         </geometry>
         <xacro:material_abb_dark_gray />
@@ -72,10 +72,10 @@
       <collision>
         <geometry>
-          <mesh filename="package://abb_crb15000_support/meshes/crb15000_12_127/collision/link_5.stl"/>
+          <mesh filename="package://abb_crb15000_support/meshes/crb15000_5_95/collision/link_5.stl"/>
         </geometry>
       </collision>
       <visual>
         <geometry>
-          <mesh filename="package://abb_crb15000_support/meshes/crb15000_12_127/visual/link_5.stl"/>
+          <mesh filename="package://abb_crb15000_support/meshes/crb15000_5_95/visual/link_5.stl"/>
         </geometry>
         <xacro:material_abb_graphite_white />
@@ -85,10 +85,10 @@
       <collision>
         <geometry>
-          <mesh filename="package://abb_crb15000_support/meshes/crb15000_12_127/collision/link_6.stl"/>
+          <mesh filename="package://abb_crb15000_support/meshes/crb15000_5_95/collision/link_6.stl"/>
         </geometry>
       </collision>
       <visual>
         <geometry>
-          <mesh filename="package://abb_crb15000_support/meshes/crb15000_12_127/visual/link_6.stl"/>
+          <mesh filename="package://abb_crb15000_support/meshes/crb15000_5_95/visual/link_6.stl"/>
         </geometry>
         <xacro:material_abb_gray_white />

Commit message: Unified mesh normals, fixed joint and speed limits.

File: abb_crb15000_support/urdf/crb15000_12_127_macro.xacro (robot description, xacro)
@@ -102,5 +102,5 @@
       <parent link="${prefix}base_link"/>
       <child link="${prefix}link_1"/>
-      <limit effort="0" lower="${radians(-180)}" upper="${radians(180)}" velocity="${radians(125)}"/>
+      <limit effort="0" lower="${radians(-270)}" upper="${radians(270)}" velocity="${radians(120)}"/>
     </joint>
     <joint type="revolute" name="${prefix}joint_2">
@@ -109,5 +109,5 @@
       <parent link="${prefix}link_1"/>
       <child link="${prefix}link_2"/>
-      <limit effort="0" lower="${radians(-180)}" upper="${radians(180)}" velocity="${radians(125)}"/>
+      <limit effort="0" lower="${radians(-180)}" upper="${radians(180)}" velocity="${radians(120)}"/>
     </joint>
     <joint type="revolute" name="${prefix}joint_3">
@@ -116,5 +116,5 @@
       <parent link="${prefix}link_2"/>
       <child link="${prefix}link_3"/>
-      <limit effort="0" lower="${radians(-225)}" upper="${radians(85)}" velocity="${radians(140)}"/>
+      <limit effort="0" lower="${radians(-225)}" upper="${radians(85)}" velocity="${radians(125)}"/>
     </joint>
     <joint type="revolute" name="${prefix}joint_4">
@@ -137,5 +137,5 @@
       <parent link="${prefix}link_5"/>
       <child link="${prefix}link_6"/>
-      <limit effort="0" lower="${radians(-180)}" upper="${radians(180)}" velocity="${radians(200)}"/>
+      <limit effort="0" lower="${radians(-270)}" upper="${radians(270)}" velocity="${radians(200)}"/>
     </joint>
     <!-- end of joint list -->
