Commit message: Change name to irb140t_6_8

File: abb_irb140_support/urdf/irb140t_6_8_macro.xacro (robot description, xacro)
@@ -1,5 +1,5 @@
 <?xml version="1.0"?>
-<robot xmlns:xacro="http://ros.org/wiki/xacro" name="irb140t_6_81">
-<xacro:macro name="abb_irb140t_6_81" params="prefix">
+<robot xmlns:xacro="http://ros.org/wiki/xacro" name="irb140t_6_8">
+<xacro:macro name="abb_irb140t_6_8" params="prefix">
   <xacro:include filename="$(find abb_resources)/urdf/common_materials.xacro"/>
   <!-- link list -->
@@ -8,5 +8,5 @@
       <origin xyz="0 0 0" rpy="0 0 0"/>
       <geometry>
-        <mesh filename="package://abb_irb140_support/meshes/irb140t_6_81/visual/base_link.stl"/>
+        <mesh filename="package://abb_irb140_support/meshes/irb140t_6_8/visual/base_link.stl"/>
       </geometry>
       <xacro:material_abb_orange/>
@@ -14,5 +14,5 @@
     <collision>
       <geometry>
-        <mesh filename="package://abb_irb140_support/meshes/irb140t_6_81/collision/base_link.stl"/>
+        <mesh filename="package://abb_irb140_support/meshes/irb140t_6_8/collision/base_link.stl"/>
       </geometry>
       <xacro:material_abb_yellow/>
@@ -23,5 +23,5 @@
       <origin xyz="0 0 0" rpy="0 0 0"/>
       <geometry>
-        <mesh filename="package://abb_irb140_support/meshes/irb140t_6_81/visual/link_1.stl"/>
+        <mesh filename="package://abb_irb140_support/meshes/irb140t_6_8/visual/link_1.stl"/>
       </geometry>
       <xacro:material_abb_orange/>
@@ -30,5 +30,5 @@
       <origin xyz="0 0 0" rpy="0 0 0"/>
       <geometry>
-        <mesh filename="package://abb_irb140_support/meshes/irb140t_6_81/collision/link_1.stl"/>
+        <mesh filename="package://abb_irb140_support/meshes/irb140t_6_8/collision/link_1.stl"/>
       </geometry>
       <xacro:material_abb_yellow/>
@@ -39,5 +39,5 @@
       <origin xyz="0 0 0" rpy="0 0 0"/>
       <geometry>
-        <mesh filename="package://abb_irb140_support/meshes/irb140t_6_81/visual/link_2.stl"/>
+        <mesh filename="package://abb_irb140_support/meshes/irb140t_6_8/visual/link_2.stl"/>
       </geometry>
       <xacro:material_abb_orange/>
@@ -46,5 +46,5 @@
       <origin xyz="0 0 0" rpy="0 0 0"/>
       <geometry>
-        <mesh filename="package://abb_irb140_support/meshes/irb140t_6_81/collision/link_2.stl"/>
+        <mesh filename="package://abb_irb140_support/meshes/irb140t_6_8/collision/link_2.stl"/>
       </geometry>
       <xacro:material_abb_yellow/>
@@ -55,5 +55,5 @@
       <origin xyz="0 0 0" rpy="0 0 0"/>
       <geometry>
-        <mesh filename="package://abb_irb140_support/meshes/irb140t_6_81/visual/link_3.stl"/>
+        <mesh filename="package://abb_irb140_support/meshes/irb140t_6_8/visual/link_3.stl"/>
       </geometry>
       <xacro:material_abb_orange/>
@@ -62,5 +62,5 @@
       <origin xyz="0 0 0" rpy="0 0 0"/>
       <geometry>
-        <mesh filename="package://abb_irb140_support/meshes/irb140t_6_81/collision/link_3.stl"/>
+        <mesh filename="package://abb_irb140_support/meshes/irb140t_6_8/collision/link_3.stl"/>
       </geometry>
       <xacro:material_abb_yellow/>
@@ -71,5 +71,5 @@
       <origin xyz="0 0 0" rpy="0 0 0"/>
       <geometry>
-        <mesh filename="package://abb_irb140_support/meshes/irb140t_6_81/visual/link_4.stl"/>
+        <mesh filename="package://abb_irb140_support/meshes/irb140t_6_8/visual/link_4.stl"/>
       </geometry>
       <xacro:material_abb_orange/>
@@ -78,5 +78,5 @@
       <origin xyz="0 0 0" rpy="0 0 0"/>
       <geometry>
-        <mesh filename="package://abb_irb140_support/meshes/irb140t_6_81/collision/link_4.stl"/>
+        <mesh filename="package://abb_irb140_support/meshes/irb140t_6_8/collision/link_4.stl"/>
       </geometry>
       <xacro:material_abb_yellow/>
@@ -87,5 +87,5 @@
       <origin xyz="0 0 0" rpy="0 0 0"/>
       <geometry>
-        <mesh filename="package://abb_irb140_support/meshes/irb140t_6_81/visual/link_5.stl"/>
+        <mesh filename="package://abb_irb140_support/meshes/irb140t_6_8/visual/link_5.stl"/>
       </geometry>
       <xacro:material_abb_orange/>
@@ -94,5 +94,5 @@
       <origin xyz="0 0 0" rpy="0 0 0"/>
       <geometry>
-        <mesh filename="package://abb_irb140_support/meshes/irb140t_6_81/collision/link_5.stl"/>
+        <mesh filename="package://abb_irb140_support/meshes/irb140t_6_8/collision/link_5.stl"/>
       </geometry>
       <xacro:material_abb_yellow/>
@@ -103,5 +103,5 @@
       <origin xyz="0 0 0" rpy="0 0 0"/>
       <geometry>
-        <mesh filename="package://abb_irb140_support/meshes/irb140t_6_81/visual/link_6.stl"/>
+        <mesh filename="package://abb_irb140_support/meshes/irb140t_6_8/visual/link_6.stl"/>
       </geometry>
       <xacro:material_abb_orange/>
@@ -110,5 +110,5 @@
       <origin xyz="0 0 0" rpy="0 0 0"/>
       <geometry>
-        <mesh filename="package://abb_irb140_support/meshes/irb140t_6_81/collision/link_6.stl"/>
+        <mesh filename="package://abb_irb140_support/meshes/irb140t_6_8/collision/link_6.stl"/>
       </geometry>
       <xacro:material_abb_yellow/>
