Commit message: Add irb1300 variants 7/1.4 and 12/1.4

File: abb_irb1300_support/urdf/irb1300_12_140_macro.xacro (robot description, xacro)
@@ -1,5 +1,5 @@
 <?xml version="1.0"?>
-<robot xmlns:xacro="http://ros.org/wiki/xacro" name="irb1300_10_115">
-<xacro:macro name="abb_irb1300_10_115" params="prefix">
+<robot xmlns:xacro="http://ros.org/wiki/xacro" name="irb1300_12_140">
+<xacro:macro name="abb_irb1300_12_140" params="prefix">
   <xacro:include filename="$(find abb_resources)/urdf/common_materials.xacro"/>
   <!-- link list -->
@@ -71,5 +71,5 @@
       <origin xyz="0 0 0" rpy="0 0 0"/>
       <geometry>
-        <mesh filename="package://abb_irb1300_support/meshes/irb1300_10_115/visual/link_4.stl"/>
+        <mesh filename="package://abb_irb1300_support/meshes/irb1300_xx_140/visual/link_4.stl"/>
       </geometry>
       <xacro:material_abb_white/>
@@ -78,5 +78,5 @@
       <origin xyz="0 0 0" rpy="0 0 0"/>
       <geometry>
-        <mesh filename="package://abb_irb1300_support/meshes/irb1300_10_115/collision/link_4.stl"/>
+        <mesh filename="package://abb_irb1300_support/meshes/irb1300_xx_140/collision/link_4.stl"/>
       </geometry>
       <xacro:material_abb_yellow/>
@@ -122,5 +122,5 @@
     <child link="${prefix}link_1"/>
     <axis xyz="0 0 1"/>
-    <limit lower="${radians(-180)}" upper="${radians(180)}" effort="0" velocity="${radians(280)}"/>
+    <limit lower="${radians(-180)}" upper="${radians(180)}" effort="0" velocity="${radians(230)}"/>
   </joint>
   <joint name="${prefix}joint_2" type="revolute">
@@ -129,5 +129,5 @@
     <child link="${prefix}link_2"/>
     <axis xyz="0 1 0"/>
-    <limit lower="${radians(-95)}" upper="${radians(155)}" effort="0" velocity="${radians(228)}"/>
+    <limit lower="${radians(-95)}" upper="${radians(155)}" effort="0" velocity="${radians(116)}"/>
   </joint>
   <joint name="${prefix}joint_3" type="revolute">
@@ -136,8 +136,8 @@
     <child link="${prefix}link_3"/>
     <axis xyz="0 1 0"/>
-    <limit lower="${radians(-210)}" upper="${radians(65)}" effort="0" velocity="${radians(336)}"/>
+    <limit lower="${radians(-210)}" upper="${radians(69)}" effort="0" velocity="${radians(138)}"/>
   </joint>
   <joint name="${prefix}joint_4" type="revolute">
-    <origin xyz="0.425 0 0.040" rpy="0 0 0"/>
+    <origin xyz="0.675 0 0.040" rpy="0 0 0"/>
     <parent link="${prefix}link_3"/>
     <child link="${prefix}link_4"/>
@@ -157,5 +157,5 @@
     <child link="${prefix}link_6"/>
     <axis xyz="1 0 0"/>
-    <limit lower="${radians(-400)}" upper="${radians(400)}" effort="0" velocity="${radians(720)}"/>
+    <limit lower="${radians(-400)}" upper="${radians(400)}" effort="0" velocity="${radians(687)}"/>
   </joint>
   <!-- end of joint list -->

File: abb_irb1300_support/urdf/irb1300_7_140_macro.xacro (robot description, xacro)
@@ -1,5 +1,5 @@
 <?xml version="1.0"?>
-<robot xmlns:xacro="http://ros.org/wiki/xacro" name="irb1300_10_115">
-<xacro:macro name="abb_irb1300_10_115" params="prefix">
+<robot xmlns:xacro="http://ros.org/wiki/xacro" name="irb1300_7_140">
+<xacro:macro name="abb_irb1300_7_140" params="prefix">
   <xacro:include filename="$(find abb_resources)/urdf/common_materials.xacro"/>
   <!-- link list -->
@@ -71,5 +71,5 @@
       <origin xyz="0 0 0" rpy="0 0 0"/>
       <geometry>
-        <mesh filename="package://abb_irb1300_support/meshes/irb1300_10_115/visual/link_4.stl"/>
+        <mesh filename="package://abb_irb1300_support/meshes/irb1300_xx_140/visual/link_4.stl"/>
       </geometry>
       <xacro:material_abb_white/>
@@ -78,5 +78,5 @@
       <origin xyz="0 0 0" rpy="0 0 0"/>
       <geometry>
-        <mesh filename="package://abb_irb1300_support/meshes/irb1300_10_115/collision/link_4.stl"/>
+        <mesh filename="package://abb_irb1300_support/meshes/irb1300_xx_140/collision/link_4.stl"/>
       </geometry>
       <xacro:material_abb_yellow/>
@@ -122,5 +122,5 @@
     <child link="${prefix}link_1"/>
     <axis xyz="0 0 1"/>
-    <limit lower="${radians(-180)}" upper="${radians(180)}" effort="0" velocity="${radians(280)}"/>
+    <limit lower="${radians(-180)}" upper="${radians(180)}" effort="0" velocity="${radians(255)}"/>
   </joint>
   <joint name="${prefix}joint_2" type="revolute">
@@ -129,5 +129,5 @@
     <child link="${prefix}link_2"/>
     <axis xyz="0 1 0"/>
-    <limit lower="${radians(-95)}" upper="${radians(155)}" effort="0" velocity="${radians(228)}"/>
+    <limit lower="${radians(-95)}" upper="${radians(155)}" effort="0" velocity="${radians(180)}"/>
   </joint>
   <joint name="${prefix}joint_3" type="revolute">
@@ -136,8 +136,8 @@
     <child link="${prefix}link_3"/>
     <axis xyz="0 1 0"/>
-    <limit lower="${radians(-210)}" upper="${radians(65)}" effort="0" velocity="${radians(336)}"/>
+    <limit lower="${radians(-210)}" upper="${radians(69)}" effort="0" velocity="${radians(247)}"/>
   </joint>
   <joint name="${prefix}joint_4" type="revolute">
-    <origin xyz="0.425 0 0.040" rpy="0 0 0"/>
+    <origin xyz="0.675 0 0.040" rpy="0 0 0"/>
     <parent link="${prefix}link_3"/>
     <child link="${prefix}link_4"/>
